File: KiCAD/distributor/distributor.sch (KiCad schematic (older format))
At the start: 22 parts, among them P1 CONN_02X03, P10 CONN_02X03, P11 CONN_02X03, P12 CONN_02X03, P13 CONN_02X03, P14 CONN_02X03, P15 CONN_02X03, P16 CONN_02X03, P17 CONN_02X03, P18 CONN_02X03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

Commit message: tight spacing 30x30x5 distributor boards done
Connections:
- net +3V3: now also P10.1 (P1), P14.1 (P1), P18.1 (P1), P2.1 (P1), P22.41 (P41), P6.1 (P1); no longer P10.6 (P6), P14.6 (P6), P18.5 (P5), P2.6 (P6), P22.3 (P3), P6.6 (P6)
- net +5V: now also P12.5 (P5), P16.5 (P5), P20.5 (P5), P22.43 (P43), P4.5 (P5), P8.5 (P5); no longer P12.2 (P2), P16.2 (P2), P20.1 (P1), P22.1 (P1), P4.2 (P2), P8.2 (P2)
- net A1_I: now also P2.3 (P3), P22.3 (P3); no longer P2.4 (P4), P22.41 (P41)
- net A1_V: now also P2.4 (P4), P22.4 (P4); no longer P2.3 (P3), P22.42 (P42)
- net A3_I: now also P22.5 (P5), P4.3 (P3); no longer P22.39 (P39), P4.4 (P4)
- net A3_V: now also P22.6 (P6), P4.4 (P4); no longer P22.40 (P40), P4.3 (P3)
- net A5_I: now also P22.7 (P7), P4.1 (P1); no longer P22.37 (P37), P4.6 (P6)
- net A5_V: now also P22.8 (P8), P4.2 (P2); no longer P22.38 (P38), P4.5 (P5)
- net AL_I: now also P2.5 (P5), P22.1 (P1); no longer P2.2 (P2), P22.43 (P43)
- net AL_V: now also P2.6 (P6), P22.2 (P2); no longer P2.1 (P1), P22.44 (P44)
- net B1_I: now also P22.11 (P11), P6.3 (P3); no longer P22.33 (P33), P6.4 (P4)
- net B1_V: now also P22.12 (P12), P6.4 (P4); no longer P22.34 (P34), P6.3 (P3)
- net B3_I: now also P22.13 (P13), P8.3 (P3); no longer P22.31 (P31), P8.4 (P4)
- net B3_V: now also P22.14 (P14), P8.4 (P4); no longer P22.32 (P32), P8.3 (P3)
- net B5_I: now also P22.15 (P15), P8.1 (P1); no longer P22.29 (P29), P8.6 (P6)
- net B5_V: now also P22.16 (P16), P8.2 (P2); no longer P22.30 (P30), P8.5 (P5)
- net BL_I: now also P22.9 (P9), P6.5 (P5); no longer P22.35 (P35), P6.2 (P2)
- net BL_V: now also P22.10 (P10), P6.6 (P6); no longer P22.36 (P36), P6.1 (P1)
- net C1_I: now also P10.3 (P3), P22.19 (P19); no longer P10.4 (P4), P22.25 (P25)
- net C1_V: now also P10.4 (P4), P22.20 (P20); no longer P10.3 (P3), P22.26 (P26)
- net C3_I: now also P12.3 (P3), P22.21 (P21); no longer P12.4 (P4), P22.23 (P23)
- net C3_V: now also P12.4 (P4), P22.22 (P22); no longer P12.3 (P3), P22.24 (P24)
- net C5_I: now also P12.1 (P1), P22.23 (P23); no longer P12.6 (P6), P22.21 (P21)
- net C5_V: now also P12.2 (P2), P22.24 (P24); no longer P12.5 (P5), P22.22 (P22)
- net CL_I: now also P10.5 (P5), P22.17 (P17); no longer P10.2 (P2), P22.27 (P27)
- net CL_V: now also P10.6 (P6), P22.18 (P18); no longer P10.1 (P1), P22.28 (P28)
- net D1_I: now also P14.3 (P3), P22.27 (P27); no longer P14.4 (P4), P22.17 (P17)
- net D1_V: now also P14.4 (P4), P22.28 (P28); no longer P14.3 (P3), P22.18 (P18)
- net D3_I: now also P16.3 (P3), P22.29 (P29); no longer P16.4 (P4), P22.15 (P15)
- net D3_V: now also P16.4 (P4), P22.30 (P30); no longer P16.3 (P3), P22.16 (P16)
- net D5_I: now also P16.1 (P1), P22.31 (P31); no longer P16.6 (P6), P22.13 (P13)
- net D5_V: now also P16.2 (P2), P22.32 (P32); no longer P16.5 (P5), P22.14 (P14)
- net DL_I: now also P14.5 (P5), P22.25 (P25); no longer P14.2 (P2), P22.19 (P19)
- net DL_V: now also P14.6 (P6), P22.26 (P26); no longer P14.1 (P1), P22.20 (P20)
- net E1_I: now also P22.35 (P35); no longer P22.9 (P9)
- net E1_V: now also P22.36 (P36); no longer P22.10 (P10)
- net E3_I: now also P22.37 (P37); no longer P22.7 (P7)
- net E3_V: now also P22.38 (P38); no longer P22.8 (P8)
- net E5_I: now also P20.1 (P1), P22.39 (P39); no longer P20.5 (P5), P22.5 (P5)
- net E5_V: now also P20.2 (P2), P22.40 (P40); no longer P20.6 (P6), P22.6 (P6)
- net EL_I: now also P18.5 (P5), P22.33 (P33); no longer P18.1 (P1), P22.11 (P11)
- net EL_V: now also P18.6 (P6), P22.34 (P34); no longer P18.2 (P2), P22.12 (P12)
- net GND: now also P12.6 (P6), P16.6 (P6), P20.6 (P6), P22.44 (P44), P4.6 (P6), P8.6 (P6); no longer P12.1 (P1), P16.1 (P1), P20.2 (P2), P22.2 (P2), P4.1 (P1), P8.1 (P1)
- net SCK: now also P10.2 (P2), P14.2 (P2), P18.2 (P2), P2.2 (P2), P22.42 (P42), P6.2 (P2); no longer P10.5 (P5), P14.5 (P5), P18.6 (P6), P2.5 (P5), P22.4 (P4), P6.5 (P5)
Changed lines of the file:
@@
 F 3 "" H 3050 1250 50  0000 C CNN
 	1    3050 2450
-	0    -1   -1   0
+	0    1    1    0
 $EndComp
 $Comp
@@
 F 3 "" H 4400 1250 50  0000 C CNN
 	1    4400 2450
-	0    -1   -1   0
+	0    1    1    0
 $EndComp
 Text GLabel 2950 2200 1    60   Input ~ 0
@@
 F 3 "" H 950 1250 50  0000 C CNN
 	1    950  2450
-	0    -1   -1   0
+	0    1    1    0
 $EndComp
 $Comp
@@
 F 3 "" H 2300 1250 50  0000 C CNN
 	1    2300 2450
-	0    -1   -1   0
+	0    1    1    0
 $EndComp
 Text GLabel 850  2200 1    60   Input ~ 0
@@
 F 3 "" H 7250 1250 50  0000 C CNN
 	1    7250 2450
-	0    -1   -1   0
+	0    1    1    0
 $EndComp
 $Comp
@@
 F 3 "" H 8600 1250 50  0000 C CNN
 	1    8600 2450
-	0    -1   -1   0
+	0    1    1    0
 $EndComp
 Text GLabel 7150 2200 1    60   Input ~ 0
@@
 F 3 "" H 5150 1250 50  0000 C CNN
 	1    5150 2450
-	0    -1   -1   0
+	0    1    1    0
 $EndComp
 $Comp
@@
 F 3 "" H 6500 1250 50  0000 C CNN
 	1    6500 2450
-	0    -1   -1   0
+	0    1    1    0
 $EndComp
 Text GLabel 5050 2200 1    60   Input ~ 0
@@
 F 3 "" H 9350 1250 50  0000 C CNN
 	1    9350 2450
-	0    -1   1    0
+	0    1    1    0
 $EndComp
 $Comp
@@
 F 3 "" H 10700 1250 50  0000 C CNN
 	1    10700 2450
-	0    -1   1    0
+	0    1    1    0
 $EndComp
 Text GLabel 9250 2200 1    60   Input ~ 0
@@
 F 3 "" H 8050 4150 50  0000 C CNN
 	1    8050 5050
-	0    1    1    0
-$EndComp
-$Comp
+	0    -1   1    0
+$EndComp
+$Comp
