File: KiCAD/distributor8/A.kicad_pcb (KiCad board)
At the start: 4 copper layers, 431.8 x 25.4 mm, 29 parts, among them P1 CONN_02X03, P11 CONN_02X03, P13 CONN_02X03, P15 CONN_02X03, P17 CONN_02X03, P19 CONN_02X03, P23 CONN_02X07, P24 CONN_02X07, P29 CONN_02X07, P3 CONN_02X03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

Commit message: distributor 8B layout done
Other:
- board text added: "v0.11"
Changed lines of the file:
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@@
   (general
     (links 125)
-    (no_connects 1)
+    (no_connects 0)
     (area -12.775001 -0.075001 419.175001 25.475001)
     (thickness 1.6)
-    (drawings 20)
+    (drawings 21)
     (tracks 1232)
     (zones 0)
@@
   (page A4)
   (layers
-    (0 F.Cu signal)
-    (1 In1.Cu signal)
-    (2 In2.Cu signal)
-    (31 B.Cu signal)
+    (0 F.Cu signal hide)
+    (1 In1.Cu signal hide)
+    (2 In2.Cu signal hide)
+    (31 B.Cu signal hide)
     (32 B.Adhes user)
     (33 F.Adhes user)
@@
   (module myParts:FTMH-103-03-L-DH (layer F.Cu)
     (at 224.7 5.763)
-    (fp_text reference P48 (at 1.6 4.55 180) (layer F.SilkS)
+    (fp_text reference P48 (at 0.04 4.947 180) (layer F.SilkS)
       (effects (font (size 1 1) (thickness 0.15)))
     )
@@
   (module myParts:FTMH-103-03-L-DH (layer F.Cu)
     (at 251.3 5.763)
-    (fp_text reference P47 (at 1.6 4.55 180) (layer F.SilkS)
+    (fp_text reference P47 (at -2.51 0.007 180) (layer F.SilkS)
       (effects (font (size 1 1) (thickness 0.15)))
     )
@@
   (module myParts:FTMH-103-03-L-DH (layer F.Cu)
     (at 192.7 5.763)
-    (fp_text reference P40 (at 1.6 4.55 180) (layer F.SilkS)
+    (fp_text reference P40 (at -0.11 4.597 180) (layer F.SilkS)
       (effects (font (size 1 1) (thickness 0.15)))
     )
@@
   (module myParts:FTMH-103-03-L-DH (layer F.Cu)
     (at 219.3 5.763)
-    (fp_text reference P39 (at 1.6 4.55 180) (layer F.SilkS)
+    (fp_text reference P39 (at -2.23 0.067 180) (layer F.SilkS)
       (effects (font (size 1 1) (thickness 0.15)))
     )
@@
   (module myParts:FTMH-103-03-L-DH (layer F.Cu)
     (at 187.3 5.763)
-    (fp_text reference P32 (at 1.6 4.55 180) (layer F.SilkS)
+    (fp_text reference P32 (at -2.46 0.047 180) (layer F.SilkS)
       (effects (font (size 1 1) (thickness 0.15)))
     )
@@
   (module myParts:FTMH-103-03-L-DH (layer F.Cu)
     (at 160.7 5.763)
-    (fp_text reference P31 (at 1.6 4.55 180) (layer F.SilkS)
+    (fp_text reference P31 (at -0.01 4.737 180) (layer F.SilkS)
       (effects (font (size 1 1) (thickness 0.15)))
     )
@@
   (module myParts:FTMH-103-03-L-DH (layer F.Cu)
     (at 155.3 5.763)
-    (fp_text reference P19 (at 1.6 4.55 180) (layer F.SilkS)
+    (fp_text reference P19 (at -2.4 -0.083 180) (layer F.SilkS)
       (effects (font (size 1 1) (thickness 0.15)))
     )
@@
   (module myParts:FTMH-103-03-L-DH (layer F.Cu)
     (at 128.7 5.763)
-    (fp_text reference P17 (at 1.6 4.55 180) (layer F.SilkS)
+    (fp_text reference P17 (at 0.09 4.657 180) (layer F.SilkS)
       (effects (font (size 1 1) (thickness 0.15)))
     )
@@
   (module myParts:FTMH-103-03-L-DH (layer F.Cu)
     (at 123.3 5.763)
-    (fp_text reference P15 (at 1.6 4.55 180) (layer F.SilkS)
+    (fp_text reference P15 (at -1.99 -0.163 180) (layer F.SilkS)
       (effects (font (size 1 1) (thickness 0.15)))
     )
@@
   (module myParts:FTMH-103-03-L-DH (layer F.Cu)
     (at 96.7 5.763)
-    (fp_text reference P13 (at 1.6 4.55 180) (layer F.SilkS)
+    (fp_text reference P13 (at 0.07 4.967 180) (layer F.SilkS)
       (effects (font (size 1 1) (thickness 0.15)))
     )
@@
   (module myParts:FTMH-103-03-L-DH (layer F.Cu)
     (at 91.3 5.763)
-    (fp_text reference P11 (at 1.6 4.55 180) (layer F.SilkS)
+    (fp_text reference P11 (at -2.04 0.047 180) (layer F.SilkS)
       (effects (font (size 1 1) (thickness 0.15)))
     )
@@
   (module myParts:FTMH-103-03-L-DH (layer F.Cu)
     (at 64.7 5.763)
-    (fp_text reference P9 (at 1.6 4.55 180) (layer F.SilkS)
+    (fp_text reference P9 (at -1.47 0.187 180) (layer F.SilkS)
       (effects (font (size 1 1) (thickness 0.15)))
     )
@@
   (module myParts:FTMH-103-03-L-DH (layer F.Cu)
     (at 59.3 5.763)
-    (fp_text reference P7 (at 1.6 4.55 180) (layer F.SilkS)
+    (fp_text reference P7 (at -1.73 0.297 180) (layer F.SilkS)
       (effects (font (size 1 1) (thickness 0.15)))
     )
@@
   (module myParts:FTMH-103-03-L-DH (layer F.Cu)
     (at 32.7 5.763)
-    (fp_text reference P5 (at 1.6 4.55 180) (layer F.SilkS)
+    (fp_text reference P5 (at -1.56 -0.013 180) (layer F.SilkS)
       (effects (font (size 1 1) (thickness 0.15)))
     )
@@
   (module myParts:FTMH-103-03-L-DH (layer F.Cu)
     (at 27.3 5.763)
-    (fp_text reference P3 (at 1.6 4.55 180) (layer F.SilkS)
+    (fp_text reference P3 (at -1.57 0.107 180) (layer F.SilkS)
       (effects (font (size 1 1) (thickness 0.15)))
     )
@@
   (module myParts:FTMH-103-03-L-DH (layer F.Cu)
     (at 0.7 5.763)
-    (fp_text reference P1 (at 1.6 4.55 180) (layer F.SilkS)
+    (fp_text reference P1 (at -1.5 -0.013 180) (layer F.SilkS)
       (effects (font (size 1 1) (thickness 0.15)))
     )
@@
     (descr "Through hole angled pin header, 2x07, 2.54mm pitch, 6mm pin length, double rows")
     (tags "Through hole angled pin header THT 2x07 2.54mm double row")
-    (fp_text reference P23 (at 5.585 -2.27 270) (layer F.SilkS)
+    (fp_text reference P23 (at -2.2 0.16 360) (layer F.SilkS)
       (effects (font (size 1 1) (thickness 0.15)))
     )
@@
       (xy 8.293997 0.976563) (xy 8.491005 0.779554)) (layer F.SilkS) (width 0.001))
   )
+  (gr_text v0.11 (at 405.79 5.69) (layer F.SilkS)
+    (effects (font (size 1.5 1.5) (thickness 0.3)))
+  )
   (gr_line (start 419.1 0) (end 419.1 25.4) (layer Edge.Cuts) (width 0.15))
