File: KiCAD/distributor8/distributor8.kicad_pcb (KiCad board)
At the start: 4 copper layers, 431.8 x 25.4 mm, 29 parts, among them P1 CONN_02X03, P11 CONN_02X03, P13 CONN_02X03, P15 CONN_02X03, P17 CONN_02X03, P19 CONN_02X03, P23 CONN_02X07, P24 CONN_02X07, P29 CONN_02X07, P3 CONN_02X03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

Commit message: adding new spring pin boards
Parts:
- P23, P24, P29, P30, P37, P38, P45, P46: footprint myParts:SSW-107-02-T-D-RA -> myParts:SSW-106-02-T-D-RA-IN14
Changed lines of the file:
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@@
   )
   (setup
-    (last_trace_width 0.56)
+    (last_trace_width 0.4)
     (user_trace_width 0.4)
     (user_trace_width 0.56)
@@
     (uvia_drill 0.1)
   )
-  (module myParts:SSW-107-02-T-D-RA (layer B.Cu)
+  (module myParts:SSW-106-02-T-D-RA-IN14 (layer B.Cu)
     (at 279.4 12.7 90)
     (descr "Through hole angled socket strip, 2x07, 2.54mm pitch, 8.51mm socket length, double rows")
@@
     (pad 14 thru_hole oval (at -2.54 -15.24 90) (size 1.7 1.7) (drill 1) (layers *.Cu *.Mask)
       (net 69 "Net-(P23-Pad14)"))
-    (model ${KIPRJMOD}/sharedLibs/myparts.3dshapes/SSW-107-02-T-D-RA.wrl
-      (at (xyz -0.1594488188976378 -0.3 0.09744094488188977))
-      (scale (xyz 0.01 0.01 0.01))
-      (rotate (xyz -90 0 90))
+    (model ${KIPRJMOD}/sharedLibs/myparts.3dshapes/SSW-106-02-T-D-RA.stp
+      (at (xyz -0.1594488188976378 -0.25 0.09744094488188977))
+      (scale (xyz 1 1 1))
+      (rotate (xyz 180 0 90))
     )
   )
-  (module myParts:SSW-107-02-T-D-RA (layer B.Cu)
+  (module myParts:SSW-106-02-T-D-RA-IN14 (layer B.Cu)
     (at 350.52 12.7 90)
     (descr "Through hole angled socket strip, 2x07, 2.54mm pitch, 8.51mm socket length, double rows")
@@
     (pad 14 thru_hole oval (at -2.54 -15.24 90) (size 1.7 1.7) (drill 1) (layers *.Cu *.Mask)
       (net 71 "Net-(P24-Pad14)"))
-    (model ${KIPRJMOD}/sharedLibs/myparts.3dshapes/SSW-107-02-T-D-RA.wrl
-      (at (xyz -0.1594488188976378 -0.3 0.09744094488188977))
-      (scale (xyz 0.01 0.01 0.01))
-      (rotate (xyz -90 0 90))
+    (model ${KIPRJMOD}/sharedLibs/myparts.3dshapes/SSW-106-02-T-D-RA.stp
+      (at (xyz -0.1594488188976378 -0.25 0.09744094488188977))
+      (scale (xyz 1 1 1))
+      (rotate (xyz 180 0 90))
     )
   )
-  (module myParts:SSW-107-02-T-D-RA (layer B.Cu)
+  (module myParts:SSW-106-02-T-D-RA-IN14 (layer B.Cu)
     (at 368.3 12.7 90)
     (descr "Through hole angled socket strip, 2x07, 2.54mm pitch, 8.51mm socket length, double rows")
@@
     (pad 14 thru_hole oval (at -2.54 -15.24 90) (size 1.7 1.7) (drill 1) (layers *.Cu *.Mask)
       (net 73 "Net-(P29-Pad14)"))
-    (model ${KIPRJMOD}/sharedLibs/myparts.3dshapes/SSW-107-02-T-D-RA.wrl
-      (at (xyz -0.1594488188976378 -0.3 0.09744094488188977))
-      (scale (xyz 0.01 0.01 0.01))
-      (rotate (xyz -90 0 90))
+    (model ${KIPRJMOD}/sharedLibs/myparts.3dshapes/SSW-106-02-T-D-RA.stp
+      (at (xyz -0.1594488188976378 -0.25 0.09744094488188977))
+      (scale (xyz 1 1 1))
+      (rotate (xyz 180 0 90))
     )
   )
-  (module myParts:SSW-107-02-T-D-RA (layer B.Cu)
+  (module myParts:SSW-106-02-T-D-RA-IN14 (layer B.Cu)
     (at 297.18 12.7 90)
     (descr "Through hole angled socket strip, 2x07, 2.54mm pitch, 8.51mm socket length, double rows")
@@
     (pad 14 thru_hole oval (at -2.54 -15.24 90) (size 1.7 1.7) (drill 1) (layers *.Cu *.Mask)
       (net 75 "Net-(P30-Pad14)"))
-    (model ${KIPRJMOD}/sharedLibs/myparts.3dshapes/SSW-107-02-T-D-RA.wrl
-      (at (xyz -0.1594488188976378 -0.3 0.09744094488188977))
-      (scale (xyz 0.01 0.01 0.01))
-      (rotate (xyz -90 0 90))
+    (model ${KIPRJMOD}/sharedLibs/myparts.3dshapes/SSW-106-02-T-D-RA.stp
+      (at (xyz -0.1594488188976378 -0.25 0.09744094488188977))
+      (scale (xyz 1 1 1))
+      (rotate (xyz 180 0 90))
     )
   )
-  (module myParts:SSW-107-02-T-D-RA (layer B.Cu)
+  (module myParts:SSW-106-02-T-D-RA-IN14 (layer B.Cu)
     (at 314.96 12.7 90)
     (descr "Through hole angled socket strip, 2x07, 2.54mm pitch, 8.51mm socket length, double rows")
@@
     (pad 14 thru_hole oval (at -2.54 -15.24 90) (size 1.7 1.7) (drill 1) (layers *.Cu *.Mask)
       (net 77 "Net-(P37-Pad14)"))
-    (model ${KIPRJMOD}/sharedLibs/myparts.3dshapes/SSW-107-02-T-D-RA.wrl
-      (at (xyz -0.1594488188976378 -0.3 0.09744094488188977))
-      (scale (xyz 0.01 0.01 0.01))
-      (rotate (xyz -90 0 90))
+    (model ${KIPRJMOD}/sharedLibs/myparts.3dshapes/SSW-106-02-T-D-RA.stp
+      (at (xyz -0.1594488188976378 -0.25 0.09744094488188977))
+      (scale (xyz 1 1 1))
+      (rotate (xyz 180 0 90))
     )
   )
-  (module myParts:SSW-107-02-T-D-RA (layer B.Cu)
+  (module myParts:SSW-106-02-T-D-RA-IN14 (layer B.Cu)
     (at 386.08 12.7 90)
     (descr "Through hole angled socket strip, 2x07, 2.54mm pitch, 8.51mm socket length, double rows")
@@
     (pad 14 thru_hole oval (at -2.54 -15.24 90) (size 1.7 1.7) (drill 1) (layers *.Cu *.Mask)
       (net 79 "Net-(P38-Pad14)"))
-    (model ${KIPRJMOD}/sharedLibs/myparts.3dshapes/SSW-107-02-T-D-RA.wrl
-      (at (xyz -0.1594488188976378 -0.3 0.09744094488188977))
-      (scale (xyz 0.01 0.01 0.01))
-      (rotate (xyz -90 0 90))
+    (model ${KIPRJMOD}/sharedLibs/myparts.3dshapes/SSW-106-02-T-D-RA.stp
+      (at (xyz -0.1594488188976378 -0.25 0.09744094488188977))
+      (scale (xyz 1 1 1))
+      (rotate (xyz 180 0 90))
     )
   )
-  (module myParts:SSW-107-02-T-D-RA (layer B.Cu)
+  (module myParts:SSW-106-02-T-D-RA-IN14 (layer B.Cu)
     (at 332.74 12.7 90)
     (descr "Through hole angled socket strip, 2x07, 2.54mm pitch, 8.51mm socket length, double rows")
@@
     (pad 14 thru_hole oval (at -2.54 -15.24 90) (size 1.7 1.7) (drill 1) (layers *.Cu *.Mask)
       (net 81 "Net-(P45-Pad14)"))
-    (model ${KIPRJMOD}/sharedLibs/myparts.3dshapes/SSW-107-02-T-D-RA.wrl
-      (at (xyz -0.1594488188976378 -0.3 0.09744094488188977))
-      (scale (xyz 0.01 0.01 0.01))
-      (rotate (xyz -90 0 90))
+    (model ${KIPRJMOD}/sharedLibs/myparts.3dshapes/SSW-106-02-T-D-RA.stp
+      (at (xyz -0.1594488188976378 -0.25 0.09744094488188977))
+      (scale (xyz 1 1 1))
+      (rotate (xyz 180 0 90))
     )
   )
-  (module myParts:SSW-107-02-T-D-RA (layer B.Cu)
+  (module myParts:SSW-106-02-T-D-RA-IN14 (layer B.Cu)
     (at 403.86 12.7 90)
     (descr "Through hole angled socket strip, 2x07, 2.54mm pitch, 8.51mm socket length, double rows")
@@
     (pad 14 thru_hole oval (at -2.54 -15.24 90) (size 1.7 1.7) (drill 1) (layers *.Cu *.Mask)
       (net 83 "Net-(P46-Pad14)"))
-    (model ${KIPRJMOD}/sharedLibs/myparts.3dshapes/SSW-107-02-T-D-RA.wrl
-      (at (xyz -0.1594488188976378 -0.3 0.09744094488188977))
-      (scale (xyz 0.01 0.01 0.01))
-      (rotate (xyz -90 0 90))
+    (model ${KIPRJMOD}/sharedLibs/myparts.3dshapes/SSW-106-02-T-D-RA.stp
+      (at (xyz -0.1594488188976378 -0.25 0.09744094488188977))
+      (scale (xyz 1 1 1))
+      (rotate (xyz 180 0 90))
     )
   )
