File: KiCAD/distributor8/distributor8.sch (KiCad schematic (older format))
At the start: 52 parts, among them P1 CONN_02X03, P10 CONN_02X03, P11 CONN_02X03, P12 CONN_02X03, P13 CONN_02X03, P14 CONN_02X03, P15 CONN_02X03, P16 CONN_02X03, P17 CONN_02X03, P18 CONN_02X03, P19 CONN_02X03, P2 CONN_02X03, P20 CONN_02X03, P21 CONN_02X07, P22 CONN_02X07, P23 CONN_02X07, P24 CONN_02X07, P25 CONN_02X03, P26 CONN_02X03, P27 CONN_02X07, P28 CONN_02X07, P29 CONN_02X07, P3 CONN_02X03, P30 CONN_02X07, P31 CONN_02X03, P32 CONN_02X03, P33 CONN_02X03, P34 CONN_02X03, P35 CONN_02X07, P36 CONN_02X07, P37 CONN_02X07, P38 CONN_02X07, P39 CONN_02X03, P4 CONN_02X03, P40 CONN_02X03, P41 CONN_02X03, P42 CONN_02X03, P43 CONN_02X07, P44 CONN_02X07, P45 CONN_02X07, P46 CONN_02X07, P47 CONN_02X03, P48 CONN_02X03, P5 CONN_02X03, P6 CONN_02X03, P7 CONN_02X03, P8 CONN_02X03, P9 CONN_02X03

Commit message: distributor 8B layout done
Other:
- moved on the sheet: P1, P12, P16, P21, P22, P23, P24, P27, P28, P29, P30, P36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

Commit message: 8ch distributor board done
Parts:
- P1, P10, P11, P12, P13, P14, P15, P16, P17, P18, P19, P2, P20, P25, P26, P3, P31, P32, P33, P34, P39, P4, P40, P41, P42, P47, P48, P5, P6, P7, P8, P9: footprint myParts:FTMH-103-03-L-DH -> myParts:TMS-103-02-L-D-SE
Changed lines of the file:
@@
 F 0 "P5" H 3400 1300 50  0000 C CNN
 F 1 "CONN_02X03" H 3400 900 50  0000 C CNN
-F 2 "myParts:FTMH-103-03-L-DH" H 3400 -100 50  0001 C CNN
+F 2 "myParts:TMS-103-02-L-D-SE" H 3400 -100 50  0001 C CNN
 F 3 "" H 3400 -100 50  0000 C CNN
 	1    3400 1100
@@
 F 0 "P7" H 4650 1300 50  0000 C CNN
 F 1 "CONN_02X03" H 4650 900 50  0000 C CNN
-F 2 "myParts:FTMH-103-03-L-DH" H 4650 -100 50  0001 C CNN
+F 2 "myParts:TMS-103-02-L-D-SE" H 4650 -100 50  0001 C CNN
 F 3 "" H 4650 -100 50  0000 C CNN
 	1    4650 1100
@@
 F 0 "P6" H 3400 2550 50  0000 C CNN
 F 1 "CONN_02X03" H 3400 2150 50  0000 C CNN
-F 2 "myParts:FTMH-103-03-L-DH" H 3400 1150 50  0001 C CNN
+F 2 "myParts:TMS-103-02-L-D-SE" H 3400 1150 50  0001 C CNN
 F 3 "" H 3400 1150 50  0000 C CNN
 	1    3400 2350
@@
 F 0 "P8" H 4650 2550 50  0000 C CNN
 F 1 "CONN_02X03" H 4650 2150 50  0000 C CNN
-F 2 "myParts:FTMH-103-03-L-DH" H 4650 1150 50  0001 C CNN
+F 2 "myParts:TMS-103-02-L-D-SE" H 4650 1150 50  0001 C CNN
 F 3 "" H 4650 1150 50  0000 C CNN
 	1    4650 2350
@@
 F 0 "P1" H 800 1400 50  0000 C CNN
 F 1 "CONN_02X03" H 800 1000 50  0000 C CNN
-F 2 "myParts:FTMH-103-03-L-DH" H 800 0   50  0001 C CNN
+F 2 "myParts:TMS-103-02-L-D-SE" H 800 0   50  0001 C CNN
 F 3 "" H 800 0   50  0000 C CNN
 	1    800  1200
@@
 F 0 "P3" H 2050 1300 50  0000 C CNN
 F 1 "CONN_02X03" H 2050 900 50  0000 C CNN
-F 2 "myParts:FTMH-103-03-L-DH" H 2050 -100 50  0001 C CNN
+F 2 "myParts:TMS-103-02-L-D-SE" H 2050 -100 50  0001 C CNN
 F 3 "" H 2050 -100 50  0000 C CNN
 	1    2050 1100
@@
 F 0 "P2" H 800 2550 50  0000 C CNN
 F 1 "CONN_02X03" H 800 2150 50  0000 C CNN
-F 2 "myParts:FTMH-103-03-L-DH" H 800 1150 50  0001 C CNN
+F 2 "myParts:TMS-103-02-L-D-SE" H 800 1150 50  0001 C CNN
 F 3 "" H 800 1150 50  0000 C CNN
 	1    800  2350
@@
 F 0 "P4" H 2050 2550 50  0000 C CNN
 F 1 "CONN_02X03" H 2050 2150 50  0000 C CNN
-F 2 "myParts:FTMH-103-03-L-DH" H 2050 1150 50  0001 C CNN
+F 2 "myParts:TMS-103-02-L-D-SE" H 2050 1150 50  0001 C CNN
 F 3 "" H 2050 1150 50  0000 C CNN
 	1    2050 2350
@@
 F 0 "P13" H 8800 1300 50  0000 C CNN
 F 1 "CONN_02X03" H 8800 900 50  0000 C CNN
-F 2 "myParts:FTMH-103-03-L-DH" H 8800 -100 50  0001 C CNN
+F 2 "myParts:TMS-103-02-L-D-SE" H 8800 -100 50  0001 C CNN
 F 3 "" H 8800 -100 50  0000 C CNN
 	1    8800 1100
@@
 F 0 "P15" H 10050 1300 50  0000 C CNN
 F 1 "CONN_02X03" H 10050 900 50  0000 C CNN
-F 2 "myParts:FTMH-103-03-L-DH" H 10050 -100 50  0001 C CNN
+F 2 "myParts:TMS-103-02-L-D-SE" H 10050 -100 50  0001 C CNN
 F 3 "" H 10050 -100 50  0000 C CNN
 	1    10050 1100
@@
 F 0 "P14" H 8800 2550 50  0000 C CNN
 F 1 "CONN_02X03" H 8800 2150 50  0000 C CNN
-F 2 "myParts:FTMH-103-03-L-DH" H 8800 1150 50  0001 C CNN
+F 2 "myParts:TMS-103-02-L-D-SE" H 8800 1150 50  0001 C CNN
 F 3 "" H 8800 1150 50  0000 C CNN
 	1    8800 2350
@@
 F 0 "P16" H 10000 2550 50  0000 C CNN
 F 1 "CONN_02X03" H 10000 2150 50  0000 C CNN
-F 2 "myParts:FTMH-103-03-L-DH" H 10000 1150 50  0001 C CNN
+F 2 "myParts:TMS-103-02-L-D-SE" H 10000 1150 50  0001 C CNN
 F 3 "" H 10000 1150 50  0000 C CNN
 	1    10000 2350
@@
 F 0 "P9" H 6000 1300 50  0000 C CNN
 F 1 "CONN_02X03" H 6000 900 50  0000 C CNN
-F 2 "myParts:FTMH-103-03-L-DH" H 6000 -100 50  0001 C CNN
+F 2 "myParts:TMS-103-02-L-D-SE" H 6000 -100 50  0001 C CNN
 F 3 "" H 6000 -100 50  0000 C CNN
 	1    6000 1100
@@
 F 0 "P11" H 7250 1300 50  0000 C CNN
 F 1 "CONN_02X03" H 7250 900 50  0000 C CNN
-F 2 "myParts:FTMH-103-03-L-DH" H 7250 -100 50  0001 C CNN
+F 2 "myParts:TMS-103-02-L-D-SE" H 7250 -100 50  0001 C CNN
 F 3 "" H 7250 -100 50  0000 C CNN
 	1    7250 1100
@@
 F 0 "P10" H 6000 2550 50  0000 C CNN
 F 1 "CONN_02X03" H 6000 2150 50  0000 C CNN
-F 2 "myParts:FTMH-103-03-L-DH" H 6000 1150 50  0001 C CNN
+F 2 "myParts:TMS-103-02-L-D-SE" H 6000 1150 50  0001 C CNN
 F 3 "" H 6000 1150 50  0000 C CNN
 	1    6000 2350
@@
 F 0 "P12" H 7200 2550 50  0000 C CNN
 F 1 "CONN_02X03" H 7200 2150 50  0000 C CNN
-F 2 "myParts:FTMH-103-03-L-DH" H 7200 1150 50  0001 C CNN
+F 2 "myParts:TMS-103-02-L-D-SE" H 7200 1150 50  0001 C CNN
 F 3 "" H 7200 1150 50  0000 C CNN
 	1    7200 2350
@@
 F 0 "P17" H 800 4350 50  0000 C CNN
 F 1 "CONN_02X03" H 800 3950 50  0000 C CNN
-F 2 "myParts:FTMH-103-03-L-DH" H 800 2950 50  0001 C CNN
+F 2 "myParts:TMS-103-02-L-D-SE" H 800 2950 50  0001 C CNN
 F 3 "" H 800 2950 50  0000 C CNN
 	1    800  4150
@@
 F 0 "P19" H 2050 4350 50  0000 C CNN
 F 1 "CONN_02X03" H 2050 3950 50  0000 C CNN
-F 2 "myParts:FTMH-103-03-L-DH" H 2050 2950 50  0001 C CNN
+F 2 "myParts:TMS-103-02-L-D-SE" H 2050 2950 50  0001 C CNN
 F 3 "" H 2050 2950 50  0000 C CNN
 	1    2050 4150
@@
 F 0 "P18" H 800 5600 50  0000 C CNN
 F 1 "CONN_02X03" H 800 5200 50  0000 C CNN
-F 2 "myParts:FTMH-103-03-L-DH" H 800 4200 50  0001 C CNN
+F 2 "myParts:TMS-103-02-L-D-SE" H 800 4200 50  0001 C CNN
 F 3 "" H 800 4200 50  0000 C CNN
 	1    800  5400
@@
 F 0 "P20" H 2050 5600 50  0000 C CNN
 F 1 "CONN_02X03" H 2050 5200 50  0000 C CNN
-F 2 "myParts:FTMH-103-03-L-DH" H 2050 4200 50  0001 C CNN
+F 2 "myParts:TMS-103-02-L-D-SE" H 2050 4200 50  0001 C CNN
 F 3 "" H 2050 4200 50  0000 C CNN
 	1    2050 5400
@@
 F 0 "P39" H 6000 4250 50  0000 C CNN
 F 1 "CONN_02X03" H 6000 3850 50  0000 C CNN
-F 2 "myParts:FTMH-103-03-L-DH" H 6000 2850 50  0001 C CNN
+F 2 "myParts:TMS-103-02-L-D-SE" H 6000 2850 50  0001 C CNN
 F 3 "" H 6000 2850 50  0000 C CNN
 	1    6000 4050
@@
 F 0 "P40" H 7250 4250 50  0000 C CNN
 F 1 "CONN_02X03" H 7250 3850 50  0000 C CNN
-F 2 "myParts:FTMH-103-03-L-DH" H 7250 2850 50  0001 C CNN
+F 2 "myParts:TMS-103-02-L-D-SE" H 7250 2850 50  0001 C CNN
 F 3 "" H 7250 2850 50  0000 C CNN
 	1    7250 4050
@@
 F 0 "P33" H 6000 5500 50  0000 C CNN
 F 1 "CONN_02X03" H 6000 5100 50  0000 C CNN
-F 2 "myParts:FTMH-103-03-L-DH" H 6000 4100 50  0001 C CNN
+F 2 "myParts:TMS-103-02-L-D-SE" H 6000 4100 50  0001 C CNN
 F 3 "" H 6000 4100 50  0000 C CNN
 	1    6000 5300
@@
 F 0 "P34" H 7250 5500 50  0000 C CNN
 F 1 "CONN_02X03" H 7250 5100 50  0000 C CNN
-F 2 "myParts:FTMH-103-03-L-DH" H 7250 4100 50  0001 C CNN
+F 2 "myParts:TMS-103-02-L-D-SE" H 7250 4100 50  0001 C CNN
 F 3 "" H 7250 4100 50  0000 C CNN
 	1    7250 5300
@@
 F 0 "P47" H 3400 4400 50  0000 C CNN
 F 1 "CONN_02X03" H 3400 4000 50  0000 C CNN
-F 2 "myParts:FTMH-103-03-L-DH" H 3400 3000 50  0001 C CNN
+F 2 "myParts:TMS-103-02-L-D-SE" H 3400 3000 50  0001 C CNN
 F 3 "" H 3400 3000 50  0000 C CNN
 	1    3400 4200
@@
 F 0 "P48" H 4650 4400 50  0000 C CNN
 F 1 "CONN_02X03" H 4650 4000 50  0000 C CNN
-F 2 "myParts:FTMH-103-03-L-DH" H 4650 3000 50  0001 C CNN
+F 2 "myParts:TMS-103-02-L-D-SE" H 4650 3000 50  0001 C CNN
 F 3 "" H 4650 3000 50  0000 C CNN
 	1    4650 4200
@@
 F 0 "P41" H 3400 5650 50  0000 C CNN
 F 1 "CONN_02X03" H 3400 5250 50  0000 C CNN
-F 2 "myParts:FTMH-103-03-L-DH" H 3400 4250 50  0001 C CNN
+F 2 "myParts:TMS-103-02-L-D-SE" H 3400 4250 50  0001 C CNN
 F 3 "" H 3400 4250 50  0000 C CNN
 	1    3400 5450
@@
 F 0 "P42" H 4600 5650 50  0000 C CNN
 F 1 "CONN_02X03" H 4600 5250 50  0000 C CNN
-F 2 "myParts:FTMH-103-03-L-DH" H 4600 4250 50  0001 C CNN
+F 2 "myParts:TMS-103-02-L-D-SE" H 4600 4250 50  0001 C CNN
 F 3 "" H 4600 4250 50  0000 C CNN
 	1    4600 5450
@@
 F 0 "P31" H 8800 4250 50  0000 C CNN
 F 1 "CONN_02X03" H 8800 3850 50  0000 C CNN
-F 2 "myParts:FTMH-103-03-L-DH" H 8800 2850 50  0001 C CNN
+F 2 "myParts:TMS-103-02-L-D-SE" H 8800 2850 50  0001 C CNN
 F 3 "" H 8800 2850 50  0000 C CNN
 	1    8800 4050
@@
 F 0 "P32" H 10050 4250 50  0000 C CNN
 F 1 "CONN_02X03" H 10050 3850 50  0000 C CNN
-F 2 "myParts:FTMH-103-03-L-DH" H 10050 2850 50  0001 C CNN
+F 2 "myParts:TMS-103-02-L-D-SE" H 10050 2850 50  0001 C CNN
 F 3 "" H 10050 2850 50  0000 C CNN
 	1    10050 4050
@@
 F 0 "P25" H 8800 5500 50  0000 C CNN
 F 1 "CONN_02X03" H 8800 5100 50  0000 C CNN
-F 2 "myParts:FTMH-103-03-L-DH" H 8800 4100 50  0001 C CNN
+F 2 "myParts:TMS-103-02-L-D-SE" H 8800 4100 50  0001 C CNN
 F 3 "" H 8800 4100 50  0000 C CNN
 	1    8800 5300
@@
 F 0 "P26" H 10050 5500 50  0000 C CNN
 F 1 "CONN_02X03" H 10050 5100 50  0000 C CNN
-F 2 "myParts:FTMH-103-03-L-DH" H 10050 4100 50  0001 C CNN
+F 2 "myParts:TMS-103-02-L-D-SE" H 10050 4100 50  0001 C CNN
 F 3 "" H 10050 4100 50  0000 C CNN
 	1    10050 5300

Commit message: switch to step for 3d
Parts:
- P1, P10, P11, P12, P13, P14, P15, P16, P17, P18, P19, P2, P20, P25, P26, P3, P31, P32, P33, P34, P39, P4, P40, P41, P42, P47, P48, P5, P6, P7, P8, P9: footprint myParts:TMS-103-02-L-D-SE -> myParts:TMS-103-01-L-D-SE
Changed lines of the file:
@@
 F 0 "P5" H 3400 1300 50  0000 C CNN
 F 1 "CONN_02X03" H 3400 900 50  0000 C CNN
-F 2 "myParts:TMS-103-02-L-D-SE" H 3400 -100 50  0001 C CNN
+F 2 "myParts:TMS-103-01-L-D-SE" H 3400 -100 50  0001 C CNN
 F 3 "" H 3400 -100 50  0000 C CNN
 	1    3400 1100
@@
 F 0 "P7" H 4650 1300 50  0000 C CNN
 F 1 "CONN_02X03" H 4650 900 50  0000 C CNN
-F 2 "myParts:TMS-103-02-L-D-SE" H 4650 -100 50  0001 C CNN
+F 2 "myParts:TMS-103-01-L-D-SE" H 4650 -100 50  0001 C CNN
 F 3 "" H 4650 -100 50  0000 C CNN
 	1    4650 1100
@@
 F 0 "P6" H 3400 2550 50  0000 C CNN
 F 1 "CONN_02X03" H 3400 2150 50  0000 C CNN
-F 2 "myParts:TMS-103-02-L-D-SE" H 3400 1150 50  0001 C CNN
+F 2 "myParts:TMS-103-01-L-D-SE" H 3400 1150 50  0001 C CNN
 F 3 "" H 3400 1150 50  0000 C CNN
 	1    3400 2350
@@
 F 0 "P8" H 4650 2550 50  0000 C CNN
 F 1 "CONN_02X03" H 4650 2150 50  0000 C CNN
-F 2 "myParts:TMS-103-02-L-D-SE" H 4650 1150 50  0001 C CNN
+F 2 "myParts:TMS-103-01-L-D-SE" H 4650 1150 50  0001 C CNN
 F 3 "" H 4650 1150 50  0000 C CNN
 	1    4650 2350
@@
 F 0 "P1" H 800 1400 50  0000 C CNN
 F 1 "CONN_02X03" H 800 1000 50  0000 C CNN
-F 2 "myParts:TMS-103-02-L-D-SE" H 800 0   50  0001 C CNN
+F 2 "myParts:TMS-103-01-L-D-SE" H 800 0   50  0001 C CNN
 F 3 "" H 800 0   50  0000 C CNN
 	1    800  1200
@@
 F 0 "P3" H 2050 1300 50  0000 C CNN
 F 1 "CONN_02X03" H 2050 900 50  0000 C CNN
-F 2 "myParts:TMS-103-02-L-D-SE" H 2050 -100 50  0001 C CNN
+F 2 "myParts:TMS-103-01-L-D-SE" H 2050 -100 50  0001 C CNN
 F 3 "" H 2050 -100 50  0000 C CNN
 	1    2050 1100
@@
 F 0 "P2" H 800 2550 50  0000 C CNN
 F 1 "CONN_02X03" H 800 2150 50  0000 C CNN
-F 2 "myParts:TMS-103-02-L-D-SE" H 800 1150 50  0001 C CNN
+F 2 "myParts:TMS-103-01-L-D-SE" H 800 1150 50  0001 C CNN
 F 3 "" H 800 1150 50  0000 C CNN
 	1    800  2350
@@
 F 0 "P4" H 2050 2550 50  0000 C CNN
 F 1 "CONN_02X03" H 2050 2150 50  0000 C CNN
-F 2 "myParts:TMS-103-02-L-D-SE" H 2050 1150 50  0001 C CNN
+F 2 "myParts:TMS-103-01-L-D-SE" H 2050 1150 50  0001 C CNN
 F 3 "" H 2050 1150 50  0000 C CNN
 	1    2050 2350
@@
 F 0 "P13" H 8800 1300 50  0000 C CNN
 F 1 "CONN_02X03" H 8800 900 50  0000 C CNN
-F 2 "myParts:TMS-103-02-L-D-SE" H 8800 -100 50  0001 C CNN
+F 2 "myParts:TMS-103-01-L-D-SE" H 8800 -100 50  0001 C CNN
 F 3 "" H 8800 -100 50  0000 C CNN
 	1    8800 1100
@@
 F 0 "P15" H 10050 1300 50  0000 C CNN
 F 1 "CONN_02X03" H 10050 900 50  0000 C CNN
-F 2 "myParts:TMS-103-02-L-D-SE" H 10050 -100 50  0001 C CNN
+F 2 "myParts:TMS-103-01-L-D-SE" H 10050 -100 50  0001 C CNN
 F 3 "" H 10050 -100 50  0000 C CNN
 	1    10050 1100
@@
 F 0 "P14" H 8800 2550 50  0000 C CNN
 F 1 "CONN_02X03" H 8800 2150 50  0000 C CNN
-F 2 "myParts:TMS-103-02-L-D-SE" H 8800 1150 50  0001 C CNN
+F 2 "myParts:TMS-103-01-L-D-SE" H 8800 1150 50  0001 C CNN
 F 3 "" H 8800 1150 50  0000 C CNN
 	1    8800 2350
@@
 F 0 "P16" H 10000 2550 50  0000 C CNN
 F 1 "CONN_02X03" H 10000 2150 50  0000 C CNN
-F 2 "myParts:TMS-103-02-L-D-SE" H 10000 1150 50  0001 C CNN
+F 2 "myParts:TMS-103-01-L-D-SE" H 10000 1150 50  0001 C CNN
 F 3 "" H 10000 1150 50  0000 C CNN
 	1    10000 2350
@@
 F 0 "P9" H 6000 1300 50  0000 C CNN
 F 1 "CONN_02X03" H 6000 900 50  0000 C CNN
-F 2 "myParts:TMS-103-02-L-D-SE" H 6000 -100 50  0001 C CNN
+F 2 "myParts:TMS-103-01-L-D-SE" H 6000 -100 50  0001 C CNN
 F 3 "" H 6000 -100 50  0000 C CNN
 	1    6000 1100
@@
 F 0 "P11" H 7250 1300 50  0000 C CNN
 F 1 "CONN_02X03" H 7250 900 50  0000 C CNN
-F 2 "myParts:TMS-103-02-L-D-SE" H 7250 -100 50  0001 C CNN
+F 2 "myParts:TMS-103-01-L-D-SE" H 7250 -100 50  0001 C CNN
 F 3 "" H 7250 -100 50  0000 C CNN
 	1    7250 1100
@@
 F 0 "P10" H 6000 2550 50  0000 C CNN
 F 1 "CONN_02X03" H 6000 2150 50  0000 C CNN
-F 2 "myParts:TMS-103-02-L-D-SE" H 6000 1150 50  0001 C CNN
+F 2 "myParts:TMS-103-01-L-D-SE" H 6000 1150 50  0001 C CNN
 F 3 "" H 6000 1150 50  0000 C CNN
 	1    6000 2350
@@
 F 0 "P12" H 7200 2550 50  0000 C CNN
 F 1 "CONN_02X03" H 7200 2150 50  0000 C CNN
-F 2 "myParts:TMS-103-02-L-D-SE" H 7200 1150 50  0001 C CNN
+F 2 "myParts:TMS-103-01-L-D-SE" H 7200 1150 50  0001 C CNN
 F 3 "" H 7200 1150 50  0000 C CNN
 	1    7200 2350
@@
 F 0 "P17" H 800 4350 50  0000 C CNN
 F 1 "CONN_02X03" H 800 3950 50  0000 C CNN
-F 2 "myParts:TMS-103-02-L-D-SE" H 800 2950 50  0001 C CNN
+F 2 "myParts:TMS-103-01-L-D-SE" H 800 2950 50  0001 C CNN
 F 3 "" H 800 2950 50  0000 C CNN
 	1    800  4150
@@
 F 0 "P19" H 2050 4350 50  0000 C CNN
 F 1 "CONN_02X03" H 2050 3950 50  0000 C CNN
-F 2 "myParts:TMS-103-02-L-D-SE" H 2050 2950 50  0001 C CNN
+F 2 "myParts:TMS-103-01-L-D-SE" H 2050 2950 50  0001 C CNN
 F 3 "" H 2050 2950 50  0000 C CNN
 	1    2050 4150
@@
 F 0 "P18" H 800 5600 50  0000 C CNN
 F 1 "CONN_02X03" H 800 5200 50  0000 C CNN
-F 2 "myParts:TMS-103-02-L-D-SE" H 800 4200 50  0001 C CNN
+F 2 "myParts:TMS-103-01-L-D-SE" H 800 4200 50  0001 C CNN
 F 3 "" H 800 4200 50  0000 C CNN
 	1    800  5400
@@
 F 0 "P20" H 2050 5600 50  0000 C CNN
 F 1 "CONN_02X03" H 2050 5200 50  0000 C CNN
-F 2 "myParts:TMS-103-02-L-D-SE" H 2050 4200 50  0001 C CNN
+F 2 "myParts:TMS-103-01-L-D-SE" H 2050 4200 50  0001 C CNN
 F 3 "" H 2050 4200 50  0000 C CNN
 	1    2050 5400
@@
 F 0 "P39" H 6000 4250 50  0000 C CNN
 F 1 "CONN_02X03" H 6000 3850 50  0000 C CNN
-F 2 "myParts:TMS-103-02-L-D-SE" H 6000 2850 50  0001 C CNN
+F 2 "myParts:TMS-103-01-L-D-SE" H 6000 2850 50  0001 C CNN
 F 3 "" H 6000 2850 50  0000 C CNN
 	1    6000 4050
@@
 F 0 "P40" H 7250 4250 50  0000 C CNN
 F 1 "CONN_02X03" H 7250 3850 50  0000 C CNN
-F 2 "myParts:TMS-103-02-L-D-SE" H 7250 2850 50  0001 C CNN
+F 2 "myParts:TMS-103-01-L-D-SE" H 7250 2850 50  0001 C CNN
 F 3 "" H 7250 2850 50  0000 C CNN
 	1    7250 4050
@@
 F 0 "P33" H 6000 5500 50  0000 C CNN
 F 1 "CONN_02X03" H 6000 5100 50  0000 C CNN
-F 2 "myParts:TMS-103-02-L-D-SE" H 6000 4100 50  0001 C CNN
+F 2 "myParts:TMS-103-01-L-D-SE" H 6000 4100 50  0001 C CNN
 F 3 "" H 6000 4100 50  0000 C CNN
 	1    6000 5300
@@
 F 0 "P34" H 7250 5500 50  0000 C CNN
 F 1 "CONN_02X03" H 7250 5100 50  0000 C CNN
-F 2 "myParts:TMS-103-02-L-D-SE" H 7250 4100 50  0001 C CNN
+F 2 "myParts:TMS-103-01-L-D-SE" H 7250 4100 50  0001 C CNN
 F 3 "" H 7250 4100 50  0000 C CNN
 	1    7250 5300
@@
 F 0 "P47" H 3400 4400 50  0000 C CNN
 F 1 "CONN_02X03" H 3400 4000 50  0000 C CNN
-F 2 "myParts:TMS-103-02-L-D-SE" H 3400 3000 50  0001 C CNN
+F 2 "myParts:TMS-103-01-L-D-SE" H 3400 3000 50  0001 C CNN
 F 3 "" H 3400 3000 50  0000 C CNN
 	1    3400 4200
@@
 F 0 "P48" H 4650 4400 50  0000 C CNN
 F 1 "CONN_02X03" H 4650 4000 50  0000 C CNN
-F 2 "myParts:TMS-103-02-L-D-SE" H 4650 3000 50  0001 C CNN
+F 2 "myParts:TMS-103-01-L-D-SE" H 4650 3000 50  0001 C CNN
 F 3 "" H 4650 3000 50  0000 C CNN
 	1    4650 4200
@@
 F 0 "P41" H 3400 5650 50  0000 C CNN
 F 1 "CONN_02X03" H 3400 5250 50  0000 C CNN
-F 2 "myParts:TMS-103-02-L-D-SE" H 3400 4250 50  0001 C CNN
+F 2 "myParts:TMS-103-01-L-D-SE" H 3400 4250 50  0001 C CNN
 F 3 "" H 3400 4250 50  0000 C CNN
 	1    3400 5450
@@
 F 0 "P42" H 4600 5650 50  0000 C CNN
 F 1 "CONN_02X03" H 4600 5250 50  0000 C CNN
-F 2 "myParts:TMS-103-02-L-D-SE" H 4600 4250 50  0001 C CNN
+F 2 "myParts:TMS-103-01-L-D-SE" H 4600 4250 50  0001 C CNN
 F 3 "" H 4600 4250 50  0000 C CNN
 	1    4600 5450
@@
 F 0 "P31" H 8800 4250 50  0000 C CNN
 F 1 "CONN_02X03" H 8800 3850 50  0000 C CNN
-F 2 "myParts:TMS-103-02-L-D-SE" H 8800 2850 50  0001 C CNN
+F 2 "myParts:TMS-103-01-L-D-SE" H 8800 2850 50  0001 C CNN
 F 3 "" H 8800 2850 50  0000 C CNN
 	1    8800 4050
@@
 F 0 "P32" H 10050 4250 50  0000 C CNN
 F 1 "CONN_02X03" H 10050 3850 50  0000 C CNN
-F 2 "myParts:TMS-103-02-L-D-SE" H 10050 2850 50  0001 C CNN
+F 2 "myParts:TMS-103-01-L-D-SE" H 10050 2850 50  0001 C CNN
 F 3 "" H 10050 2850 50  0000 C CNN
 	1    10050 4050
@@
 F 0 "P25" H 8800 5500 50  0000 C CNN
 F 1 "CONN_02X03" H 8800 5100 50  0000 C CNN
-F 2 "myParts:TMS-103-02-L-D-SE" H 8800 4100 50  0001 C CNN
+F 2 "myParts:TMS-103-01-L-D-SE" H 8800 4100 50  0001 C CNN
 F 3 "" H 8800 4100 50  0000 C CNN
 	1    8800 5300
@@
 F 0 "P26" H 10050 5500 50  0000 C CNN
 F 1 "CONN_02X03" H 10050 5100 50  0000 C CNN
-F 2 "myParts:TMS-103-02-L-D-SE" H 10050 4100 50  0001 C CNN
+F 2 "myParts:TMS-103-01-L-D-SE" H 10050 4100 50  0001 C CNN
 F 3 "" H 10050 4100 50  0000 C CNN
 	1    10050 5300

Commit message: change d8 header
Parts:
- P21, P22, P23, P24, P27, P28, P29, P30, P35, P36, P37, P38, P43, P44, P45, P46: footprint Pin_Headers:Pin_Header_Angled_2x07_Pitch2.54mm -> myParts:SSW-107-02-T-D-RA
- P47: footprint myParts:TMS-103-01-L-D-SE -> myParts:SSW-107-02-T-D-RA
Changed lines of the file:
@@
 LIBS:valves
 LIBS:distributor8-cache
-EELAYER 25 0
+EELAYER 26 0
 EELAYER END
 $Descr A4 11693 8268
@@
 F 0 "P47" H 3400 4400 50  0000 C CNN
 F 1 "CONN_02X03" H 3400 4000 50  0000 C CNN
-F 2 "myParts:TMS-103-01-L-D-SE" H 3400 3000 50  0001 C CNN
+F 2 "myParts:SSW-107-02-T-D-RA" H 3400 3000 50  0001 C CNN
 F 3 "" H 3400 3000 50  0000 C CNN
 	1    3400 4200
@@
 F 0 "P21" H 2750 2750 50  0000 C CNN
 F 1 "CONN_02X07" V 2750 2350 50  0000 C CNN
-F 2 "Pin_Headers:Pin_Header_Angled_2x07_Pitch2.54mm" H 2750 1150 50  0001 C CNN
+F 2 "myParts:SSW-107-02-T-D-RA" H 2750 1150 50  0001 C CNN
 F 3 "" H 2750 1150 50  0000 C CNN
 	1    2750 2350
@@
 F 0 "P23" H 2700 1600 50  0000 C CNN
 F 1 "CONN_02X07" V 2700 1200 50  0000 C CNN
-F 2 "Pin_Headers:Pin_Header_Angled_2x07_Pitch2.54mm" H 2700 0   50  0001 C CNN
+F 2 "myParts:SSW-107-02-T-D-RA" H 2700 0   50  0001 C CNN
 F 3 "" H 2700 0   50  0000 C CNN
 	1    2700 1200
@@
 F 0 "P28" H 5350 2900 50  0000 C CNN
 F 1 "CONN_02X07" V 5350 2500 50  0000 C CNN
-F 2 "Pin_Headers:Pin_Header_Angled_2x07_Pitch2.54mm" H 5350 1300 50  0001 C CNN
+F 2 "myParts:SSW-107-02-T-D-RA" H 5350 1300 50  0001 C CNN
 F 3 "" H 5350 1300 50  0000 C CNN
 	1    5350 2500
@@
 F 0 "P30" H 5300 1550 50  0000 C CNN
 F 1 "CONN_02X07" V 5300 1150 50  0000 C CNN
-F 2 "Pin_Headers:Pin_Header_Angled_2x07_Pitch2.54mm" H 5300 -50 50  0001 C CNN
+F 2 "myParts:SSW-107-02-T-D-RA" H 5300 -50 50  0001 C CNN
 F 3 "" H 5300 -50 50  0000 C CNN
 	1    5300 1150
@@
 F 0 "P35" H 8000 2650 50  0000 C CNN
 F 1 "CONN_02X07" V 8000 2250 50  0000 C CNN
-F 2 "Pin_Headers:Pin_Header_Angled_2x07_Pitch2.54mm" H 8000 1050 50  0001 C CNN
+F 2 "myParts:SSW-107-02-T-D-RA" H 8000 1050 50  0001 C CNN
 F 3 "" H 8000 1050 50  0000 C CNN
 	1    8000 2250
@@
 F 0 "P37" H 7900 1600 50  0000 C CNN
 F 1 "CONN_02X07" V 7900 1200 50  0000 C CNN
-F 2 "Pin_Headers:Pin_Header_Angled_2x07_Pitch2.54mm" H 7900 0   50  0001 C CNN
+F 2 "myParts:SSW-107-02-T-D-RA" H 7900 0   50  0001 C CNN
 F 3 "" H 7900 0   50  0000 C CNN
 	1    7900 1200
@@
 F 0 "P43" H 10800 2750 50  0000 C CNN
 F 1 "CONN_02X07" V 10800 2350 50  0000 C CNN
-F 2 "Pin_Headers:Pin_Header_Angled_2x07_Pitch2.54mm" H 10800 1150 50  0001 C CNN
+F 2 "myParts:SSW-107-02-T-D-RA" H 10800 1150 50  0001 C CNN
 F 3 "" H 10800 1150 50  0000 C CNN
 	1    10800 2350
@@
 F 0 "P45" H 10800 1600 50  0000 C CNN
 F 1 "CONN_02X07" V 10800 1200 50  0000 C CNN
-F 2 "Pin_Headers:Pin_Header_Angled_2x07_Pitch2.54mm" H 10800 0   50  0001 C CNN
+F 2 "myParts:SSW-107-02-T-D-RA" H 10800 0   50  0001 C CNN
 F 3 "" H 10800 0   50  0000 C CNN
 	1    10800 1200
@@
 F 0 "P22" H 2750 6100 50  0000 C CNN
 F 1 "CONN_02X07" V 2750 5700 50  0000 C CNN
-F 2 "Pin_Headers:Pin_Header_Angled_2x07_Pitch2.54mm" H 2750 4500 50  0001 C CNN
+F 2 "myParts:SSW-107-02-T-D-RA" H 2750 4500 50  0001 C CNN
 F 3 "" H 2750 4500 50  0000 C CNN
 	1    2750 5700
@@
 F 0 "P24" H 2700 4650 50  0000 C CNN
 F 1 "CONN_02X07" V 2700 4250 50  0000 C CNN
-F 2 "Pin_Headers:Pin_Header_Angled_2x07_Pitch2.54mm" H 2700 3050 50  0001 C CNN
+F 2 "myParts:SSW-107-02-T-D-RA" H 2700 3050 50  0001 C CNN
 F 3 "" H 2700 3050 50  0000 C CNN
 	1    2700 4250
@@
 F 0 "P27" H 10800 5700 50  0000 C CNN
 F 1 "CONN_02X07" V 10800 5300 50  0000 C CNN
-F 2 "Pin_Headers:Pin_Header_Angled_2x07_Pitch2.54mm" H 10800 4100 50  0001 C CNN
+F 2 "myParts:SSW-107-02-T-D-RA" H 10800 4100 50  0001 C CNN
 F 3 "" H 10800 4100 50  0000 C CNN
 	1    10800 5300
@@
 F 0 "P29" H 10700 4550 50  0000 C CNN
 F 1 "CONN_02X07" V 10700 4150 50  0000 C CNN
-F 2 "Pin_Headers:Pin_Header_Angled_2x07_Pitch2.54mm" H 10700 2950 50  0001 C CNN
+F 2 "myParts:SSW-107-02-T-D-RA" H 10700 2950 50  0001 C CNN
 F 3 "" H 10700 2950 50  0000 C CNN
 	1    10700 4150
@@
 F 0 "P36" H 7950 5700 50  0000 C CNN
 F 1 "CONN_02X07" V 7950 5300 50  0000 C CNN
-F 2 "Pin_Headers:Pin_Header_Angled_2x07_Pitch2.54mm" H 7950 4100 50  0001 C CNN
+F 2 "myParts:SSW-107-02-T-D-RA" H 7950 4100 50  0001 C CNN
 F 3 "" H 7950 4100 50  0000 C CNN
 	1    7950 5300
@@
 F 0 "P38" H 8050 4550 50  0000 C CNN
 F 1 "CONN_02X07" V 8050 4150 50  0000 C CNN
-F 2 "Pin_Headers:Pin_Header_Angled_2x07_Pitch2.54mm" H 8050 2950 50  0001 C CNN
+F 2 "myParts:SSW-107-02-T-D-RA" H 8050 2950 50  0001 C CNN
 F 3 "" H 8050 2950 50  0000 C CNN
 	1    8050 4150
@@
 F 0 "P44" H 5350 5850 50  0000 C CNN
 F 1 "CONN_02X07" V 5350 5450 50  0000 C CNN
-F 2 "Pin_Headers:Pin_Header_Angled_2x07_Pitch2.54mm" H 5350 4250 50  0001 C CNN
+F 2 "myParts:SSW-107-02-T-D-RA" H 5350 4250 50  0001 C CNN
 F 3 "" H 5350 4250 50  0000 C CNN
 	1    5350 5450
@@
 F 0 "P46" H 5300 4700 50  0000 C CNN
 F 1 "CONN_02X07" V 5300 4300 50  0000 C CNN
-F 2 "Pin_Headers:Pin_Header_Angled_2x07_Pitch2.54mm" H 5300 3100 50  0001 C CNN
+F 2 "myParts:SSW-107-02-T-D-RA" H 5300 3100 50  0001 C CNN
 F 3 "" H 5300 3100 50  0000 C CNN
 	1    5300 4300
