File: KiCAD/referencePhotodiodeArray/reference-photodiode-array.sch (KiCad schematic (older format))
At the start: 22 parts

Commit message: made new photodiode array, fixed springpin board
Parts:
- D1, D2, D3, D4, D5, D6: footprint testPad:BPW34 -> myParts:BPW34
- W1, W10, W11, W12, W13, W14, W15, W16, W17, W2, W20, W3, W4, W5, W6, W7: footprint testPad:SolderWirePad_single_SMD_5x2.3mm -> myParts:SolderWirePad_single_SMD_4.7x3.2mm
Changed lines of the file:
@@
 LIBS:valves
 LIBS:reference-photodiode-array-cache
-EELAYER 25 0
+EELAYER 26 0
 EELAYER END
 $Descr A4 11693 8268
@@
 F 0 "D2" H 2420 2370 50  0000 L CNN
 F 1 "D_Photo" H 2360 2190 50  0000 C CNN
-F 2 "testPad:BPW34" H 2350 2300 50  0001 C CNN
+F 2 "myParts:BPW34" H 2350 2300 50  0001 C CNN
 F 3 "" H 2350 2300 50  0000 C CNN
 	1    2400 2300
@@
 F 0 "D3" H 2870 1670 50  0000 L CNN
 F 1 "D_Photo" H 2810 1490 50  0000 C CNN
-F 2 "testPad:BPW34" H 2800 1600 50  0001 C CNN
+F 2 "myParts:BPW34" H 2800 1600 50  0001 C CNN
 F 3 "" H 2800 1600 50  0000 C CNN
 	1    2850 1600
@@
 F 0 "D1" H 2420 1670 50  0000 L CNN
 F 1 "D_Photo" H 2360 1490 50  0000 C CNN
-F 2 "testPad:BPW34" H 2350 1600 50  0001 C CNN
+F 2 "myParts:BPW34" H 2350 1600 50  0001 C CNN
 F 3 "" H 2350 1600 50  0000 C CNN
 	1    2400 1600
@@
 F 0 "D5" H 3320 1670 50  0000 L CNN
 F 1 "D_Photo" H 3260 1490 50  0000 C CNN
-F 2 "testPad:BPW34" H 3250 1600 50  0001 C CNN
+F 2 "myParts:BPW34" H 3250 1600 50  0001 C CNN
 F 3 "" H 3250 1600 50  0000 C CNN
 	1    3300 1600
@@
 F 0 "D4" H 2870 2370 50  0000 L CNN
 F 1 "D_Photo" H 2810 2190 50  0000 C CNN
-F 2 "testPad:BPW34" H 2800 2300 50  0001 C CNN
+F 2 "myParts:BPW34" H 2800 2300 50  0001 C CNN
 F 3 "" H 2800 2300 50  0000 C CNN
 	1    2850 2300
@@
 F 0 "D6" H 3320 2370 50  0000 L CNN
 F 1 "D_Photo" H 3260 2190 50  0000 C CNN
-F 2 "testPad:BPW34" H 3250 2300 50  0001 C CNN
+F 2 "myParts:BPW34" H 3250 2300 50  0001 C CNN
 F 3 "" H 3250 2300 50  0000 C CNN
 	1    3300 2300
@@
 F 0 "W2" H 2400 1620 50  0000 C CNN
 F 1 "TEST_1P" H 2400 1550 50  0000 C CNN
-F 2 "testPad:SolderWirePad_single_SMD_5x2.3mm" H 2600 1350 50  0001 C CNN
+F 2 "myParts:SolderWirePad_single_SMD_4.7x3.2mm" H 2600 1350 50  0001 C CNN
 F 3 "" H 2600 1350 50  0000 C CNN
 	1    2400 1350
@@
 F 0 "W4" H 2850 1620 50  0000 C CNN
 F 1 "TEST_1P" H 2850 1550 50  0000 C CNN
-F 2 "testPad:SolderWirePad_single_SMD_5x2.3mm" H 3050 1350 50  0001 C CNN
+F 2 "myParts:SolderWirePad_single_SMD_4.7x3.2mm" H 3050 1350 50  0001 C CNN
 F 3 "" H 3050 1350 50  0000 C CNN
 	1    2850 1350
@@
 F 0 "W6" H 3300 1620 50  0000 C CNN
 F 1 "TEST_1P" H 3300 1550 50  0000 C CNN
-F 2 "testPad:SolderWirePad_single_SMD_5x2.3mm" H 3500 1350 50  0001 C CNN
+F 2 "myParts:SolderWirePad_single_SMD_4.7x3.2mm" H 3500 1350 50  0001 C CNN
 F 3 "" H 3500 1350 50  0000 C CNN
 	1    3300 1350
@@
 F 0 "W1" H 2050 2220 50  0000 C CNN
 F 1 "TEST_1P" H 2050 2150 50  0000 C CNN
-F 2 "testPad:SolderWirePad_single_SMD_5x2.3mm" H 2250 1950 50  0001 C CNN
+F 2 "myParts:SolderWirePad_single_SMD_4.7x3.2mm" H 2250 1950 50  0001 C CNN
 F 3 "" H 2250 1950 50  0000 C CNN
 	1    2050 1950
@@
 F 0 "W10" H 4100 2220 50  0000 C CNN
 F 1 "TEST_1P" H 4100 2150 50  0000 C CNN
-F 2 "testPad:SolderWirePad_single_SMD_5x2.3mm" H 4300 1950 50  0001 C CNN
+F 2 "myParts:SolderWirePad_single_SMD_4.7x3.2mm" H 4300 1950 50  0001 C CNN
 F 3 "" H 4300 1950 50  0000 C CNN
 	1    4100 1950
@@
 F 0 "W3" H 2400 2820 50  0000 C CNN
 F 1 "TEST_1P" H 2400 2750 50  0000 C CNN
-F 2 "testPad:SolderWirePad_single_SMD_5x2.3mm" H 2600 2550 50  0001 C CNN
+F 2 "myParts:SolderWirePad_single_SMD_4.7x3.2mm" H 2600 2550 50  0001 C CNN
 F 3 "" H 2600 2550 50  0000 C CNN
 	1    2400 2550
@@
 F 0 "W5" H 2850 2820 50  0000 C CNN
 F 1 "TEST_1P" H 2850 2750 50  0000 C CNN
-F 2 "testPad:SolderWirePad_single_SMD_5x2.3mm" H 3050 2550 50  0001 C CNN
+F 2 "myParts:SolderWirePad_single_SMD_4.7x3.2mm" H 3050 2550 50  0001 C CNN
 F 3 "" H 3050 2550 50  0000 C CNN
 	1    2850 2550
@@
 F 0 "W7" H 3300 2820 50  0000 C CNN
 F 1 "TEST_1P" H 3300 2750 50  0000 C CNN
-F 2 "testPad:SolderWirePad_single_SMD_5x2.3mm" H 3500 2550 50  0001 C CNN
+F 2 "myParts:SolderWirePad_single_SMD_4.7x3.2mm" H 3500 2550 50  0001 C CNN
 F 3 "" H 3500 2550 50  0000 C CNN
 	1    3300 2550
@@
 F 0 "W12" H 2400 1620 50  0000 C CNN
 F 1 "TEST_1P" H 2400 1550 50  0000 C CNN
-F 2 "testPad:SolderWirePad_single_SMD_5x2.3mm" H 2600 1350 50  0001 C CNN
+F 2 "myParts:SolderWirePad_single_SMD_4.7x3.2mm" H 2600 1350 50  0001 C CNN
 F 3 "" H 2600 1350 50  0000 C CNN
 	1    2400 1350
@@
 F 0 "W14" H 2850 1620 50  0000 C CNN
 F 1 "TEST_1P" H 2850 1550 50  0000 C CNN
-F 2 "testPad:SolderWirePad_single_SMD_5x2.3mm" H 3050 1350 50  0001 C CNN
+F 2 "myParts:SolderWirePad_single_SMD_4.7x3.2mm" H 3050 1350 50  0001 C CNN
 F 3 "" H 3050 1350 50  0000 C CNN
 	1    2850 1350
@@
 F 0 "W16" H 3300 1620 50  0000 C CNN
 F 1 "TEST_1P" H 3300 1550 50  0000 C CNN
-F 2 "testPad:SolderWirePad_single_SMD_5x2.3mm" H 3500 1350 50  0001 C CNN
+F 2 "myParts:SolderWirePad_single_SMD_4.7x3.2mm" H 3500 1350 50  0001 C CNN
 F 3 "" H 3500 1350 50  0000 C CNN
 	1    3300 1350
@@
 F 0 "W17" H 3300 2820 50  0000 C CNN
 F 1 "TEST_1P" H 3300 2750 50  0000 C CNN
-F 2 "testPad:SolderWirePad_single_SMD_5x2.3mm" H 3500 2550 50  0001 C CNN
+F 2 "myParts:SolderWirePad_single_SMD_4.7x3.2mm" H 3500 2550 50  0001 C CNN
 F 3 "" H 3500 2550 50  0000 C CNN
 	1    3300 2550
@@
 F 0 "W15" H 2850 2820 50  0000 C CNN
 F 1 "TEST_1P" H 2850 2750 50  0000 C CNN
-F 2 "testPad:SolderWirePad_single_SMD_5x2.3mm" H 3050 2550 50  0001 C CNN
+F 2 "myParts:SolderWirePad_single_SMD_4.7x3.2mm" H 3050 2550 50  0001 C CNN
 F 3 "" H 3050 2550 50  0000 C CNN
 	1    2850 2550
@@
 F 0 "W13" H 2400 2820 50  0000 C CNN
 F 1 "TEST_1P" H 2400 2750 50  0000 C CNN
-F 2 "testPad:SolderWirePad_single_SMD_5x2.3mm" H 2600 2550 50  0001 C CNN
+F 2 "myParts:SolderWirePad_single_SMD_4.7x3.2mm" H 2600 2550 50  0001 C CNN
 F 3 "" H 2600 2550 50  0000 C CNN
 	1    2400 2550
@@
 F 0 "W11" H 2050 2220 50  0000 C CNN
 F 1 "TEST_1P" H 2050 2150 50  0000 C CNN
-F 2 "testPad:SolderWirePad_single_SMD_5x2.3mm" H 2250 1950 50  0001 C CNN
+F 2 "myParts:SolderWirePad_single_SMD_4.7x3.2mm" H 2250 1950 50  0001 C CNN
 F 3 "" H 2250 1950 50  0000 C CNN
 	1    2050 1950
@@
 F 0 "W20" H 4100 2220 50  0000 C CNN
 F 1 "TEST_1P" H 4100 2150 50  0000 C CNN
-F 2 "testPad:SolderWirePad_single_SMD_5x2.3mm" H 4300 1950 50  0001 C CNN
+F 2 "myParts:SolderWirePad_single_SMD_4.7x3.2mm" H 4300 1950 50  0001 C CNN
 F 3 "" H 4300 1950 50  0000 C CNN
 	1    4100 1950
