File: KiCAD/plane8/plane8.kicad_pcb (KiCad board)
At the start: 4 copper layers, 273 x 30 mm, 48 parts, among them CON1 AVR-JTAG-10, J1 CONN_02X03, J10 CONN_02X04, J11 CONN_01X04, J12 CONN_02X04, J2 CONN_01X04, J3 CONN_02X04, J4 CONN_02X04, J5 CONN_02X04, J6 CONN_02X04, J7 CONN_02X04, J8 CONN_02X04, J9 CONN_02X04, P1 CONN_02X07, P10 CONN_02X07, P11 CONN_02X07, P12 CONN_02X07, P13 CONN_02X07, P14 CONN_02X07, P15 CONN_02X07, P16 CONN_02X07, P17 CONN_02X04, P18 CONN_01X02, P19 CONN_01X17, P2 CONN_02X07, P20 CONN_01X17, P21 CONN_01X02, P22 CONN_01X02, P3 CONN_02X07, P4 CONN_02X07, P5 CONN_02X07, P6 CONN_02X07, P7 CONN_02X07, P8 CONN_02X07, P9 CONN_02X07, U1 ARDUINO_MICRO

Commit message: fix silk
Other:
- board text added: "c60b50c"
Changed lines of the file:
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@@
     (area -2.238001 -18.30028 273.075001 16.491333)
     (thickness 1.6)
-    (drawings 22)
+    (drawings 23)
     (tracks 784)
     (zones 0)
@@
     (tags "resistor 0805")
     (attr smd)
-    (fp_text reference R5 (at 0 -1.7 90) (layer F.SilkS)
+    (fp_text reference R5 (at -0.05 1.98 90) (layer F.SilkS)
       (effects (font (size 1 1) (thickness 0.15)))
     )
@@
     (descr "Through hole straight pin header, 2x04, 2.54mm pitch, double rows")
     (tags "Through hole pin header THT 2x04 2.54mm double row")
-    (fp_text reference J3 (at 1.27 -2.33) (layer F.SilkS)
+    (fp_text reference J3 (at -2.59 0.02) (layer F.SilkS)
       (effects (font (size 1 1) (thickness 0.15)))
     )
@@
     (descr "Through hole straight pin header, 2x04, 2.54mm pitch, double rows")
     (tags "Through hole pin header THT 2x04 2.54mm double row")
-    (fp_text reference J5 (at 1.27 -2.33) (layer F.SilkS)
+    (fp_text reference J5 (at -2.69 -0.04) (layer F.SilkS)
       (effects (font (size 1 1) (thickness 0.15)))
     )
@@
     (descr "Through hole straight pin header, 2x04, 2.54mm pitch, double rows")
     (tags "Through hole pin header THT 2x04 2.54mm double row")
-    (fp_text reference J6 (at 1.27 -2.33) (layer F.SilkS)
+    (fp_text reference J6 (at -2.8 -0.15) (layer F.SilkS)
       (effects (font (size 1 1) (thickness 0.15)))
     )
@@
     (descr "Through hole straight pin header, 2x04, 2.54mm pitch, double rows")
     (tags "Through hole pin header THT 2x04 2.54mm double row")
-    (fp_text reference J7 (at 1.27 -2.33) (layer F.SilkS)
+    (fp_text reference J7 (at -2.86 0.02) (layer F.SilkS)
       (effects (font (size 1 1) (thickness 0.15)))
     )
@@
     (descr "Through hole straight pin header, 2x04, 2.54mm pitch, double rows")
     (tags "Through hole pin header THT 2x04 2.54mm double row")
-    (fp_text reference J8 (at 1.27 -2.33) (layer F.SilkS)
+    (fp_text reference J8 (at -2.82 -0.04) (layer F.SilkS)
       (effects (font (size 1 1) (thickness 0.15)))
     )
@@
     (descr "Through hole straight pin header, 2x04, 2.54mm pitch, double rows")
     (tags "Through hole pin header THT 2x04 2.54mm double row")
-    (fp_text reference J9 (at 1.27 -2.33) (layer F.SilkS)
+    (fp_text reference J9 (at -2.84 -0.04) (layer F.SilkS)
       (effects (font (size 1 1) (thickness 0.15)))
     )
@@
     (descr "Through hole straight pin header, 2x04, 2.54mm pitch, double rows")
     (tags "Through hole pin header THT 2x04 2.54mm double row")
-    (fp_text reference J12 (at 1.27 -2.33) (layer F.SilkS)
+    (fp_text reference J12 (at -3.41 -0.09) (layer F.SilkS)
       (effects (font (size 1 1) (thickness 0.15)))
     )
@@
     )
   )
+  (gr_text c60b50c (at 251.62 -12.88) (layer F.SilkS)
+    (effects (font (size 1.5 1.5) (thickness 0.3)))
+  )
   (gr_text H (at 153.67 -6.35) (layer F.SilkS)

Commit message: update commit silk
Other:
- board text added: "84dc42b"
- board text removed: "c60b50c"
Changed lines of the file:
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@@
     )
   )
-  (gr_text c60b50c (at 251.62 -12.88) (layer F.SilkS)
+  (gr_text 84dc42b (at 251.62 -12.88) (layer F.SilkS)
     (effects (font (size 1.5 1.5) (thickness 0.3)))
   )

Commit message: fix plane8 connector spacing
Parts:
- moved P1 1.27 mm to (17.8, -6.38)
- moved P10 1.27 mm to (88.9, 6.38)
- moved P11 1.27 mm to (106.7, -6.38)
- moved P12 1.27 mm to (106.7, 6.38)
- moved P13 1.27 mm to (124.5, -6.38)
- moved P14 1.27 mm to (124.5, 6.38)
- moved P15 1.27 mm to (142.2, -6.38)
- moved P16 1.27 mm to (142.2, 6.38)
- moved P2 1.27 mm to (17.8, 6.38)
- moved P3 1.27 mm to (35.6, -6.38)
- moved P4 1.27 mm to (35.6, 6.38)
- moved P5 1.27 mm to (53.3, -6.38)
- moved P6 1.27 mm to (53.3, 6.38)
- moved P7 1.27 mm to (71.1, -6.38)
- moved P8 1.27 mm to (71.1, 6.38)
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Routing:
- net MISO: track 341.1 -> 229.1 mm, vias 5 -> 1
- net GND: track 1.36 -> 69.9 mm
- net SDA: track 281.9 -> 230.4 mm, vias 5 -> 0
- net MOSI: track 260.7 -> 213.7 mm, vias 5 -> 0
- net SCL: track 265.6 -> 234.2 mm, vias 4 -> 0
- net TDO: track 45.9 -> 77.1 mm, vias 1 -> 0
- net SCK: track 219.0 -> 240.2 mm, vias 1 -> 2
- net A_I+: track 163.1 -> 175.0 mm
- net A_V+: track 173.2 -> 161.5 mm, vias 0 -> 1
- net Net-(J10-Pad6): track 103.2 -> 114.6 mm
- net LIM_B: track 70.3 -> 61.6 mm, vias 0 -> 1
- net A_V-: track 162.7 -> 169.5 mm
- net TDI: track 68.5 -> 74.7 mm
- net Net-(J2-Pad4): track 111.7 -> 117.8 mm, vias 1 -> 0
- net H_I+: track 44.9 -> 39.1 mm
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
Commit message: update commit silk
Other:
- board text added: "1d49a91"
- board text removed: "84dc42b"
Changed lines of the file:
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@@
     )
   )
-  (gr_text 84dc42b (at 251.62 -12.88) (layer F.SilkS)
+  (gr_text 1d49a91 (at 251.62 -12.88) (layer F.SilkS)
     (effects (font (size 1.5 1.5) (thickness 0.3)))
   )

Commit message: add mounting holes
Parts:
- added J13: TEST_1P, Mounting_Holes:MountingHole_2.2mm_M2_Pad, F.Cu at (152.4, 7.00)
- added J14: TEST_1P, Mounting_Holes:MountingHole_2.2mm_M2_Pad, F.Cu at (152.4, -7.00)
- moved J4 5.68 mm to (161.3, 1.27)
- moved J10 5.08 mm to (161.3, -10.2)
- moved R6 2.62 mm to (168.9, -7.00)
- moved C1 2.54 mm to (168.9, -9.00)
Routing:
- net GND: track 69.9 -> 464.2 mm
- net MISO: track 229.1 -> 257.7 mm, vias 1 -> 2
- net TCK: track 65.2 -> 40.3 mm
- net Net-(J10-Pad6): track 114.6 -> 98.2 mm
- net TDO: track 77.1 -> 63.0 mm
- net Net-(J2-Pad2): track 113.1 -> 101.2 mm
- net SCK: track 240.2 -> 230.3 mm, vias 2 -> 0
- net Net-(C1-Pad2): track 116.1 -> 125.2 mm
- net SDA: track 230.4 -> 237.4 mm
- net TDI: track 74.7 -> 68.0 mm
- net /ANODE: track 186.6 -> 179.9 mm
- net MOSI: track 213.7 -> 220.0 mm
- net H_V+: track 38.4 -> 44.4 mm
- net A_I-: track 164.7 -> 170.5 mm
- net Net-(J2-Pad1): track 108.5 -> 102.9 mm, vias 0 -> 1
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
Commit message: update plane8 commit silk
Other:
- board text added: "b61f9ad"
- board text removed: "1d49a91"
Changed lines of the file:
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@@
       (net 214 "Net-(J14-Pad1)"))
   )
-  (gr_text 1d49a91 (at 251.62 -12.88) (layer F.SilkS)
+  (gr_text b61f9ad (at 251.62 -12.88) (layer F.SilkS)
     (effects (font (size 1.5 1.5) (thickness 0.3)))
   )

Commit message: generate order packages
Other:
- board text added: "17e0726"
- board text removed: "b61f9ad"
Changed lines of the file:
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@@
     (pcbplotparams
       (layerselection 0x010fc_ffffffff)
-      (usegerberextensions false)
+      (usegerberextensions true)
       (excludeedgelayer true)
       (linewidth 0.150000)
@@
       (plotinvisibletext false)
       (padsonsilk false)
-      (subtractmaskfromsilk false)
+      (subtractmaskfromsilk true)
       (outputformat 1)
       (mirror false)
@@
       (net 214 "Net-(J14-Pad1)"))
   )
-  (gr_text b61f9ad (at 251.62 -12.88) (layer F.SilkS)
+  (gr_text 17e0726 (at 251.62 -12.88) (layer F.SilkS)
     (effects (font (size 1.5 1.5) (thickness 0.3)))
   )

Commit message: fix pwr/gnd swap, fix extra clock signal name, fix pin hole sizes
Connections:
- P10 pad 5: SCK -> +3V3
- P10 pad 6: CLK -> SCK
- P10 pad 7: GND -> +5V
- P10 pad 8: +5V -> GND
- P12 pad 5: SCK -> +3V3
- P12 pad 6: CLK -> SCK
- P12 pad 7: GND -> +5V
- P12 pad 8: +5V -> GND
- P14 pad 5: SCK -> +3V3
- P14 pad 6: CLK -> SCK
- P14 pad 7: GND -> +5V
- P14 pad 8: +5V -> GND
- P16 pad 5: SCK -> +3V3
- P16 pad 6: CLK -> SCK
- P16 pad 7: GND -> +5V
- P16 pad 8: +5V -> GND
- P2 pad 5: SCK -> +3V3
- P2 pad 6: CLK -> SCK
- P2 pad 7: GND -> +5V
- P2 pad 8: +5V -> GND
- P4 pad 5: SCK -> +3V3
- P4 pad 6: CLK -> SCK
- P4 pad 7: GND -> +5V
- P4 pad 8: +5V -> GND
- P6 pad 5: SCK -> +3V3
- P6 pad 6: CLK -> SCK
- P6 pad 7: GND -> +5V
- P6 pad 8: +5V -> GND
- P8 pad 5: SCK -> +3V3
- P8 pad 6: CLK -> SCK
- P8 pad 7: GND -> +5V
- P8 pad 8: +5V -> GND
Routing:
- net +5V: track 0.00 -> 477.7 mm, vias 0 -> 3
- net GND: track 464.2 -> 0.00 mm, vias 1 -> 0
- net +3V3: track 0.00 -> 271.6 mm, vias 0 -> 2
- net CLK: track 135.0 -> 0.00 mm
- net SCK: track 230.3 -> 221.0 mm
- net /CATHODE: track 174.2 -> 177.0 mm
- net Net-(J2-Pad2): track 101.2 -> 103.0 mm
- added copper zone on B.Cu, net +5V
- added copper zone on F.Cu, net GND
- removed copper zone on F.Cu, net +5V
- removed copper zone on B.Cu, net GND
