File: KiCAD/plane8/plane8.sch (KiCad schematic (older format))
At the start: 47 parts, among them CON1 AVR-JTAG-10, J1 CONN_02X03, J10 CONN_02X04, J11 CONN_01X04, J12 CONN_02X04, J2 CONN_01X04, J3 CONN_02X04, J4 CONN_02X04, J5 CONN_02X04, J6 CONN_02X04, J7 CONN_02X04, J8 CONN_02X04, J9 CONN_02X04, P1 CONN_02X07, P10 CONN_02X07, P11 CONN_02X07, P12 CONN_02X07, P13 CONN_02X07, P14 CONN_02X07, P15 CONN_02X07, P16 CONN_02X07, P17 CONN_02X04, P18 CONN_01X02, P19 CONN_01X17, P2 CONN_02X07, P20 CONN_01X17, P21 CONN_01X02, P22 CONN_01X02, P3 CONN_02X07, P4 CONN_02X07, P5 CONN_02X07, P6 CONN_02X07, P7 CONN_02X07, P8 CONN_02X07, P9 CONN_02X07, U1 ARDUINO_MICRO

Commit message: add mounting holes
Parts:
- added J13, J14: TEST_1P, Mounting_Holes:MountingHole_2.2mm_M2_Pad, symbol TEST_1P
Connections:
- no-connect marks 143 -> 145
Changed lines of the file:
@@
 NoConn ~ 10400 1700
 $Comp
-L GND #PWR01
+L GND #PWR19
 U 1 1 590B0B39
 P 8700 2200
-F 0 "#PWR01" H 8700 1950 50  0001 C CNN
+F 0 "#PWR19" H 8700 1950 50  0001 C CNN
 F 1 "GND" H 8700 2050 50  0000 C CNN
 F 2 "" H 8700 2200 50  0000 C CNN
@@
 1
 $Comp
-L +5V #PWR02
+L +5V #PWR23
 U 1 1 590B0B40
 P 10600 950
-F 0 "#PWR02" H 10600 800 50  0001 C CNN
+F 0 "#PWR23" H 10600 800 50  0001 C CNN
 F 1 "+5V" H 10600 1090 28  0000 C CNN
 F 2 "" H 10600 950 50  0000 C CNN
@@
 $EndComp
 $Comp
-L GND #PWR03
+L GND #PWR27
 U 1 1 590B0B46
 P 10800 1600
-F 0 "#PWR03" H 10800 1350 50  0001 C CNN
+F 0 "#PWR27" H 10800 1350 50  0001 C CNN
 F 1 "GND" H 10800 1450 50  0000 C CNN
 F 2 "" H 10800 1600 50  0000 C CNN
@@
 $EndComp
 $Comp
-L +3.3V #PWR04
+L +3.3V #PWR24
 U 1 1 590B0B4C
 P 10700 950
-F 0 "#PWR04" H 10700 800 50  0001 C CNN
+F 0 "#PWR24" H 10700 800 50  0001 C CNN
 F 1 "+3.3V" H 10700 1090 28  0000 C CNN
 F 2 "" H 10700 950 50  0000 C CNN
@@
 SCK
 $Comp
-L +5V #PWR05
+L +5V #PWR20
 U 1 1 590B0B75
 P 9950 3100
-F 0 "#PWR05" H 9950 2950 50  0001 C CNN
+F 0 "#PWR20" H 9950 2950 50  0001 C CNN
 F 1 "+5V" H 9950 3240 28  0000 C CNN
 F 2 "" H 9950 3100 50  0000 C CNN
@@
 $EndComp
 $Comp
-L GND #PWR06
+L GND #PWR21
 U 1 1 590B0B7B
 P 10200 3300
-F 0 "#PWR06" H 10200 3050 50  0001 C CNN
+F 0 "#PWR21" H 10200 3050 50  0001 C CNN
 F 1 "GND" H 10200 3150 50  0000 C CNN
 F 2 "" H 10200 3300 50  0000 C CNN
@@
 SCL
 $Comp
-L +5V #PWR07
+L +5V #PWR30
 U 1 1 590B0BC8
 P 11150 3150
-F 0 "#PWR07" H 11150 3000 50  0001 C CNN
+F 0 "#PWR30" H 11150 3000 50  0001 C CNN
 F 1 "+5V" H 11150 3290 28  0000 C CNN
 F 2 "" H 11150 3150 50  0000 C CNN
@@
 $EndComp
 $Comp
-L +3.3V #PWR08
+L +3.3V #PWR33
 U 1 1 590B0408
 P 11850 750
-F 0 "#PWR08" H 11850 600 50  0001 C CNN
+F 0 "#PWR33" H 11850 600 50  0001 C CNN
 F 1 "+3.3V" H 11850 890 28  0000 C CNN
 F 2 "" H 11850 750 50  0000 C CNN
@@
 $EndComp
 $Comp
-L +5V #PWR09
+L +5V #PWR32
 U 1 1 590B040E
 P 11700 750
-F 0 "#PWR09" H 11700 600 50  0001 C CNN
+F 0 "#PWR32" H 11700 600 50  0001 C CNN
 F 1 "+5V" H 11700 890 28  0000 C CNN
 F 2 "" H 11700 750 50  0000 C CNN
@@
 $EndComp
 $Comp
-L GND #PWR010
+L GND #PWR31
 U 1 1 590B0414
 P 11550 800
-F 0 "#PWR010" H 11550 550 50  0001 C CNN
+F 0 "#PWR31" H 11550 550 50  0001 C CNN
 F 1 "GND" H 11550 650 50  0000 C CNN
 F 2 "" H 11550 800 50  0000 C CNN
@@
 $EndComp
 $Comp
-L PWR_FLAG #FLG011
+L PWR_FLAG #FLG1
 U 1 1 590B041A
 P 11550 750
-F 0 "#FLG011" H 11550 825 50  0001 C CNN
+F 0 "#FLG1" H 11550 825 50  0001 C CNN
 F 1 "PWR_FLAG" H 11550 900 50  0001 C CNN
 F 2 "" H 11550 750 50  0000 C CNN
@@
 $EndComp
 $Comp
-L PWR_FLAG #FLG012
+L PWR_FLAG #FLG2
 U 1 1 590B0420
 P 11700 800
-F 0 "#FLG012" H 11700 875 50  0001 C CNN
+F 0 "#FLG2" H 11700 875 50  0001 C CNN
 F 1 "PWR_FLAG" H 11700 950 50  0001 C CNN
 F 2 "" H 11700 800 50  0000 C CNN
@@
 $EndComp
 $Comp
-L PWR_FLAG #FLG013
+L PWR_FLAG #FLG3
 U 1 1 590B0426
 P 11850 800
-F 0 "#FLG013" H 11850 875 50  0001 C CNN
+F 0 "#FLG3" H 11850 875 50  0001 C CNN
 F 1 "PWR_FLAG" H 11850 950 50  0001 C CNN
 F 2 "" H 11850 800 50  0000 C CNN
@@
 $EndComp
 $Comp
-L +5V #PWR014
+L +5V #PWR25
 U 1 1 590B1376
 P 10700 5000
-F 0 "#PWR014" H 10700 4850 50  0001 C CNN
+F 0 "#PWR25" H 10700 4850 50  0001 C CNN
 F 1 "+5V" H 10700 5140 28  0000 C CNN
 F 2 "" H 10700 5000 50  0000 C CNN
@@
 NoConn ~ 10150 4050
 $Comp
-L GND #PWR015
+L GND #PWR28
 U 1 1 590B138F
 P 10800 4250
-F 0 "#PWR015" H 10800 4000 50  0001 C CNN
+F 0 "#PWR28" H 10800 4000 50  0001 C CNN
 F 1 "GND" H 10800 4100 50  0000 C CNN
 F 2 "" H 10800 4250 50  0000 C CNN
@@
 $EndComp
 $Comp
-L +5V #PWR016
+L +5V #PWR29
 U 1 1 590B1395
 P 10900 3750
-F 0 "#PWR016" H 10900 3600 50  0001 C CNN
+F 0 "#PWR29" H 10900 3600 50  0001 C CNN
 F 1 "+5V" H 10900 3890 28  0000 C CNN
 F 2 "" H 10900 3750 50  0000 C CNN
@@
 $EndComp
 $Comp
-L +5V #PWR017
+L +5V #PWR17
 U 1 1 590B13A4
 P 8650 3550
-F 0 "#PWR017" H 8650 3400 50  0001 C CNN
+F 0 "#PWR17" H 8650 3400 50  0001 C CNN
 F 1 "+5V" H 8650 3690 28  0000 C CNN
 F 2 "" H 8650 3550 50  0000 C CNN
@@
 $EndComp
 $Comp
-L GND #PWR018
+L GND #PWR18
 U 1 1 590B13B1
 P 8650 4350
-F 0 "#PWR018" H 8650 4100 50  0001 C CNN
+F 0 "#PWR18" H 8650 4100 50  0001 C CNN
 F 1 "GND" H 8650 4200 50  0000 C CNN
 F 2 "" H 8650 4350 50  0000 C CNN
@@
 AIN0
 $Comp
-L GND #PWR019
+L GND #PWR26
 U 1 1 590B13B8
 P 10700 6250
-F 0 "#PWR019" H 10700 6000 50  0001 C CNN
+F 0 "#PWR26" H 10700 6000 50  0001 C CNN
 F 1 "GND" H 10700 6100 50  0000 C CNN
 F 2 "" H 10700 6250 50  0000 C CNN
@@
 EN
 $Comp
-L GND #PWR020
+L GND #PWR22
 U 1 1 590B2F0E
 P 10400 4700
-F 0 "#PWR020" H 10400 4450 50  0001 C CNN
+F 0 "#PWR22" H 10400 4450 50  0001 C CNN
 F 1 "GND" H 10400 4550 50  0000 C CNN
 F 2 "" H 10400 4700 50  0000 C CNN
@@
 B_I-
 $Comp
-L GND #PWR021
+L GND #PWR3
 U 1 1 590B5DB1
 P 2550 2600
-F 0 "#PWR021" H 2550 2350 50  0001 C CNN
+F 0 "#PWR3" H 2550 2350 50  0001 C CNN
 F 1 "GND" H 2550 2450 50  0000 C CNN
 F 2 "" H 2550 2600 50  0000 C CNN
@@
 CLK
 $Comp
-L +5V #PWR022
+L +5V #PWR4
 U 1 1 590C204F
 P 2550 3950
-F 0 "#PWR022" H 2550 3800 50  0001 C CNN
+F 0 "#PWR4" H 2550 3800 50  0001 C CNN
 F 1 "+5V" H 2550 4090 28  0000 C CNN
 F 2 "" H 2550 3950 50  0000 C CNN
@@
 $EndComp
 $Comp
-L +5V #PWR023
+L +5V #PWR8
 U 1 1 590C2464
 P 4100 4000
-F 0 "#PWR023" H 4100 3850 50  0001 C CNN
+F 0 "#PWR8" H 4100 3850 50  0001 C CNN
 F 1 "+5V" H 4100 4140 28  0000 C CNN
 F 2 "" H 4100 4000 50  0000 C CNN
@@
 	2450 2600 2450 3050
 $Comp
-L +5V #PWR024
+L +5V #PWR12
 U 1 1 590C33D5
 P 5650 3950
-F 0 "#PWR024" H 5650 3800 50  0001 C CNN
+F 0 "#PWR12" H 5650 3800 50  0001 C CNN
 F 1 "+5V" H 5650 4090 28  0000 C CNN
 F 2 "" H 5650 3950 50  0000 C CNN
@@
 $EndComp
 $Comp
-L +5V #PWR025
+L +5V #PWR16
 U 1 1 590C3442
 P 7300 4000
-F 0 "#PWR025" H 7300 3850 50  0001 C CNN
+F 0 "#PWR16" H 7300 3850 50  0001 C CNN
 F 1 "+5V" H 7300 4140 28  0000 C CNN
 F 2 "" H 7300 4000 50  0000 C CNN
@@
 $EndComp
 $Comp
-L +5V #PWR026
+L +5V #PWR2
 U 1 1 590C34AF
 P 1000 7600
-F 0 "#PWR026" H 1000 7450 50  0001 C CNN
+F 0 "#PWR2" H 1000 7450 50  0001 C CNN
 F 1 "+5V" H 1000 7740 28  0000 C CNN
 F 2 "" H 1000 7600 50  0000 C CNN
@@
 $EndComp
 $Comp
-L +5V #PWR027
+L +5V #PWR6
 U 1 1 590C36A4
 P 2600 7650
-F 0 "#PWR027" H 2600 7500 50  0001 C CNN
+F 0 "#PWR6" H 2600 7500 50  0001 C CNN
 F 1 "+5V" H 2600 7790 28  0000 C CNN
 F 2 "" H 2600 7650 50  0000 C CNN
@@
 $EndComp
 $Comp
-L +5V #PWR028
+L +5V #PWR10
 U 1 1 590C3711
 P 4150 7600
-F 0 "#PWR028" H 4150 7450 50  0001 C CNN
+F 0 "#PWR10" H 4150 7450 50  0001 C CNN
 F 1 "+5V" H 4150 7740 28  0000 C CNN
 F 2 "" H 4150 7600 50  0000 C CNN
@@
 $EndComp
 $Comp
-L +5V #PWR029
+L +5V #PWR14
 U 1 1 590C38D5
 P 5750 7600
-F 0 "#PWR029" H 5750 7450 50  0001 C CNN
+F 0 "#PWR14" H 5750 7450 50  0001 C CNN
 F 1 "+5V" H 5750 7740 28  0000 C CNN
 F 2 "" H 5750 7600 50  0000 C CNN
@@
 	2450 3950 2450 3550
 $Comp
-L GND #PWR030
+L GND #PWR7
 U 1 1 590C4991
 P 4100 2650
-F 0 "#PWR030" H 4100 2400 50  0001 C CNN
+F 0 "#PWR7" H 4100 2400 50  0001 C CNN
 F 1 "GND" H 4100 2500 50  0000 C CNN
 F 2 "" H 4100 2650 50  0000 C CNN
@@
 $EndComp
 $Comp
-L GND #PWR031
+L GND #PWR11
 U 1 1 590C49FE
 P 5650 2600
-F 0 "#PWR031" H 5650 2350 50  0001 C CNN
+F 0 "#PWR11" H 5650 2350 50  0001 C CNN
 F 1 "GND" H 5650 2450 50  0000 C CNN
 F 2 "" H 5650 2600 50  0000 C CNN
@@
 $EndComp
 $Comp
-L GND #PWR032
+L GND #PWR15
 U 1 1 590C4A6B
 P 7300 2650
-F 0 "#PWR032" H 7300 2400 50  0001 C CNN
+F 0 "#PWR15" H 7300 2400 50  0001 C CNN
 F 1 "GND" H 7300 2500 50  0000 C CNN
 F 2 "" H 7300 2650 50  0000 C CNN
@@
 $EndComp
 $Comp
-L GND #PWR033
+L GND #PWR1
 U 1 1 590C4D55
 P 1000 6250
-F 0 "#PWR033" H 1000 6000 50  0001 C CNN
+F 0 "#PWR1" H 1000 6000 50  0001 C CNN
 F 1 "GND" H 1000 6100 50  0000 C CNN
 F 2 "" H 1000 6250 50  0000 C CNN
@@
 $EndComp
 $Comp
-L GND #PWR034
+L GND #PWR5
 U 1 1 590C4DC2
 P 2600 6300
-F 0 "#PWR034" H 2600 6050 50  0001 C CNN
+F 0 "#PWR5" H 2600 6050 50  0001 C CNN
 F 1 "GND" H 2600 6150 50  0000 C CNN
 F 2 "" H 2600 6300 50  0000 C CNN
@@
 $EndComp
 $Comp
-L GND #PWR035
+L GND #PWR9
 U 1 1 590C4E2F
 P 4150 6250
-F 0 "#PWR035" H 4150 6000 50  0001 C CNN
+F 0 "#PWR9" H 4150 6000 50  0001 C CNN
 F 1 "GND" H 4150 6100 50  0000 C CNN
 F 2 "" H 4150 6250 50  0000 C CNN
@@
 $EndComp
 $Comp
-L GND #PWR036
+L GND #PWR13
 U 1 1 590C4FC2
 P 5750 6250
-F 0 "#PWR036" H 5750 6000 50  0001 C CNN
+F 0 "#PWR13" H 5750 6000 50  0001 C CNN
 F 1 "GND" H 5750 6100 50  0000 C CNN
 F 2 "" H 5750 6250 50  0000 C CNN
@@
 Text Notes 7250 5250 0    60   ~ 0
 SWITCH PROTECTION
+$Comp
+L TEST_1P J13
+U 1 1 590BBDCD
+P 700 700
+F 0 "J13" H 758 820 50  0000 L CNN
+F 1 "TEST_1P" H 758 729 50  0000 L CNN
+F 2 "Mounting_Holes:MountingHole_2.2mm_M2_Pad" H 900 700 50  0001 C CNN
+F 3 "" H 900 700 50  0001 C CNN
+	1    700  700
+	1    0    0    -1
+$EndComp
+$Comp
+L TEST_1P J14
+U 1 1 590BBF13
+P 700 1050
+F 0 "J14" H 758 1170 50  0000 L CNN
+F 1 "TEST_1P" H 758 1079 50  0000 L CNN
+F 2 "Mounting_Holes:MountingHole_2.2mm_M2_Pad" H 900 1050 50  0001 C CNN
+F 3 "" H 900 1050 50  0001 C CNN
+	1    700  1050
+	1    0    0    -1
+$EndComp
+NoConn ~ 700  1050
+NoConn ~ 700  700
 $EndSCHEMATC

Commit message: fix pwr/gnd swap, fix extra clock signal name, fix pin hole sizes
Connections:
- net +3V3: now also P10.5 (P5), P12.5 (P5), P14.5 (P5), P16.5 (P5), P2.5 (P5), P4.5 (P5), P6.5 (P5), P8.5 (P5)
- net +5V: now also P10.7 (P7), P12.7 (P7), P14.7 (P7), P16.7 (P7), P2.7 (P7), P4.7 (P7), P6.7 (P7), P8.7 (P7); no longer P10.8 (P8), P12.8 (P8), P14.8 (P8), P16.8 (P8), P2.8 (P8), P4.8 (P8), P6.8 (P8), P8.8 (P8)
- net CLK: no longer P10.6 (P6), P12.6 (P6), P14.6 (P6), P16.6 (P6), P2.6 (P6), P4.6 (P6), P6.6 (P6), P8.6 (P6)
- net GND: now also P10.8 (P8), P12.8 (P8), P14.8 (P8), P16.8 (P8), P2.8 (P8), P4.8 (P8), P6.8 (P8), P8.8 (P8); no longer P10.7 (P7), P12.7 (P7), P14.7 (P7), P16.7 (P7), P2.7 (P7), P4.7 (P7), P6.7 (P7), P8.7 (P7)
- net SCK: now also P10.6 (P6), P12.6 (P6), P14.6 (P6), P16.6 (P6), P2.6 (P6), P4.6 (P6), P6.6 (P6), P8.6 (P6); no longer P10.5 (P5), P12.5 (P5), P14.5 (P5), P16.5 (P5), P2.5 (P5), P4.5 (P5), P6.5 (P5), P8.5 (P5)
