File: KiCAD/ald_solenoidControl/ald_solenoidControl.sch (KiCad schematic (older format))
At the start: 36 parts, among them J1 Conn_01x14, J2 Conn_02x06_Odd_Even, J3 Conn_02x06_Odd_Even, J4 Conn_01x14, U1 ASSR-1611, U10 ASSR-1611, U11 ASSR-1611, U12 ASSR-1611, U13 ASSR-1611, U14 ASSR-1611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

Commit message: make spring pin board pin holders smaller, update base1x, update mux design controller board
Parts:
- added RN1, RN2, RN3, RN4: R_Pack04, SMD_Packages:DIP-8_SMD, symbol R_Pack04
- R1: value 830K -> R; footprint Resistors_SMD:R_2010_HandSoldering -> Resistors_SMD:R_1206
Connections:
- net labels added: V_D_EN_L
- net labels removed: PRE_GND
- wire segments 140 -> 179
Other:
- moved on the sheet: U1, U10, U11, U12, U13, U14, U15, U16, U17, U18, U19, U2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
