File: KiCAD/springPins28x28NoWindow/springPins28x28NoWindow.kicad_pcb (KiCad board)
At the start: 2 copper layers, 28 x 28 mm, 23 parts, among them J1 CONN_02X06, J2 CONN_02X06

Commit message: new 28x28 spring pin board done
Parts:
- removed 100k1: R, Resistors_SMD:R_0805_HandSoldering
- added G***: value, myParts:logo_small, B.Cu at (14.0, -14.0)
- added G***: value, myParts:logo_small, F.Cu at (14.0, -14.0)
- added R1: 100k, Resistors_SMD:R_0805_HandSoldering, B.Cu at (8.65, -4.00)
- J1, J2: moved to B.Cu
- moved J1 14.6 mm to (7.65, -7.65)
- moved J2 14.4 mm to (17.8, -7.65)
- moved TP10 1.80 mm to (12.5, -2.00)
- moved TP11 1.12 mm to (15.5, -26.0)
- moved TP12 1.12 mm to (15.5, -2.00)
- moved TP9 1.12 mm to (12.5, -26.0)
Connections:
- J1 pad 1: T_I -> Net-(J1-Pad1)
- J1 pad 10: 2_V -> 8_V
- J1 pad 11: Net-(100k1-Pad2) -> T_I
- J1 pad 12: Net-(100k1-Pad1) -> T_V
- J1 pad 2: T_V -> Net-(J1-Pad2)
- J1 pad 3: 8_I -> 2_I
- J1 pad 4: 8_V -> 2_V
- J1 pad 5: 6_I -> 4_I
- J1 pad 6: 6_V -> 4_V
- J1 pad 7: 4_I -> 6_I
- J1 pad 8: 4_V -> 6_V
- J1 pad 9: 2_I -> 8_I
- J2 pad 1: Net-(J2-Pad1) -> B_V
- J2 pad 10: 1_I -> 7_I
- J2 pad 11: B_V -> BOT_CU
- J2 pad 12: B_I -> TOP_CU
- J2 pad 2: Net-(J2-Pad2) -> B_I
- J2 pad 3: 7_V -> 1_V
- J2 pad 4: 7_I -> 1_I
- J2 pad 5: 5_V -> 3_V
- J2 pad 6: 5_I -> 3_I
- J2 pad 7: 3_V -> 5_V
- J2 pad 8: 3_I -> 5_I
- J2 pad 9: 1_V -> 7_V
Routing:
- net 7_V: track 0.00 -> 12.6 mm
- net B_I: track 0.00 -> 11.5 mm
- net T_I: track 0.00 -> 11.4 mm
- net 2_I: track 0.00 -> 11.4 mm
- net 1_I: track 0.00 -> 11.4 mm
- net 4_V: track 0.00 -> 10.7 mm
- net 8_I: track 0.00 -> 10.5 mm
- net 2_V: track 0.00 -> 10.3 mm
- net 8_V: track 0.00 -> 10.3 mm
- net 1_V: track 0.00 -> 10.3 mm
- net 5_V: track 0.00 -> 9.74 mm
- net 3_V: track 0.00 -> 9.43 mm
- net 6_V: track 0.00 -> 8.82 mm
- net 7_I: track 0.00 -> 7.80 mm
- net B_V: track 0.00 -> 7.25 mm
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- added copper zone on B.Cu, net BOT_CU
- added copper zone on F.Cu, net TOP_CU
Other:
- board text added: "+"
- board text added: "1I"
- board text added: "1V"
- board text added: "2I"
- board text added: "2V"
- board text added: "3I"
- board text added: "3V"
- board text added: "4V"
- board text added: "5I"
- board text added: "5V"
- board text added: "6"
- board text added: "6I"
- board text added: "6V"
- board text added: "7"
- board text added: "7I"
- board text added: "7V"
- board text added: "8"
- board text added: "8I"
- board text added: "8V"
- board text added: "BCu"
- board text added: "BI"
- board text added: "BV"
- board text added: "RA"
- board text added: "RB"
- board text added: "TCu"
- board text added: "TI"
- board text added: "TV"
- board text added: "°"
- board text removed: "0"

Commit message: nowindow pin boards done
Parts:
- removed the G*** at (14.0, -14.0) (x2)
- added G***: value, myParts:logo_small, B.Cu at (0.00, 0.00)
- added G***: value, myParts:logo_small, F.Cu at (0.00, 0.00)
- moved TP8 22.0 mm to (-12.0, 12.0)
- moved J1 19.8 mm to (-6.35, 6.35)
- moved R1 19.8 mm to (-5.35, 10.0)
- moved TP1 19.8 mm to (-12.0, -12.0)
- moved TP10 19.8 mm to (-1.50, 12.0)
- moved TP11 19.8 mm to (1.50, -12.0)
- moved TP12 19.8 mm to (1.50, 12.0)
- moved TP13 19.8 mm to (12.0, -12.0)
- moved TP14 19.8 mm to (12.0, -9.00)
- moved TP15 19.8 mm to (12.0, -5.00)
- moved TP16 19.8 mm to (12.0, -2.00)
- moved TP17 19.8 mm to (12.0, 2.00)
- moved TP18 19.8 mm to (12.0, 5.00)
- moved TP19 19.8 mm to (12.0, 9.00)
- moved TP2 19.8 mm to (-12.0, -9.00)
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Connections:
- net 2_I renamed /V2
- net 3_I renamed /I3
- net 7_V renamed /V7
- J1 pad 1: Net-(J1-Pad1) -> /I2
- J1 pad 10: 8_V -> /V8
- J1 pad 11: T_I -> /V6
- J1 pad 12: T_V -> /I8
- J1 pad 2: Net-(J1-Pad2) -> /RH
- J1 pad 4: 2_V -> /RL
- J1 pad 5: 4_I -> /I4
- J1 pad 6: 4_V -> /VT
- J1 pad 7: 6_I -> /V4
- J1 pad 8: 6_V -> /IT
- J1 pad 9: 8_I -> /I6
- J2 pad 1: B_V -> FCu
- J2 pad 10: 7_I -> /I5
- J2 pad 11: BOT_CU -> /I7
- J2 pad 12: TOP_CU -> /V5
- J2 pad 2: B_I -> /I1
- J2 pad 3: 1_V -> BCu
- J2 pad 4: 1_I -> /V1
- J2 pad 5: 3_V -> /VB
- J2 pad 7: 5_V -> /IB
- J2 pad 8: 5_I -> /V3
- R1 pad 1: Net-(J1-Pad2) -> /RL
- R1 pad 2: Net-(J1-Pad1) -> /RH
- TP1 pad 1: 8_I -> /V8
- TP10 pad 1: B_I -> /IB
- TP11 pad 1: T_I -> /VT
- TP12 pad 1: B_V -> /VB
- TP14 pad 1: 7_I -> /I7
- TP15 pad 1: 5_V -> /V5
- TP16 pad 1: 5_I -> /I5
- TP17 pad 1: 3_V -> /V3
- TP19 pad 1: 1_V -> /V1
- TP2 pad 1: 8_V -> /I8
- TP20 pad 1: 1_I -> /I1
- TP3 pad 1: 6_I -> /V6
- TP4 pad 1: 6_V -> /I6
- TP5 pad 1: 4_I -> /V4
- TP6 pad 1: 4_V -> /I4
- TP8 pad 1: 2_V -> /I2
- TP9 pad 1: T_V -> /IT
Routing:
- net /V8: track 0.00 -> 17.3 mm
- net /VT: track 0.00 -> 15.5 mm
- net /IB: track 0.00 -> 15.5 mm
- net /IT: track 0.00 -> 12.6 mm
- net /VB: track 0.00 -> 11.7 mm
- net B_I: track 11.5 -> 0.00 mm
- net T_I: track 11.4 -> 0.00 mm
- net 1_I: track 11.4 -> 0.00 mm
- net 4_V: track 10.7 -> 0.00 mm
- net 8_I: track 10.5 -> 0.00 mm
- net 2_V: track 10.3 -> 0.00 mm
- net 8_V: track 10.3 -> 0.00 mm
- net 1_V: track 10.3 -> 0.00 mm
- net 5_V: track 9.74 -> 0.00 mm
- net 3_V: track 9.43 -> 0.00 mm
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- added copper zone on B.Cu, net BCu
- added copper zone on F.Cu, net FCu
- removed copper zone on B.Cu, net BOT_CU
- removed copper zone on F.Cu, net TOP_CU
Other:
- board text added: "4I"
- board text added: "FCu"
- board text added: "RH"
- board text added: "RL"
- board text removed: "RA"
- board text removed: "RB"
- board text removed: "TCu"

Commit message: update silk
Other:
- board text added: "e90ef44"
- board text removed: "efbba54"
Changed lines of the file:
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@@
 (kicad_pcb (version 4) (host pcbnew 4.0.6)
   (general
-    (links 0)
-    (no_connects 2)
-    (area -14.075001 -14.075001 14.075001 14.075001)
+    (links 22)
+    (no_connects 0)
+    (area -14.075001 -14.075001 14.075001 14.806)
     (thickness 1.6)
     (drawings 76)
@@
   )
   (setup
-    (last_trace_width 0.56)
+    (last_trace_width 0.25)
     (user_trace_width 0.2)
     (user_trace_width 0.56)
@@
     (effects (font (size 1 1) (thickness 0.25)) (justify mirror))
   )
-  (gr_text efbba54 (at 6.5 -12.5) (layer B.SilkS)
+  (gr_text e90ef44 (at 6.5 -12.5) (layer B.SilkS)
     (effects (font (size 0.7 0.7) (thickness 0.175)) (justify mirror))
   )
@@
     (effects (font (size 1 1) (thickness 0.25)))
   )
-  (gr_text efbba54 (at 6.5 -12.5) (layer F.SilkS)
+  (gr_text e90ef44 (at 6.5 -12.5) (layer F.SilkS)
     (effects (font (size 0.7 0.7) (thickness 0.175)))
   )

Commit message: spruce up 28x28NoWindow
Parts:
- removed the G*** at (0.00, 0.00)
- added L1: GREY@CHRISTOFORO.NET, myParts:logo_small, F.Cu at (0.00, 0.00)
Changed lines of the file:
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@@
-(kicad_pcb (version 4) (host pcbnew 4.0.6)
+(kicad_pcb (version 4) (host pcbnew 4.0.7)
   (general
     (links 22)
     (no_connects 0)
-    (area -14.075001 -14.075001 14.075001 14.806)
+    (area -14.075001 -14.075001 14.075001 14.075001)
     (thickness 1.6)
     (drawings 76)
@@
     (add_net /VB)
     (add_net /VT)
-    (add_net BCu)
-    (add_net FCu)
   )
   (module myParts:logo_small (layer B.Cu)
@@
   (module myParts:logo_small (layer F.Cu)
     (at 0 0 90)
-    (fp_text reference G*** (at 0 -4 90) (layer F.SilkS) hide
+    (fp_text reference L1 (at 0 -4 90) (layer F.SilkS) hide
       (effects (font (thickness 0.2)))
     )
-    (fp_text value value (at 0 4 90) (layer F.SilkS) hide
+    (fp_text value GREY@CHRISTOFORO.NET (at 0 4 90) (layer F.SilkS) hide
       (effects (font (thickness 0.2)))
     )

Commit message: 28x28noWindow new silk and order.zip
Other:
- board text added: "2ffcf70"
- board text removed: "e90ef44"
Changed lines of the file:
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@@
     (area -14.075001 -14.075001 14.075001 14.075001)
     (thickness 1.6)
-    (drawings 76)
+    (drawings 75)
     (tracks 56)
     (zones 0)
@@
     (add_net /VB)
     (add_net /VT)
+    (add_net BCu)
+    (add_net FCu)
   )
   (module myParts:logo_small (layer B.Cu)
@@
     (effects (font (size 1 1) (thickness 0.25)) (justify mirror))
   )
-  (gr_text e90ef44 (at 6.5 -12.5) (layer B.SilkS)
-    (effects (font (size 0.7 0.7) (thickness 0.175)) (justify mirror))
-  )
   (gr_text 6 (at -10.5 -3.5 270) (layer F.SilkS)
     (effects (font (size 1 1) (thickness 0.25)))
@@
     (effects (font (size 1 1) (thickness 0.25)))
   )
-  (gr_text e90ef44 (at 6.5 -12.5) (layer F.SilkS)
+  (gr_text 2ffcf70 (at 6.5 -12.5) (layer F.SilkS)
     (effects (font (size 0.7 0.7) (thickness 0.175)))
   )

Commit message: update silk
Other:
- board text added: "1ad7c5f"
- board text removed: "2ffcf70"
Changed lines of the file:
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@@
     (effects (font (size 1 1) (thickness 0.25)))
   )
-  (gr_text 2ffcf70 (at 6.5 -12.5) (layer F.SilkS)
+  (gr_text 1ad7c5f (at 6.5 -12.5) (layer F.SilkS)
     (effects (font (size 0.7 0.7) (thickness 0.175)))
   )

Commit message: make spring pin board pin holders smaller, update base1x, update mux design controller board
Parts:
- added JP1: Jumper_NC_Small, Connectors:GS2, B.Cu at (3.81, 9.78)
Connections:
- J2 pad 1: FCu -> /FCu
- J2 pad 3: BCu -> /BCu
Routing:
- net /FCu: track 0.00 -> 2.79 mm
- added copper zone on B.Cu, net /BCu
- added copper zone on F.Cu, net /FCu
- removed copper zone on B.Cu, net BCu
- removed copper zone on F.Cu, net FCu
