File: KiCAD/controller/controller.kicad_pcb (KiCad board)
At the start: 4 copper layers, 45.1 x 110 mm, 38 parts, among them CON1 AVR-JTAG-10, J1 Conn_02x05_Counter_Clockwise, J2 Conn_01x17, J3 Screw_Terminal_01x02, J4 Conn_01x17, J5 Conn_02x03_Odd_Even, J6 Conn_02x03_Odd_Even, SW1 SW_Grayhill_94H_Coded, SW2 SW_Grayhill_94H_Coded, SW3 SW_Push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

Commit message: update silk
Other:
- board text added: "c75b306"
- board text removed: "deadbeef"
Changed lines of the file:
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@@
     (visible_elements FFFFFF7F)
     (pcbplotparams
-      (layerselection 0x010fc_80000001)
+      (layerselection 0x010fc_ffffffff)
       (usegerberextensions false)
       (usegerberattributes true)
@@
     (tags "test point SMD S1751-46R")
     (attr virtual)
-    (fp_text reference TP1 (at 0 -2.8 90) (layer F.SilkS)
+    (fp_text reference TP1 (at 3.212 -0.188 180) (layer F.SilkS)
       (effects (font (size 1 1) (thickness 0.15)))
     )
@@
     )
   )
-  (gr_text deadbeef (at 19.05 -48.26) (layer F.SilkS)
+  (gr_text c75b306 (at 19.05 -48.26) (layer F.SilkS)
     (effects (font (size 1 1) (thickness 0.25)))
   )
