File: KiCAD/ald_solenoidControl/moreEfficientCircuits/ALD_solenoidDriverCircuit_rev0.kicad_pcb (KiCad board)
At the start: 2 copper layers, 135 x 110 mm, 37 parts

Commit message: small fixes for disconnects
Parts:
- R1, R2: footprint Resistors_THT:R_Axial_DIN0309_L9.0mm_D3.2mm_P12.70mm_Horizontal -> Resistors_SMD:R_2010_HandSoldering
- mountingHole2, mountingHole4, mountingHole_1, mountingHole_3: footprint ALD_custom:3mmDrillHole -> Mounting_Holes:MountingHole_3mm_Pad
- moved R2 5.87 mm to (179.0, 123.2)
- moved R1 5.85 mm to (185.0, 123.2)
Connections:
- arduino_RHS_1 pad 10: Net-(arduino_RHS_1-Pad10) -> (no net)
- arduino_RHS_1 pad 11: Net-(arduino_RHS_1-Pad11) -> (no net)
- arduino_RHS_1 pad 13: Net-(arduino_RHS_1-Pad13) -> (no net)
- arduino_RHS_1 pad 2: Net-(arduino_RHS_1-Pad2) -> (no net)
- sol_stab_0 pad 1: Net-(sol_stab_0-Pad1) -> (no net)
- sol_stab_0 pad 2: Net-(sol_stab_0-Pad2) -> (no net)
- sol_stab_0 pad 3: Net-(sol_stab_0-Pad3) -> (no net)
- sol_stab_0 pad 4: Net-(sol_stab_0-Pad4) -> (no net)
- sol_stab_1 pad 1: Net-(sol_stab_1-Pad1) -> (no net)
- sol_stab_1 pad 2: Net-(sol_stab_1-Pad2) -> (no net)
- sol_stab_1 pad 3: Net-(sol_stab_1-Pad3) -> (no net)
- sol_stab_1 pad 4: Net-(sol_stab_1-Pad4) -> (no net)
- sol_stab_10 pad 1: Net-(sol_stab_10-Pad1) -> (no net)
- sol_stab_10 pad 2: Net-(sol_stab_10-Pad2) -> (no net)
- sol_stab_10 pad 3: Net-(sol_stab_10-Pad3) -> (no net)
- sol_stab_10 pad 4: Net-(sol_stab_10-Pad4) -> (no net)
- sol_stab_11 pad 1: Net-(sol_stab_11-Pad1) -> (no net)
- sol_stab_11 pad 2: Net-(sol_stab_11-Pad2) -> (no net)
- sol_stab_11 pad 3: Net-(sol_stab_11-Pad3) -> (no net)
- sol_stab_11 pad 4: Net-(sol_stab_11-Pad4) -> (no net)
- sol_stab_2 pad 1: Net-(sol_stab_2-Pad1) -> (no net)
- sol_stab_2 pad 2: Net-(sol_stab_2-Pad2) -> (no net)
- sol_stab_2 pad 3: Net-(sol_stab_2-Pad3) -> (no net)
- sol_stab_2 pad 4: Net-(sol_stab_2-Pad4) -> (no net)
- sol_stab_3 pad 1: Net-(sol_stab_3-Pad1) -> (no net)
- sol_stab_3 pad 2: Net-(sol_stab_3-Pad2) -> (no net)
- sol_stab_3 pad 3: Net-(sol_stab_3-Pad3) -> (no net)
- sol_stab_3 pad 4: Net-(sol_stab_3-Pad4) -> (no net)
- sol_stab_4 pad 1: Net-(sol_stab_4-Pad1) -> (no net)
- sol_stab_4 pad 2: Net-(sol_stab_4-Pad2) -> (no net)
- sol_stab_4 pad 3: Net-(sol_stab_4-Pad3) -> (no net)
- sol_stab_4 pad 4: Net-(sol_stab_4-Pad4) -> (no net)
- sol_stab_5 pad 1: Net-(sol_stab_5-Pad1) -> (no net)
- sol_stab_5 pad 2: Net-(sol_stab_5-Pad2) -> (no net)
- sol_stab_5 pad 3: Net-(sol_stab_5-Pad3) -> (no net)
- sol_stab_5 pad 4: Net-(sol_stab_5-Pad4) -> (no net)
- sol_stab_6 pad 1: Net-(sol_stab_6-Pad1) -> (no net)
- sol_stab_6 pad 2: Net-(sol_stab_6-Pad2) -> (no net)
- sol_stab_6 pad 3: Net-(sol_stab_6-Pad3) -> (no net)
- sol_stab_6 pad 4: Net-(sol_stab_6-Pad4) -> (no net)
- sol_stab_7 pad 1: Net-(sol_stab_7-Pad1) -> (no net)
- sol_stab_7 pad 2: Net-(sol_stab_7-Pad2) -> (no net)
- sol_stab_7 pad 3: Net-(sol_stab_7-Pad3) -> (no net)
- sol_stab_7 pad 4: Net-(sol_stab_7-Pad4) -> (no net)
- sol_stab_8 pad 1: Net-(sol_stab_8-Pad1) -> (no net)
- sol_stab_8 pad 2: Net-(sol_stab_8-Pad2) -> (no net)
- sol_stab_8 pad 3: Net-(sol_stab_8-Pad3) -> (no net)
- sol_stab_8 pad 4: Net-(sol_stab_8-Pad4) -> (no net)
- sol_stab_9 pad 1: Net-(sol_stab_9-Pad1) -> (no net)
- sol_stab_9 pad 2: Net-(sol_stab_9-Pad2) -> (no net)
- sol_stab_9 pad 3: Net-(sol_stab_9-Pad3) -> (no net)
- sol_stab_9 pad 4: Net-(sol_stab_9-Pad4) -> (no net)
Routing:
- net pwr_GND: track 687.2 -> 0.00 mm
- net signal_GND: track 441.9 -> 0.00 mm, vias 1 -> 0
- net +24V: track 220.2 -> 142.7 mm
- net SDA: track 109.9 -> 82.5 mm, vias 1 -> 0
- net SCL: track 105.6 -> 80.8 mm, vias 1 -> 0
- net solenoid_9: track 129.2 -> 123.9 mm
- net solenoid_11: track 143.3 -> 138.7 mm
- net solenoid_10: track 131.7 -> 130.0 mm
- net +5V: track 79.4 -> 78.7 mm, vias 0 -> 2
- added copper zone on F.Cu, net pwr_GND
- added copper zone on B.Cu, net signal_GND

Commit message: add mounting holes to add in card, make zones, move current limiting resistor
Connections:
- sol_conn_0 pad 1: signal_GND -> pwr_GND
- sol_conn_0 pad 2: pwr_GND -> signal_GND
- sol_conn_1 pad 1: signal_GND -> pwr_GND
- sol_conn_1 pad 2: pwr_GND -> signal_GND
- sol_conn_10 pad 1: signal_GND -> pwr_GND
- sol_conn_10 pad 2: pwr_GND -> signal_GND
- sol_conn_11 pad 1: signal_GND -> pwr_GND
- sol_conn_11 pad 2: pwr_GND -> signal_GND
- sol_conn_2 pad 1: signal_GND -> pwr_GND
- sol_conn_2 pad 2: pwr_GND -> signal_GND
- sol_conn_3 pad 1: signal_GND -> pwr_GND
- sol_conn_3 pad 2: pwr_GND -> signal_GND
- sol_conn_4 pad 1: signal_GND -> pwr_GND
- sol_conn_4 pad 2: pwr_GND -> signal_GND
- sol_conn_5 pad 1: signal_GND -> pwr_GND
- sol_conn_5 pad 2: pwr_GND -> signal_GND
- sol_conn_6 pad 1: signal_GND -> pwr_GND
- sol_conn_6 pad 2: pwr_GND -> signal_GND
- sol_conn_7 pad 1: signal_GND -> pwr_GND
- sol_conn_7 pad 2: pwr_GND -> signal_GND
- sol_conn_8 pad 1: signal_GND -> pwr_GND
- sol_conn_8 pad 2: pwr_GND -> signal_GND
- sol_conn_9 pad 1: signal_GND -> pwr_GND
- sol_conn_9 pad 2: pwr_GND -> signal_GND
Changed lines of the file:
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@@
   (general
     (links 75)
-    (no_connects 0)
-    (area 83.823809 45.449999 221.176191 155.575)
+    (no_connects 12)
+    (area 84.949999 45.449999 220.050001 155.550001)
     (thickness 1.6)
     (drawings 10)
@@
   )
   (setup
-    (last_trace_width 2)
+    (last_trace_width 0.25)
     (user_trace_width 0.25)
     (user_trace_width 0.5)
@@
     )
     (pad 1 thru_hole rect (at 0 0) (size 1.7 1.7) (drill 1) (layers *.Cu *.Mask)
-      (net 29 signal_GND))
-    (pad 2 thru_hole oval (at 0 2.54) (size 1.7 1.7) (drill 1) (layers *.Cu *.Mask)
-      (net 31 pwr_GND))
+      (net 31 pwr_GND))
+    (pad 2 thru_hole oval (at 0 2.54) (size 1.7 1.7) (drill 1) (layers *.Cu *.Mask)
+      (net 29 signal_GND))
     (pad 3 thru_hole oval (at 0 5.08) (size 1.7 1.7) (drill 1) (layers *.Cu *.Mask)
       (net 8 solenoid_0))
@@
     )
     (pad 1 thru_hole rect (at 0 0) (size 1.7 1.7) (drill 1) (layers *.Cu *.Mask)
-      (net 29 signal_GND))
-    (pad 2 thru_hole oval (at 0 2.54) (size 1.7 1.7) (drill 1) (layers *.Cu *.Mask)
-      (net 31 pwr_GND))
+      (net 31 pwr_GND))
+    (pad 2 thru_hole oval (at 0 2.54) (size 1.7 1.7) (drill 1) (layers *.Cu *.Mask)
+      (net 29 signal_GND))
     (pad 3 thru_hole oval (at 0 5.08) (size 1.7 1.7) (drill 1) (layers *.Cu *.Mask)
       (net 9 solenoid_1))
@@
     )
     (pad 1 thru_hole rect (at 0 0) (size 1.7 1.7) (drill 1) (layers *.Cu *.Mask)
-      (net 29 signal_GND))
-    (pad 2 thru_hole oval (at 0 2.54) (size 1.7 1.7) (drill 1) (layers *.Cu *.Mask)
-      (net 31 pwr_GND))
+      (net 31 pwr_GND))
+    (pad 2 thru_hole oval (at 0 2.54) (size 1.7 1.7) (drill 1) (layers *.Cu *.Mask)
+      (net 29 signal_GND))
     (pad 3 thru_hole oval (at 0 5.08) (size 1.7 1.7) (drill 1) (layers *.Cu *.Mask)
       (net 10 solenoid_2))
@@
     )
     (pad 1 thru_hole rect (at 0 0) (size 1.7 1.7) (drill 1) (layers *.Cu *.Mask)
-      (net 29 signal_GND))
-    (pad 2 thru_hole oval (at 0 2.54) (size 1.7 1.7) (drill 1) (layers *.Cu *.Mask)
-      (net 31 pwr_GND))
+      (net 31 pwr_GND))
+    (pad 2 thru_hole oval (at 0 2.54) (size 1.7 1.7) (drill 1) (layers *.Cu *.Mask)
+      (net 29 signal_GND))
     (pad 3 thru_hole oval (at 0 5.08) (size 1.7 1.7) (drill 1) (layers *.Cu *.Mask)
       (net 11 solenoid_3))
@@
     )
     (pad 1 thru_hole rect (at 0 0) (size 1.7 1.7) (drill 1) (layers *.Cu *.Mask)
-      (net 29 signal_GND))
-    (pad 2 thru_hole oval (at 0 2.54) (size 1.7 1.7) (drill 1) (layers *.Cu *.Mask)
-      (net 31 pwr_GND))
+      (net 31 pwr_GND))
+    (pad 2 thru_hole oval (at 0 2.54) (size 1.7 1.7) (drill 1) (layers *.Cu *.Mask)
+      (net 29 signal_GND))
     (pad 3 thru_hole oval (at 0 5.08) (size 1.7 1.7) (drill 1) (layers *.Cu *.Mask)
       (net 12 solenoid_4))
@@
     )
     (pad 1 thru_hole rect (at 0 0) (size 1.7 1.7) (drill 1) (layers *.Cu *.Mask)
-      (net 29 signal_GND))
-    (pad 2 thru_hole oval (at 0 2.54) (size 1.7 1.7) (drill 1) (layers *.Cu *.Mask)
-      (net 31 pwr_GND))
+      (net 31 pwr_GND))
+    (pad 2 thru_hole oval (at 0 2.54) (size 1.7 1.7) (drill 1) (layers *.Cu *.Mask)
+      (net 29 signal_GND))
     (pad 3 thru_hole oval (at 0 5.08) (size 1.7 1.7) (drill 1) (layers *.Cu *.Mask)
       (net 13 solenoid_5))
@@
     )
     (pad 1 thru_hole rect (at 0 0) (size 1.7 1.7) (drill 1) (layers *.Cu *.Mask)
-      (net 29 signal_GND))
-    (pad 2 thru_hole oval (at 0 2.54) (size 1.7 1.7) (drill 1) (layers *.Cu *.Mask)
-      (net 31 pwr_GND))
+      (net 31 pwr_GND))
+    (pad 2 thru_hole oval (at 0 2.54) (size 1.7 1.7) (drill 1) (layers *.Cu *.Mask)
+      (net 29 signal_GND))
     (pad 3 thru_hole oval (at 0 5.08) (size 1.7 1.7) (drill 1) (layers *.Cu *.Mask)
       (net 14 solenoid_6))
@@
     )
     (pad 1 thru_hole rect (at 0 0) (size 1.7 1.7) (drill 1) (layers *.Cu *.Mask)
-      (net 29 signal_GND))
-    (pad 2 thru_hole oval (at 0 2.54) (size 1.7 1.7) (drill 1) (layers *.Cu *.Mask)
-      (net 31 pwr_GND))
+      (net 31 pwr_GND))
+    (pad 2 thru_hole oval (at 0 2.54) (size 1.7 1.7) (drill 1) (layers *.Cu *.Mask)
+      (net 29 signal_GND))
     (pad 3 thru_hole oval (at 0 5.08) (size 1.7 1.7) (drill 1) (layers *.Cu *.Mask)
       (net 15 solenoid_7))
@@
     )
     (pad 1 thru_hole rect (at 0 0) (size 1.7 1.7) (drill 1) (layers *.Cu *.Mask)
-      (net 29 signal_GND))
-    (pad 2 thru_hole oval (at 0 2.54) (size 1.7 1.7) (drill 1) (layers *.Cu *.Mask)
-      (net 31 pwr_GND))
+      (net 31 pwr_GND))
+    (pad 2 thru_hole oval (at 0 2.54) (size 1.7 1.7) (drill 1) (layers *.Cu *.Mask)
+      (net 29 signal_GND))
     (pad 3 thru_hole oval (at 0 5.08) (size 1.7 1.7) (drill 1) (layers *.Cu *.Mask)
       (net 16 solenoid_8))
@@
     )
     (pad 1 thru_hole rect (at 0 0) (size 1.7 1.7) (drill 1) (layers *.Cu *.Mask)
-      (net 29 signal_GND))
-    (pad 2 thru_hole oval (at 0 2.54) (size 1.7 1.7) (drill 1) (layers *.Cu *.Mask)
-      (net 31 pwr_GND))
+      (net 31 pwr_GND))
+    (pad 2 thru_hole oval (at 0 2.54) (size 1.7 1.7) (drill 1) (layers *.Cu *.Mask)
+      (net 29 signal_GND))
     (pad 3 thru_hole oval (at 0 5.08) (size 1.7 1.7) (drill 1) (layers *.Cu *.Mask)
       (net 19 solenoid_9))
@@
     )
     (pad 1 thru_hole rect (at 0 0) (size 1.7 1.7) (drill 1) (layers *.Cu *.Mask)
-      (net 29 signal_GND))
-    (pad 2 thru_hole oval (at 0 2.54) (size 1.7 1.7) (drill 1) (layers *.Cu *.Mask)
-      (net 31 pwr_GND))
+      (net 31 pwr_GND))
+    (pad 2 thru_hole oval (at 0 2.54) (size 1.7 1.7) (drill 1) (layers *.Cu *.Mask)
+      (net 29 signal_GND))
     (pad 3 thru_hole oval (at 0 5.08) (size 1.7 1.7) (drill 1) (layers *.Cu *.Mask)
       (net 20 solenoid_10))
@@
     )
     (pad 1 thru_hole rect (at 0 0) (size 1.7 1.7) (drill 1) (layers *.Cu *.Mask)
-      (net 29 signal_GND))
-    (pad 2 thru_hole oval (at 0 2.54) (size 1.7 1.7) (drill 1) (layers *.Cu *.Mask)
-      (net 31 pwr_GND))
+      (net 31 pwr_GND))
+    (pad 2 thru_hole oval (at 0 2.54) (size 1.7 1.7) (drill 1) (layers *.Cu *.Mask)
+      (net 29 signal_GND))
     (pad 3 thru_hole oval (at 0 5.08) (size 1.7 1.7) (drill 1) (layers *.Cu *.Mask)
       (net 21 solenoid_11))

Commit message: random mods
Other:
- board text added: "Augustin Zaininger 022ff63"
- board text removed: "Augustin Zaininger 05/02/2018"
Changed lines of the file:
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@@
   (general
     (links 75)
-    (no_connects 12)
-    (area 84.949999 45.449999 220.050001 155.550001)
+    (no_connects 0)
+    (area 83.823809 45.449999 221.176191 155.575)
     (thickness 1.6)
     (drawings 10)
@@
     (effects (font (size 2 2) (thickness 0.4)))
   )
-  (gr_text "Augustin Zaininger 05/02/2018" (at 115.5 77) (layer F.SilkS)
+  (gr_text "Augustin Zaininger 022ff63" (at 115.5 77) (layer F.SilkS)
     (effects (font (size 2 2) (thickness 0.4)))
   )
