File: KiCAD/base1x/base1x.kicad_pcb (KiCad board)
At the start: 4 copper layers, 40 x 88.9 mm, 36 parts, among them J1 Conn_01x14, J2 Conn_02x06_Odd_Even, J3 Conn_02x06_Odd_Even, J4 Conn_01x14, U1 ASSR-1611, U10 ASSR-1611, U11 ASSR-1611, U12 ASSR-1611, U13 ASSR-1611, U14 ASSR-1611, U15 ASSR-1611, U16 ASSR-1611, U17 ASSR-1611, U18 ASSR-1611, U19 ASSR-1611, U2 ASSR-1611, U20 ASSR-1611, U21 ASSR-1611, U22 MCP23S17, U3 ASSR-1611, U4 ASSR-1611, U5 ASSR-1611, U6 ASSR-1611, U7 ASSR-1611, U8 ASSR-1611, U9 ASSR-1611

Commit message: fixed up newMux so that parts don't collide
Parts:
- removed U1, U10, U11, U12, U13, U14, U15, U16, U17, U18, U19, U20, U21, U7, U8, U9: ASSR-1611, Housings_DIP:DIP-6_W7.62mm
- removed U22: MCP23S17, Housings_DIP:DIP-28_W7.62mm
- added CON1: AVR-JTAG-10, Connectors_Multicomp:Multicomp_MC9A12-1034_2x05x2.54mm_Straight, F.Cu at (216.5, -72.5)
- added J5: Screw_Terminal_01x02, Connectors_Phoenix:PhoenixContact_MC-GF_02x3.50mm_Angled_ThreadedFlange_MountHole, F.Cu at (42.5, -5.71)
- added J6: Conn_02x14_Counter_Clockwise, Socket_Strips:Socket_Strip_Straight_2x14_Pitch2.54mm, F.Cu at (23.5, -61.0)
- added J7: Screw_Terminal_01x04, Connectors_Phoenix:PhoenixContact_MC-GF_04x3.50mm_Angled_ThreadedFlange_MountHole, F.Cu at (57.1, -7.62)
- added MK1: Mounting_Hole_PAD, Mounting_Holes:MountingHole_4mm_Pad, F.Cu at (253.5, -85.5)
- added MK2: Mounting_Hole_PAD, Mounting_Holes:MountingHole_4mm_Pad, F.Cu at (273.2, -99.9)
- added MK3: Mounting_Hole_PAD, Mounting_Holes:MountingHole_4mm_Pad, F.Cu at (196.6, -50.0)
- added MK4: Mounting_Hole_PAD, Mounting_Holes:MountingHole_4mm_Pad, F.Cu at (236.3, -60.0)
- added RN1: 1k, Housings_DIP:DIP-16_W7.62mm, F.Cu at (29.8, -62.9)
- added RN2: 1k, Housings_DIP:DIP-16_W7.62mm, F.Cu at (198.1, -118.1)
- added SW1: SW_DIP_x04, Buttons_Switches_THT:SW_DIP_x4_W7.62mm_Piano, F.Cu at (48.9, -38.1)
- added SW2: SW_Grayhill_94H_Coded, myParts:Grayhill_94H, F.Cu at (48.9, -69.8)
- added SW3: SW_Grayhill_94H_Coded, myParts:Grayhill_94H, F.Cu at (33.0, -69.2)
- added SW4: SW_Push, Buttons_Switches_THT:SW_PUSH_6mm, F.Cu at (54.0, -74.9)
- added SW5: SW_DIP_x04, Buttons_Switches_THT:SW_DIP_x4_W7.62mm_Piano, F.Cu at (35.6, -30.5)
- C1: moved to F.Cu
- J1: value Conn_01x14 -> Conn_02x04_Counter_Clockwise; footprint Pin_Headers:Pin_Header_Straight_1x14_Pitch2.54mm -> Socket_Strips:Socket_Strip_Straight_2x04_Pitch2.54mm; moved to F.Cu
- J2: value Conn_02x06_Odd_Even -> Conn_01x17; footprint Socket_Strips:Socket_Strip_Straight_2x06_Pitch2.54mm -> Socket_Strips:Socket_Strip_Straight_1x17_Pitch2.54mm
- J3: value Conn_02x06_Odd_Even -> Conn_02x14_Counter_Clockwise; footprint Socket_Strips:Socket_Strip_Straight_2x06_Pitch2.54mm -> Socket_Strips:Socket_Strip_Straight_2x14_Pitch2.54mm
- J4: value Conn_01x14 -> Conn_01x17; footprint Pin_Headers:Pin_Header_Straight_1x14_Pitch2.54mm -> Socket_Strips:Socket_Strip_Straight_1x17_Pitch2.54mm; moved to F.Cu
- JP1, JP6: value Jumper_NC_Small -> Jumper_NO_Small; footprint Connect:GS2 -> Connectors:GS2; moved to F.Cu
- JP2: value Jumper_NC_Dual -> Jumper_NO_Small; footprint Connect:GS3 -> Connectors:GS2; moved to F.Cu
- JP3, JP4, JP5: footprint Connect:GS3 -> Connectors:GS3; moved to F.Cu
- R1: value 830K -> 10K; footprint Resistors_SMD:R_2010_HandSoldering -> Resistors_SMD:R_0805_HandSoldering
- R2: value 500K -> 10K; moved to F.Cu
- U2, U3: value ASSR-1611 -> 74LS249; footprint Housings_DIP:DIP-6_W7.62mm -> Housings_DIP:DIP-16_W7.62mm
- U4, U5: value ASSR-1611 -> KCSC02-123; footprint Housings_DIP:DIP-6_W7.62mm -> Displays_7-Segment:KCSC02-123
- U6: value ASSR-1611 -> MCP23S17; footprint Housings_DIP:DIP-6_W7.62mm -> Housings_DIP:DIP-28_W7.62mm
- moved JP1 255.0 mm to (274.5, -113.3), turned to 0 degrees
- moved U3 237.1 mm to (238.8, -116.8), turned to 0 degrees
- moved JP4 224.0 mm to (277.3, -87.5), turned to 0 degrees
- moved JP2 222.2 mm to (280.1, -113.3), turned to 0 degrees
- moved JP5 203.1 mm to (254.1, -62.0), turned to 0 degrees
- moved JP6 193.1 mm to (248.7, -72.6), turned to 0 degrees
- moved JP3 190.6 mm to (246.3, -59.4), turned to 0 degrees
- moved R2 164.0 mm to (181.6, -77.8), turned to 0 degrees
- moved J2 133.2 mm to (142.9, -117.5), turned to 0 degrees
- moved C1 129.4 mm to (176.3, -78.2)
- moved U6 126.7 mm to (95.2, -121.3), turned to 0 degrees
- moved R1 125.6 mm to (171.5, -77.7), turned to 0 degrees
- moved J4 117.4 mm to (164.1, -116.9), turned to 0 degrees
- moved U4 82.4 mm to (30.5, -83.2), turned to 0 degrees
- moved U5 81.9 mm to (47.0, -83.2), turned to 0 degrees
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Connections:
- J1 pad 1: +5V -> MISO
- J1 pad 2: +3V3 -> SCK
- J1 pad 3: V_D -> (no net)
- J1 pad 6: Net-(J1-Pad6) -> GND
- J1 pad 7: MISO -> MOSI
- J1 pad 8: MOSI -> +5V
- J2 pad 1: /I2 -> MOSI
- J2 pad 10: /V8 -> ~CS_LED_SW
- J2 pad 11: /V6 -> (no net)
- J2 pad 12: /I8 -> (no net)
- J2 pad 2: V_D -> (no net)
- J2 pad 3: /V2 -> (no net)
- J2 pad 4: GND -> (no net)
- J2 pad 5: /I4 -> RESET
- J2 pad 6: /VT -> GND
- J2 pad 7: /V4 -> SDA
- J2 pad 8: /IT -> SCL
- J2 pad 9: /I6 -> ~CS0
- J3 pad 1: GND -> +5V
- J3 pad 10: /I5 -> SCL
- J3 pad 11: /I7 -> ~CSL
- J3 pad 12: /V5 -> ~CS0
- J3 pad 2: /I1 -> +5V
- J3 pad 3: GND -> +3V3
- J3 pad 4: /V1 -> +3V3
- J3 pad 5: /VB -> ADC0
- J3 pad 6: /I3 -> ADC0
- J3 pad 7: /IB -> SDA
- J3 pad 8: /V3 -> SDA
- J3 pad 9: /V7 -> SCL
- J4 pad 1: +5V -> SCK
- J4 pad 10: I+ -> (no net)
- J4 pad 11: V+ -> TCK
- J4 pad 12: V- -> TMS
- J4 pad 13: I- -> TDO
- J4 pad 14: GND -> TDI
- J4 pad 2: +3V3 -> MISO
- J4 pad 3: V_D -> /Vin
- J4 pad 4: SDA -> GND
- J4 pad 5: SCL -> RESET
- J4 pad 6: Net-(J4-Pad6) -> +5V
- J4 pad 7: MISO -> (no net)
- J4 pad 8: MOSI -> (no net)
- J4 pad 9: SCK -> ADC0
- JP1 pad 1: ~CS -> ~CSL
- JP1 pad 2: Net-(J1-Pad6) -> ~CS0
- JP2 pad 2: A0 -> /Vin
- JP3 pad 2: A1 -> A0_SW
- JP4 pad 2: A2 -> A1_SW
- JP5 pad 2: ~CS -> A2_SW
- JP6 pad 1: Net-(J4-Pad6) -> ~CS0
- JP6 pad 2: ~CS -> ~CSR
- R1 pad 1: GND -> +5V
- R1 pad 2: /PRE_GND -> SDA
- R2 pad 1: Net-(R2-Pad1) -> +5V
- R2 pad 2: V_D -> SCL
- U2 pad 1: /P1 -> BCD_S_B
- U2 pad 2: /PRE_GND -> BCD_S_C
- U2 pad 3: (no net) -> +5V
- U2 pad 4: V+ -> (no net)
- U2 pad 5: (no net) -> +5V
- U2 pad 6: /V1 -> BCD_S_D
- U3 pad 1: /P2 -> BCD_P_B
- U3 pad 2: /PRE_GND -> BCD_P_C
- U3 pad 3: (no net) -> +5V
- U3 pad 4: V+ -> (no net)
- U3 pad 5: (no net) -> +5V
- U3 pad 6: /V2 -> BCD_P_D
- U4 pad 1: /P3 -> Net-(RN1-Pad5)
- U4 pad 2: /PRE_GND -> Net-(RN1-Pad4)
- U4 pad 3: (no net) -> GND
- U4 pad 4: V+ -> Net-(RN1-Pad3)
- U4 pad 5: (no net) -> Net-(RN1-Pad8)
- U4 pad 6: /V3 -> Net-(RN1-Pad2)
- U5 pad 1: /P4 -> Net-(RN2-Pad5)
- U5 pad 2: /PRE_GND -> Net-(RN2-Pad4)
- U5 pad 3: (no net) -> GND
- U5 pad 4: V+ -> Net-(RN2-Pad3)
- U5 pad 5: (no net) -> Net-(RN2-Pad8)
- U5 pad 6: /V4 -> Net-(RN2-Pad2)
- U6 pad 1: /P5 -> BCD_P_A
- U6 pad 2: /PRE_GND -> BCD_P_B
- U6 pad 3: (no net) -> BCD_P_C
- U6 pad 4: V+ -> BCD_P_D
- U6 pad 5: (no net) -> BCD_S_A
- U6 pad 6: /V5 -> BCD_S_B
Routing:
- net /PRE_GND: track 196.8 -> 0.00 mm, vias 1 -> 0
- net GND: track 132.5 -> 0.00 mm, vias 4 -> 0
- net /BOT: track 108.7 -> 0.00 mm
- net /P3: track 106.2 -> 0.00 mm
- net V+: track 105.6 -> 0.00 mm, vias 1 -> 0
- net /P5: track 103.0 -> 0.00 mm
- net /P4: track 101.8 -> 0.00 mm, vias 3 -> 0
- net /P8: track 87.8 -> 0.00 mm, vias 2 -> 0
- net /TOP: track 84.0 -> 0.00 mm, vias 3 -> 0
- net /P2: track 83.8 -> 0.00 mm, vias 1 -> 0
- net /V_D_EN: track 83.2 -> 0.00 mm
- net /P7: track 82.9 -> 0.00 mm, vias 1 -> 0
- net /P1: track 81.9 -> 0.00 mm
- net I+: track 80.4 -> 0.00 mm, vias 3 -> 0
- net SCK: track 78.4 -> 0.00 mm, vias 2 -> 0
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- removed copper zone on F.Cu, net +5V
- removed copper zone on B.Cu, net /PRE_GND
- removed copper zone on B.Cu, net GND
- removed copper zone on F.Cu, net I+
Other:
- net class Default: trace_width 0.4 -> 0.25
- board text removed: "ac10c1a"

Commit message: wip for base1x
Parts:
- removed J7: Screw_Terminal_01x04, Connectors_Phoenix:PhoenixContact_MC-GF_04x3.50mm_Angled_ThreadedFlange_MountHole
- removed MK3, MK4: Mounting_Hole_PAD, Mounting_Holes:MountingHole_4mm_Pad
- removed SW4: SW_Push, Buttons_Switches_THT:SW_PUSH_6mm
- removed SW5: SW_DIP_x04, Buttons_Switches_THT:SW_DIP_x4_W7.62mm_Piano
- J5: value Screw_Terminal_01x02 -> Screw_Terminal_01x06; footprint Connectors_Phoenix:PhoenixContact_MC-GF_02x3.50mm_Angled_ThreadedFlange_MountHole -> Connectors_Phoenix:PhoenixContact_MC-GF_06x3.50mm_Angled_ThreadedFlange_MountHole; moved to B.Cu
- MK1, MK2: footprint Mounting_Holes:MountingHole_4mm_Pad -> Mounting_Holes:MountingHole_2.2mm_M2_Pad
- SW1: value SW_DIP_x04 -> SW_Grayhill_94H_Coded; footprint Buttons_Switches_THT:SW_DIP_x4_W7.62mm_Piano -> myParts:Grayhill_94H
- SW3: value SW_Grayhill_94H_Coded -> SW_Push; footprint myParts:Grayhill_94H -> Buttons_Switches_THT:SW_PUSH_6mm
- moved MK2 290.6 mm to (-13.1, -50.0)
- moved MK1 243.1 mm to (13.1, -50.0)
- moved U4 221.5 mm to (226.4, -186.5)
- moved J1 220.2 mm to (165.2, -186.5)
- moved SW1 219.2 mm to (213.9, -182.4)
- moved RN1 214.8 mm to (192.6, -202.9)
- moved U5 197.1 mm to (222.8, -172.1)
- moved U2 195.3 mm to (182.5, -202.9)
- moved SW3 195.0 mm to (210.2, -150.7)
- moved SW2 147.5 mm to (176.9, -143.1)
- moved JP2 145.2 mm to (137.6, -141.3)
- moved JP6 135.3 mm to (132.1, -141.3)
- moved U3 104.2 mm to (145.5, -163.3)
- moved JP5 100.9 mm to (200.1, -147.3)
- moved JP1 97.7 mm to (228.4, -199.4)
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Connections:
- CON1 pad 7: (no net) -> Net-(CON1-Pad7)
- CON1 pad 8: (no net) -> Net-(CON1-Pad8)
- J1 pad 3: (no net) -> Net-(J1-Pad3)
- J2 pad 11: (no net) -> /6(**/A7)
- J2 pad 12: (no net) -> /7
- J2 pad 13: (no net) -> /8
- J2 pad 14: (no net) -> /9(**/A9)
- J2 pad 17: (no net) -> /12(A11)
- J2 pad 2: (no net) -> /SS
- J2 pad 3: (no net) -> /1(Tx1)
- J2 pad 4: (no net) -> /0(Rx1)
- J3 pad 19: Net-(J3-Pad19) -> GND
- J3 pad 20: I+ -> GND
- J3 pad 21: Net-(J3-Pad21) -> I+
- J3 pad 22: V+ -> I+
- J3 pad 23: Net-(J3-Pad23) -> V+
- J3 pad 24: V- -> V+
- J3 pad 25: Net-(J3-Pad25) -> V-
- J3 pad 26: I- -> V-
- J3 pad 27: GND -> I-
- J3 pad 28: GND -> I-
- J4 pad 10: (no net) -> /A4
- J4 pad 15: (no net) -> /AREF
- J4 pad 17: (no net) -> /13(**)
- J4 pad 7: (no net) -> /NC0
- J4 pad 8: (no net) -> /NC1
- J5 pad 1: /Vin -> I+
- J5 pad 2: GND -> V+
- J6 pad 19: I+ -> GND
- J6 pad 20: Net-(J6-Pad20) -> GND
- J6 pad 21: V+ -> I+
- J6 pad 22: Net-(J6-Pad22) -> I+
- J6 pad 23: V- -> V+
- J6 pad 24: Net-(J6-Pad24) -> V+
- J6 pad 25: I- -> V-
- J6 pad 26: Net-(J6-Pad26) -> V-
- J6 pad 27: GND -> I-
- J6 pad 28: GND -> I-
- RN1 pad 9: (no net) -> Net-(RN1-Pad9)
- RN2 pad 9: (no net) -> Net-(RN2-Pad9)
- SW1 pad 1: I+ -> SWS1
- SW1 pad 2: V+ -> SWS2
- SW1 pad 4: I- -> SWS4
- SW1 pad 8: Net-(J3-Pad19) -> SWS8
- SW2 pad 1: SWS1 -> SWP1
- SW2 pad 2: SWS2 -> SWP2
- SW2 pad 4: SWS4 -> SWP4
- SW2 pad 8: SWS8 -> SWP8
- SW3 pad 1: SWP1 -> INT_BUT
- SW3 pad 2: SWP2 -> GND
- U2 pad 4: (no net) -> Net-(U2-Pad4)
- U3 pad 4: (no net) -> Net-(U3-Pad4)
- U6 pad 19: (no net) -> Net-(U6-Pad19)
Other:
- board size 40 x 88.9 mm -> 45.1 x 110 mm

Commit message: make spring pin board pin holders smaller, update base1x, update mux design controller board
Parts:
- removed CON1: AVR-JTAG-10, Connectors_Multicomp:Multicomp_MC9A12-1034_2x05x2.54mm_Straight
- removed JP1: Jumper_NO_Small, Connectors:GS2
- removed RN1, RN2: 1k, Housings_DIP:DIP-16_W7.62mm
- removed SW1, SW2: SW_Grayhill_94H_Coded, myParts:Grayhill_94H
- removed SW3: SW_Push, Buttons_Switches_THT:SW_PUSH_6mm
- removed U2, U3: 74LS249, Housings_DIP:DIP-16_W7.62mm
- removed U4, U5: KCSC02-123, Displays_7-Segment:KCSC02-123
- removed U6: MCP23S17, Housings_DIP:DIP-28_W7.62mm
- added D1: BPW21, myParts:BPW21, F.Cu at (28.0, -6.20)
- added D2: BPW21, myParts:BPW21, F.Cu at (28.0, 6.20)
- added J7: Conn_02x06_Counter_Clockwise, Socket_Strips:Socket_Strip_Straight_2x06_Pitch2.54mm, F.Cu at (-6.35, 6.35)
- added J8: Conn_02x06_Counter_Clockwise, Socket_Strips:Socket_Strip_Straight_2x06_Pitch2.54mm, F.Cu at (3.81, 6.35)
- added MK3: Mounting_Hole, Mounting_Holes:MountingHole_6mm, F.Cu at (33.8, -11.7)
- added MK4: Mounting_Hole, Mounting_Holes:MountingHole_6mm, F.Cu at (33.8, 12.8)
- added MK5: Mounting_Hole, Mounting_Holes:MountingHole_3.2mm_M3, F.Cu at (35.4, -40.6)
- added MK6: Mounting_Hole, Mounting_Holes:MountingHole_4.3mm_M4, F.Cu at (33.8, 0.56)
- added MK7: Mounting_Hole, Mounting_Holes:MountingHole_3.2mm_M3, F.Cu at (7.55, -30.1)
- added MK8: Mounting_Hole, Mounting_Holes:MountingHole_3.2mm_M3, F.Cu at (35.4, 19.4)
- added P1: CONN_01X02, Pin_Headers:Pin_Header_Straight_1x02_Pitch2.54mm, F.Cu at (33.0, -27.2)
- added P2: CONN_01X02, Pin_Headers:Pin_Header_Straight_1x02_Pitch2.54mm, F.Cu at (29.0, 24.8)
- added R3: 10K, Resistors_SMD:R_0805_HandSoldering, B.Cu at (26.2, -3.25)
- added R4: 10K, Resistors_SMD:R_0805_HandSoldering, B.Cu at (28.2, -4.00)
- added TP1: Test_Point, myParts:Test_Point_S1751-46R, F.Cu at (-20.0, 49.5)
- added TP2: Test_Point, myParts:Test_Point_S1751-46R, F.Cu at (25.0, -19.0)
- added U1: ADS1115, Housings_SSOP:MSOP-10_3x3mm_Pitch0.5mm, B.Cu at (25.8, -11.3)
- C1: value 0.1uF -> 1uF; footprint Capacitors_SMD:C_0603_HandSoldering -> Capacitors_SMD:C_0805_HandSoldering; moved to B.Cu
- J1: value Conn_02x04_Counter_Clockwise -> Conn_02x05_Odd_Even; footprint Socket_Strips:Socket_Strip_Straight_2x04_Pitch2.54mm -> Pin_Headers:Pin_Header_Angled_2x05_Pitch2.54mm
- J2: value Conn_01x17 -> GS3; footprint Socket_Strips:Socket_Strip_Straight_1x17_Pitch2.54mm -> Connectors:GS3
- J4: value Conn_01x17 -> GS3; footprint Socket_Strips:Socket_Strip_Straight_1x17_Pitch2.54mm -> Connectors:GS3; moved to B.Cu
- JP3, JP4, JP5: value Jumper_NC_Dual -> Jumper_NO_Small; footprint Connectors:GS3 -> Connectors:GS2
- R1, R2: value 10K -> 1.2K
- moved JP4 252.4 mm to (24.0, 0.50)
- moved JP6 229.5 mm to (-5.25, 42.5)
- moved JP5 225.6 mm to (34.9, 6.25), turned to 90 degrees
- moved J4 222.9 mm to (28.2, 1.00), turned to 90 degrees
- moved JP3 221.7 mm to (34.8, -6.00), turned to 90 degrees
- moved J1 220.1 mm to (-6.00, -48.3), turned to 90 degrees
- moved J2 214.9 mm to (0.25, -17.2), turned to 90 degrees
- moved C1 180.3 mm to (25.8, -17.3), turned to 90 degrees
- moved R2 176.9 mm to (31.0, -21.2), turned to 90 degrees
- moved R1 159.8 mm to (30.5, -35.2), turned to 90 degrees
- moved JP2 154.0 mm to (30.5, -30.8)
- moved L1 92.2 mm to (0.00, 46.0)
Connections:
- J1 pad 2: SCK -> +5V
- J1 pad 3: Net-(J1-Pad3) -> SCK
- J1 pad 4: SDA -> MOSI
- J1 pad 5: SCL -> V_D_EXT
- J1 pad 7: MOSI -> SDA
- J1 pad 8: +5V -> SCL
- J2 pad 1: MOSI -> V_D_EXT
- J2 pad 2: /SS -> V_D
- J2 pad 3: /1(Tx1) -> V_D_LOC
- J3 pad 11: ~CSL -> ~CS0
- J3 pad 12: ~CS0 -> /~CSL
- J3 pad 22: I+ -> /I+L
- J3 pad 24: V+ -> /V+L
- J3 pad 26: V- -> /V-L
- J3 pad 28: I- -> /I-L
- J3 pad 5: ADC0 -> V_D
- J3 pad 6: ADC0 -> V_D
- J4 pad 1: SCK -> GND
- J4 pad 2: MISO -> Net-(J4-Pad2)
- J4 pad 3: /Vin -> +5V
- J6 pad 11: ~CS0 -> /~CSR
- J6 pad 12: ~CSR -> ~CS0
- J6 pad 21: I+ -> /I+R
- J6 pad 23: V+ -> /V+R
- J6 pad 25: V- -> /V-R
- J6 pad 27: I- -> /I-R
- J6 pad 5: ADC0 -> V_D
- J6 pad 6: ADC0 -> V_D
- JP2 pad 1: +5V -> Net-(JP2-Pad1)
- JP2 pad 2: /Vin -> /ANODE_A
- JP3 pad 1: +5V -> /CATHODE_A
- JP3 pad 2: A0_SW -> GND
- JP4 pad 1: +5V -> Net-(JP4-Pad1)
- JP4 pad 2: A1_SW -> /ANODE_B
- JP5 pad 1: +5V -> /CATHODE_B
- JP5 pad 2: A2_SW -> GND
- JP6 pad 1: ~CS0 -> +5V
- JP6 pad 2: ~CSR -> /Vin
- R1 pad 1: +5V -> Net-(JP2-Pad1)
- R1 pad 2: SDA -> +5V
- R2 pad 1: +5V -> Net-(JP4-Pad1)
- R2 pad 2: SCL -> +5V
Routing:
- net /Vin: track 0.00 -> 118.6 mm, vias 0 -> 3
- net SCL: track 0.00 -> 104.1 mm, vias 0 -> 2
- net MOSI: track 0.00 -> 99.2 mm, vias 0 -> 1
- net SCK: track 0.00 -> 98.9 mm, vias 0 -> 1
- net SDA: track 0.00 -> 95.8 mm, vias 0 -> 1
- net MISO: track 0.00 -> 93.6 mm, vias 0 -> 1
- net ~CS0: track 0.00 -> 90.8 mm, vias 0 -> 2
- net I+: track 0.00 -> 77.6 mm, vias 0 -> 1
- net V+: track 0.00 -> 75.1 mm, vias 0 -> 1
- net V-: track 0.00 -> 72.5 mm, vias 0 -> 1
- net I-: track 0.00 -> 70.0 mm, vias 0 -> 1
- net V_D: track 0.00 -> 48.3 mm, vias 0 -> 2
- net +3V3: track 0.00 -> 42.5 mm
- net V_D_EXT: track 0.00 -> 31.1 mm
- net V_D_LOC: track 0.00 -> 29.8 mm, vias 0 -> 2
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- added copper zone on F.Cu, net +5V
- added copper zone on B.Cu, net GND
Other:
- board size 45.1 x 110 mm -> 62.2 x 110 mm
- board text added: "GND"

Commit message: update silk
Other:
- board text added: "c75b306"
Changed lines of the file:
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@@
   (general
     (thickness 1.6)
-    (drawings 26)
+    (drawings 27)
     (tracks 204)
     (zones 0)
@@
     (visible_elements FFFFFF7F)
     (pcbplotparams
-      (layerselection 0x010fc_80000001)
+      (layerselection 0x010fc_ffffffff)
       (usegerberextensions false)
       (usegerberattributes true)
@@
     (pad 1 np_thru_hole circle (at 0 0) (size 4.3 4.3) (drill 4.3) (layers *.Cu *.Mask))
   )
+  (gr_text c75b306 (at 14.5 43.75) (layer F.SilkS)
+    (effects (font (size 1 1) (thickness 0.25)))
+  )
   (gr_text GND (at -17 49.5 90) (layer F.SilkS)

Commit message: wip commit
Parts:
- removed J5: Screw_Terminal_01x06, Connectors_Phoenix:PhoenixContact_MC-GF_06x3.50mm_Angled_ThreadedFlange_MountHole
- added J9: Screw_Terminal_01x08, Connectors_Phoenix:PhoenixContact_MC-GF_08x3.50mm_Angled_ThreadedFlange_MountHole, B.Cu at (12.2, 49.1)
- added P3: CONN_01X02, Pin_Headers:Pin_Header_Straight_1x02_Pitch2.54mm, F.Cu at (23.0, 40.0)
- added P4: CONN_01X02, Pin_Headers:Pin_Header_Straight_1x02_Pitch2.54mm, F.Cu at (1.50, 42.5)
- added R5: 1, Resistors_SMD:R_2512_HandSoldering, F.Cu at (2.00, 32.0)
- added TP3: Test_Point, myParts:Test_Point_S1751-46R, F.Cu at (52.3, -4.40)
- added TP4: Test_Point, myParts:Test_Point_S1751-46R, F.Cu at (92.1, -16.3)
- added TP5: Test_Point, myParts:Test_Point_S1751-46R, F.Cu at (73.9, -11.7)
Connections:
- J3 pad 12: /~CSL -> (no net)
- J3 pad 22: /I+L -> (no net)
- J3 pad 24: /V+L -> (no net)
- J3 pad 26: /V-L -> (no net)
- J3 pad 28: /I-L -> (no net)
- J6 pad 11: /~CSR -> (no net)
- J6 pad 21: /I+R -> (no net)
- J6 pad 23: /V+R -> (no net)
- J6 pad 25: /V-R -> (no net)
- J6 pad 27: /I-R -> (no net)
- J7 pad 1: Net-(J7-Pad1) -> (no net)
- J7 pad 10: Net-(J7-Pad10) -> (no net)
- J7 pad 11: Net-(J7-Pad11) -> (no net)
- J7 pad 12: Net-(J7-Pad12) -> (no net)
- J7 pad 2: Net-(J7-Pad2) -> (no net)
- J7 pad 3: Net-(J7-Pad3) -> (no net)
- J7 pad 4: Net-(J7-Pad4) -> (no net)
- J7 pad 5: Net-(J7-Pad5) -> (no net)
- J7 pad 6: Net-(J7-Pad6) -> (no net)
- J7 pad 7: Net-(J7-Pad7) -> (no net)
- J7 pad 8: Net-(J7-Pad8) -> (no net)
- J7 pad 9: Net-(J7-Pad9) -> (no net)
- J8 pad 1: Net-(J8-Pad1) -> (no net)
- J8 pad 10: Net-(J8-Pad10) -> (no net)
- J8 pad 11: Net-(J8-Pad11) -> (no net)
- J8 pad 12: Net-(J8-Pad12) -> (no net)
- J8 pad 2: Net-(J8-Pad2) -> (no net)
- J8 pad 3: Net-(J8-Pad3) -> (no net)
- J8 pad 4: Net-(J8-Pad4) -> (no net)
- J8 pad 5: Net-(J8-Pad5) -> (no net)
- J8 pad 6: Net-(J8-Pad6) -> (no net)
- J8 pad 7: Net-(J8-Pad7) -> (no net)
- J8 pad 8: Net-(J8-Pad8) -> (no net)
- J8 pad 9: Net-(J8-Pad9) -> (no net)
- TP2 pad 1: Net-(TP2-Pad1) -> I-
- U1 pad 5: Net-(TP2-Pad1) -> I-
Routing:
- net I-: track 70.0 -> 85.3 mm, vias 1 -> 2
- net Net-(TP2-Pad1): track 15.3 -> 0.00 mm, vias 1 -> 0
