File: KiCAD/base1x/base1x.kicad_pcb (KiCad board)
At the start: 4 copper layers, 130 x 110 mm, 87 parts, among them J1 Conn_02x05_Odd_Even, J10 Conn_01x03, J11 Conn_01x03, J12 Conn_01x03, J13 Conn_01x03, J14 Conn_01x03, J15 Conn_01x08, J16 Conn_02x05_Odd_Even, J17 Conn_01x03, J18 Conn_01x03, J19 Conn_01x03, J2 Conn_01x03, J20 Conn_01x03, J3 Conn_02x14_Counter_Clockwise, J4 Conn_01x03, J5 Conn_01x03, J6 Conn_01x14_Counter_Clockwise, J7 Conn_02x06_Counter_Clockwise, J8 Conn_02x06_Counter_Clockwise, J9 Screw_Terminal_01x08, U1 AD8616, U2 ads122c04, U3 AD8615, U5 ads122c04, U8 LT1963EQ-2.5, U9 LT3015EQ-2.5

Commit message: update silk
Other:
- board text added: "8694043"
- board text removed: "20b2bb8"
Changed lines of the file:
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@@
   )
   (setup
-    (last_trace_width 2)
+    (last_trace_width 0.25)
     (user_trace_width 0.3)
     (user_trace_width 0.4)
@@
       (usegerberextensions true)
       (usegerberattributes true)
-      (usegerberadvancedattributes true)
+      (usegerberadvancedattributes false)
       (creategerberjobfile false)
       (excludeedgelayer true)
@@
       (plotinvisibletext false)
       (padsonsilk false)
-      (subtractmaskfromsilk false)
+      (subtractmaskfromsilk true)
       (outputformat 1)
       (mirror false)
@@
     (effects (font (size 1.5 1.5) (thickness 0.3)) (justify left))
   )
-  (gr_text 20b2bb8 (at 25.4 -16.51 270) (layer F.SilkS)
+  (gr_text 8694043 (at 25.4 -16.51 270) (layer F.SilkS)
     (effects (font (size 1.5 1.5) (thickness 0.3)))
   )
@@
   (gr_line (start -20 55) (end 104 55) (angle 90) (layer Edge.Cuts) (width 0.15))
   (gr_line (start -20 -55) (end 104 -55) (angle 90) (layer Edge.Cuts) (width 0.15))
-  (via (at 42.164 -40.64) (size 0.6) (drill 0.4) (layers F.Cu B.Cu) (net 25))
-  (via (at 46.99 -33.274) (size 0.6) (drill 0.4) (layers F.Cu B.Cu) (net 25))
-  (via (at 41.402 51.816) (size 0.6) (drill 0.4) (layers F.Cu B.Cu) (net 28))
-  (via (at 46.99 1.016) (size 0.6) (drill 0.4) (layers F.Cu B.Cu) (net 19))
-  (via (at 47.752 -12.192) (size 0.6) (drill 0.4) (layers F.Cu B.Cu) (net 18))
-  (via (at 46.736 -26.416) (size 0.6) (drill 0.4) (layers F.Cu B.Cu) (net 18))
-  (via (at 41.656 -22.86) (size 0.6) (drill 0.4) (layers F.Cu B.Cu) (net 18))
-  (via (at 42.4815 -15.367) (size 0.6) (drill 0.4) (layers F.Cu B.Cu) (net 18))
-  (via (at 39.3065 -15.4305) (size 0.6) (drill 0.4) (layers F.Cu B.Cu) (net 18))
-  (via (at 43.815 38.6715) (size 0.6) (drill 0.4) (layers F.Cu B.Cu) (net 5))
-  (via (at 37.719 15.5575) (size 0.6) (drill 0.4) (layers F.Cu B.Cu) (net 5))
-  (via (at 46.1645 47.879) (size 0.6) (drill 0.4) (layers F.Cu B.Cu) (net 19))
-  (via (at 45.72 41.3385) (size 0.6) (drill 0.4) (layers F.Cu B.Cu) (net 17))
-  (via (at 44.45 42.164) (size 0.6) (drill 0.4) (layers F.Cu B.Cu) (net 2))
-  (via (at 41.402 21.463) (size 0.6) (drill 0.4) (layers F.Cu B.Cu) (net 19))
-  (via (at 41.148 14.986) (size 0.6) (drill 0.4) (layers F.Cu B.Cu) (net 2))
-  (via (at 41.783 12.1285) (size 0.6) (drill 0.4) (layers F.Cu B.Cu) (net 17))
-  (via (at 41.91 -5.334) (size 0.6) (drill 0.4) (layers F.Cu B.Cu) (net 17))
-  (via (at 45.72 1.524) (size 0.6) (drill 0.4) (layers F.Cu B.Cu) (net 19))
-  (via (at 44.45 1.524) (size 0.6) (drill 0.4) (layers F.Cu B.Cu) (net 18))
-  (via (at 45.72 -5.08) (size 0.6) (drill 0.4) (layers F.Cu B.Cu) (net 18))
-  (via (at 45.72 -48.26) (size 0.6) (drill 0.4) (layers F.Cu B.Cu) (net 14))
-  (via (at 8.89 -41.275) (size 0.6) (drill 0.4) (layers F.Cu B.Cu) (net 14))
-  (via (at 12.4 -48.4) (size 0.6) (drill 0.4) (layers F.Cu B.Cu) (net 5))
-  (via (at 12.4 -51.4) (size 0.6) (drill 0.4) (layers F.Cu B.Cu) (net 5))
-  (via (at 37.25 42.75) (size 0.6) (drill 0.4) (layers F.Cu B.Cu) (net 18))
-  (via (at 40.25 42.75) (size 0.6) (drill 0.4) (layers F.Cu B.Cu) (net 18))
-  (via (at 24 50) (size 0.6) (drill 0.4) (layers F.Cu B.Cu) (net 21))
-  (via (at 26.5 50) (size 0.6) (drill 0.4) (layers F.Cu B.Cu) (net 21))
-  (via (at 35.5 50.25) (size 0.6) (drill 0.4) (layers F.Cu B.Cu) (net 21))
-  (via (at 38 50.25) (size 0.6) (drill 0.4) (layers F.Cu B.Cu) (net 21))
   (segment (start -21.27 -1.26) (end -18.73 -1.26) (width 1) (layer In1.Cu) (net 1) (status 30))
   (via (at -12.7 -10.16) (size 0.6) (drill 0.4) (layers F.Cu B.Cu) (net 1))
@@
   (segment (start -5.08 -46.9964) (end -1.2636 -43.18) (width 0.4) (layer In1.Cu) (net 1))
   (segment (start 26.67 -43.18) (end 26.67 -48.26) (width 0.4) (layer F.Cu) (net 1))
+  (via (at 44.45 42.164) (size 0.6) (drill 0.4) (layers F.Cu B.Cu) (net 2))
+  (via (at 41.148 14.986) (size 0.6) (drill 0.4) (layers F.Cu B.Cu) (net 2))
   (segment (start -18.73 -16.5) (end -21.27 -16.5) (width 2) (layer F.Cu) (net 2) (status 30))
   (segment (start 40.554 15.305764) (end 40.554 18.437) (width 0.4) (layer F.Cu) (net 2))
@@
   (segment (start -2.54 -50.8) (end 0 -53.34) (width 0.4) (layer In1.Cu) (net 4))
   (segment (start 0 -53.34) (end 26.67 -53.34) (width 0.4) (layer In1.Cu) (net 4))
+  (via (at 43.815 38.6715) (size 0.6) (drill 0.4) (layers F.Cu B.Cu) (net 5))
+  (via (at 37.719 15.5575) (size 0.6) (drill 0.4) (layers F.Cu B.Cu) (net 5))
+  (via (at 12.4 -48.4) (size 0.6) (drill 0.4) (layers F.Cu B.Cu) (net 5))
+  (via (at 12.4 -51.4) (size 0.6) (drill 0.4) (layers F.Cu B.Cu) (net 5))
   (segment (start -21.27 6.36) (end -18.73 6.36) (width 1) (layer B.Cu) (net 5) (status 30))
   (segment (start 16.55 -46.888731) (end 16.55 -50) (width 2) (layer B.Cu) (net 5))
@@
   (segment (start -13.1 -3.8) (end -18.73 -3.8) (width 0.4) (layer F.Cu) (net 13))
   (segment (start -8.6 -8.3) (end -13.1 -3.8) (width 0.4) (layer F.Cu) (net 13))
+  (via (at 45.72 -48.26) (size 0.6) (drill 0.4) (layers F.Cu B.Cu) (net 14))
+  (via (at 8.89 -41.275) (size 0.6) (drill 0.4) (layers F.Cu B.Cu) (net 14))
   (segment (start 9.189999 -41.574999) (end 8.89 -41.275) (width 2) (layer In2.Cu) (net 14))
   (segment (start 13.694989 -46.079989) (end 9.189999 -41.574999) (width 2) (layer In2.Cu) (net 14))
@@
   (segment (start 33 38.095092) (end 33 41.656) (width 2) (layer In2.Cu) (net 16))
   (segment (start 33 41.656) (end 33 42.609999) (width 2) (layer In2.Cu) (net 16))
+  (via (at 45.72 41.3385) (size 0.6) (drill 0.4) (layers F.Cu B.Cu) (net 17))
+  (via (at 41.783 12.1285) (size 0.6) (drill 0.4) (layers F.Cu B.Cu) (net 17))
+  (via (at 41.91 -5.334) (size 0.6) (drill 0.4) (layers F.Cu B.Cu) (net 17))
   (via (at 26.971508 47.950846) (size 0.6) (drill 0.4) (layers F.Cu B.Cu) (net 17))
   (segment (start 41.854 12.1995) (end 41.854 13.687) (width 0.4) (layer F.Cu) (net 17))
@@
   (segment (start -1.003293 53.660001) (end 27.94 53.660001) (width 2) (layer In2.Cu) (net 17))
   (segment (start 27.94 53.660001) (end 49.592801 53.660001) (width 2) (layer In2.Cu) (net 17))
+  (via (at 47.752 -12.192) (size 0.6) (drill 0.4) (layers F.Cu B.Cu) (net 18))
+  (via (at 46.736 -26.416) (size 0.6) (drill 0.4) (layers F.Cu B.Cu) (net 18))
+  (via (at 41.656 -22.86) (size 0.6) (drill 0.4) (layers F.Cu B.Cu) (net 18))
+  (via (at 42.4815 -15.367) (size 0.6) (drill 0.4) (layers F.Cu B.Cu) (net 18))
+  (via (at 39.3065 -15.4305) (size 0.6) (drill 0.4) (layers F.Cu B.Cu) (net 18))
+  (via (at 44.45 1.524) (size 0.6) (drill 0.4) (layers F.Cu B.Cu) (net 18))
+  (via (at 45.72 -5.08) (size 0.6) (drill 0.4) (layers F.Cu B.Cu) (net 18))
+  (via (at 37.25 42.75) (size 0.6) (drill 0.4) (layers F.Cu B.Cu) (net 18))
+  (via (at 40.25 42.75) (size 0.6) (drill 0.4) (layers F.Cu B.Cu) (net 18))
   (segment (start 29.664999 -7.075001) (end 30.165001 -6.574999) (width 2) (layer B.Cu) (net 18))
   (segment (start 29.664999 -13.691801) (end 29.664999 -7.075001) (width 2) (layer B.Cu) (net 18))
@@
   (segment (start 45.085 -19.431) (end 41.656 -22.86) (width 2) (layer B.Cu) (net 18))
   (segment (start 51.749 -19.431) (end 45.085 -19.431) (width 2) (layer B.Cu) (net 18))
+  (via (at 46.99 1.016) (size 0.6) (drill 0.4) (layers F.Cu B.Cu) (net 19))
+  (via (at 46.1645 47.879) (size 0.6) (drill 0.4) (layers F.Cu B.Cu) (net 19))
+  (via (at 41.402 21.463) (size 0.6) (drill 0.4) (layers F.Cu B.Cu) (net 19))
+  (via (at 45.72 1.524) (size 0.6) (drill 0.4) (layers F.Cu B.Cu) (net 19))
   (via (at 30.471508 46.950846) (size 0.6) (drill 0.4) (layers F.Cu B.Cu) (net 19))
   (segment (start 41.8465 19.5945) (end 41.854 19.587) (width 0.4) (layer F.Cu) (net 19))
@@
   (segment (start 29.0125 52.9875) (end 30 52) (width 1) (layer F.Cu) (net 20))
   (segment (start 26.5 52.9875) (end 29.0125 52.9875) (width 1) (layer F.Cu) (net 20))
+  (via (at 24 50) (size 0.6) (drill 0.4) (layers F.Cu B.Cu) (net 21))
+  (via (at 26.5 50) (size 0.6) (drill 0.4) (layers F.Cu B.Cu) (net 21))
+  (via (at 35.5 50.25) (size 0.6) (drill 0.4) (layers F.Cu B.Cu) (net 21))
+  (via (at 38 50.25) (size 0.6) (drill 0.4) (layers F.Cu B.Cu) (net 21))
   (segment (start 24.539154 46.000846) (end 24.5 46.04) (width 1) (layer F.Cu) (net 21))
   (segment (start 27.161508 46.000846) (end 24.539154 46.000846) (width 1) (layer F.Cu) (net 21))
@@
   (segment (start 51.2715 -17.243499) (end 51.749 -17.720999) (width 2) (layer F.Cu) (net 24))
   (segment (start 51.2715 -12.192) (end 51.2715 -17.243499) (width 2) (layer F.Cu) (net 24))
+  (via (at 42.164 -40.64) (size 0.6) (drill 0.4) (layers F.Cu B.Cu) (net 25))
+  (via (at 46.99 -33.274) (size 0.6) (drill 0.4) (layers F.Cu B.Cu) (net 25))
   (segment (start 54.527 -22.831) (end 55.51999 -21.83801) (width 2) (layer F.Cu) (net 25))
   (segment (start 51.749 -22.831) (end 54.527 -22.831) (width 2) (layer F.Cu) (net 25))
@@
   (segment (start 26.245001 6.985001) (end 33.654999 6.985001) (width 0.5) (layer In2.Cu) (net 27))
   (segment (start 44.45 -3.81) (end 44.45 -4.605) (width 0.5) (layer F.Cu) (net 27))
+  (via (at 41.402 51.816) (size 0.6) (drill 0.4) (layers F.Cu B.Cu) (net 28))
   (segment (start 42.4545 -10.922) (end 42.4545 -8.382) (width 0.5) (layer F.Cu) (net 28))
   (segment (start 43.18 -7.6565) (end 43.18 -4.605) (width 0.5) (layer F.Cu) (net 28))
