File: KiCAD/base1x/base1x.sch (KiCad schematic (older format))
At the start: 35 parts, among them CON1 AVR-JTAG-10, J1 Conn_02x04_Counter_Clockwise, J2 Conn_01x17, J3 Conn_02x14_Counter_Clockwise, J4 Conn_01x17, J5 Screw_Terminal_01x02, J6 Conn_02x14_Counter_Clockwise, J7 Screw_Terminal_01x04, SW1 SW_DIP_x04, SW2 SW_Grayhill_94H_Coded, SW3 SW_Grayhill_94H_Coded, SW4 SW_Push, SW5 SW_DIP_x04, U1 ARDUINO_MICRO, U2 74LS249, U3 74LS249, U4 KCSC02-123, U5 KCSC02-123, U6 MCP23S17

Commit message: fixed up newMux so that parts don't collide
Parts:
- J3, J6: symbol Conn_02x14_Counter_Clockwise -> Conn_02x14_Odd_Even
- SW2, SW3: footprint (none) -> myParts:Grayhill_94H
Changed lines of the file:
@@
 $EndComp
 $Comp
-L Conn_02x14_Counter_Clockwise J3
+L Conn_02x14_Odd_Even J3
 U 1 1 59C14E89
 P 1700 6800
@@
 V_D
 $Comp
-L Conn_02x14_Counter_Clockwise J6
+L Conn_02x14_Odd_Even J6
 U 1 1 59C14E79
 P 9950 5450
@@
 L SW_DIP_x04 SW5
 U 1 1 59C92248
-P 10550 5950
-F 0 "SW5" H 10550 6417 50  0000 C CNN
-F 1 "SW_DIP_x04" H 10550 6326 50  0000 C CNN
-F 2 "Buttons_Switches_THT:SW_DIP_x4_W7.62mm_Piano" H 10550 5950 50  0001 C CNN
-F 3 "" H 10550 5950 50  0001 C CNN
-	1    10550 5950
-	1    0    0    -1
+P 10550 5850
+F 0 "SW5" H 10550 6317 50  0000 C CNN
+F 1 "SW_DIP_x04" H 10550 6226 50  0000 C CNN
+F 2 "Buttons_Switches_THT:SW_DIP_x4_W7.62mm_Piano" H 10550 5850 50  0001 C CNN
+F 3 "" H 10550 5850 50  0001 C CNN
+	1    10550 5850
+	-1   0    0    1
 $EndComp
 $Comp
@@
 F 0 "SW2" H 3780 3675 50  0000 C CNN
 F 1 "SW_Grayhill_94H_Coded" H 3780 3584 50  0000 C CNN
-F 2 "" H 3625 3225 50  0001 C CNN
+F 2 "myParts:Grayhill_94H" H 3625 3225 50  0001 C CNN
 F 3 "" H 3625 3225 50  0001 C CNN
 	1    3650 3200
@@
 F 0 "SW3" H 3880 1625 50  0000 C CNN
 F 1 "SW_Grayhill_94H_Coded" H 3880 1534 50  0000 C CNN
-F 2 "" H 3725 1175 50  0001 C CNN
+F 2 "myParts:Grayhill_94H" H 3725 1175 50  0001 C CNN
 F 3 "" H 3725 1175 50  0001 C CNN
 	1    3750 1150

Commit message: wip for base1x
Parts:
- removed J5: Screw_Terminal_01x02, Connectors_Phoenix:PhoenixContact_MC-GF_02x3.50mm_Angled_ThreadedFlange_MountHole, symbol Screw_Terminal_01x02
- removed J7: Screw_Terminal_01x04, Connectors_Phoenix:PhoenixContact_MC-GF_04x3.50mm_Angled_ThreadedFlange_MountHole, symbol Screw_Terminal_01x04
- removed MK1, MK2: Mounting_Hole_PAD, Mounting_Holes:MountingHole_4mm_Pad, symbol Mounting_Hole_PAD
- removed SW1, SW5: SW_DIP_x04, Buttons_Switches_THT:SW_DIP_x4_W7.62mm_Piano, symbol SW_DIP_x04
- added J5: Screw_Terminal_01x06, Connectors_Phoenix:PhoenixContact_MC-GF_06x3.50mm_Angled_ThreadedFlange_MountHole, symbol Screw_Terminal_01x06
- MK1: renamed from MK3; footprint Mounting_Holes:MountingHole_4mm_Pad -> Mounting_Holes:MountingHole_2.2mm_M2_Pad
- MK2: renamed from MK4; footprint Mounting_Holes:MountingHole_4mm_Pad -> Mounting_Holes:MountingHole_2.2mm_M2_Pad
- renumbered SW2 to SW1, SW3 to SW2, SW4 to SW3
Connections:
- wire segments 125 -> 123

Commit message: make spring pin board pin holders smaller, update base1x, update mux design controller board
Parts:
- removed C1: 0.1uF, Capacitors_SMD:C_0603_HandSoldering, symbol C
- removed CON1: AVR-JTAG-10, Connectors_Multicomp:Multicomp_MC9A12-1034_2x05x2.54mm_Straight, symbol AVR-JTAG-10
- removed J1: Conn_02x04_Counter_Clockwise, Socket_Strips:Socket_Strip_Straight_2x04_Pitch2.54mm, symbol Conn_02x04_Counter_Clockwise
- removed J2, J4: Conn_01x17, Socket_Strips:Socket_Strip_Straight_1x17_Pitch2.54mm, symbol Conn_01x17
- removed JP1, JP6: Jumper_NO_Small, Connectors:GS2, symbol Jumper_NO_Small
- removed JP3, JP4, JP5: Jumper_NC_Dual, Connectors:GS3, symbol Jumper_NC_Dual
- removed R1, R2: 10K, Resistors_SMD:R_0805_HandSoldering, symbol R
- removed RN1, RN2: 1k, Housings_DIP:DIP-16_W7.62mm, symbol R_Pack08
- removed SW1, SW2: SW_Grayhill_94H_Coded, myParts:Grayhill_94H, symbol SW_Grayhill_94H_Coded
- removed SW3: SW_Push, Buttons_Switches_THT:SW_PUSH_6mm, symbol SW_Push
- removed U1: ARDUINO_MICRO, myparts:arduino_micro, symbol ARDUINO_MICRO
- removed U2, U3: 74LS249, Housings_DIP:DIP-16_W7.62mm, symbol 74LS249
- removed U4, U5: KCSC02-123, Displays_7-Segment:KCSC02-123, symbol KCSC02-123
- removed U6: MCP23S17, Housings_DIP:DIP-28_W7.62mm, symbol MCP23S17
- added C1: 1uF, Capacitors_SMD:C_0805_HandSoldering, symbol C_Small
- added D1, D2: BPW21, myParts:BPW21, symbol D_Photo
- added J1: Conn_02x05_Odd_Even, Pin_Headers:Pin_Header_Angled_2x05_Pitch2.54mm, symbol Conn_02x05_Odd_Even
- added J2, J4: GS3, Connectors:GS3, symbol GS3
- added J7, J8: Conn_02x06_Counter_Clockwise, Socket_Strips:Socket_Strip_Straight_2x06_Pitch2.54mm, symbol Conn_02x06_Counter_Clockwise
- added JP2, JP3, JP4, JP5: Jumper_NO_Small, Connectors:GS2, symbol Jumper_NO_Small
- added MK3, MK4: Mounting_Hole, Mounting_Holes:MountingHole_6mm, symbol Mounting_Hole
- added MK5, MK7, MK8: Mounting_Hole, Mounting_Holes:MountingHole_3.2mm_M3, symbol Mounting_Hole
- added MK6: Mounting_Hole, Mounting_Holes:MountingHole_4.3mm_M4, symbol Mounting_Hole
- added P1, P2: CONN_01X02, Pin_Headers:Pin_Header_Straight_1x02_Pitch2.54mm, symbol Conn_01x02
- added R1, R2: 1.2K, Resistors_SMD:R_0805_HandSoldering, symbol R_Small
- added R3, R4: 10K, Resistors_SMD:R_0805_HandSoldering, symbol R_Small
- added TP1, TP2: Test_Point, myParts:Test_Point_S1751-46R, symbol Test_Point
- added U1: ADS1115, Housings_SSOP:MSOP-10_3x3mm_Pitch0.5mm, symbol ADS1115
- J5: farnellCode (none) -> 2776336+1793013
- renumbered JP2 to JP6
Connections:
- net labels added: ANODE_A, ANODE_B, CATHODE_A, CATHODE_B, I+L, I+R, I-L, I-R, V+L, V+R, V-L, V-R, V_D_EXT, V_D_LOC
- net labels removed: +3.3V, 0(Rx1), 1(Tx1), 10(A10), 11(**), 12(A11), 13(**), 4(A6), 5(**), 6(**/A7), 7, 8, 9(**/A9), A0_SW, A1_SW, A2_SW, A4, ADC0, ADC0(A5), AREF, BCD_P_A, BCD_P_B, BCD_P_C, BCD_P_D, BCD_S_A, BCD_S_B, BCD_S_C, BCD_S_D, INT_BUT, INT_SW, NC0, NC1, RESET, SS, SWP1, SWP2, SWP4, SWP8, SWS1, SWS2, SWS4, SWS8, TCK, TDI, TDO, TMS, ~CS_LED_SW
- wire segments 123 -> 82
- no-connect marks 21 -> 34
Other:
- note removed: "1"
- note removed: "2(SDA)"
- note removed: "3(**/SCL)"
- note removed: "Analog Pins"
- note removed: "Digital Pins"
- note removed: "Pixel indicator"
- note removed: "Pixel selector"
- note removed: "Read divider sense volage with ADC0"
- note removed: "Substrate indicator"
- note removed: "Substrate selector"
- note removed: "USB_SIDE"

Commit message: wip commit
Parts:
- added J9: Screw_Terminal_01x08, Connectors_Phoenix:PhoenixContact_MC-GF_08x3.50mm_Angled_ThreadedFlange_MountHole, symbol Screw_Terminal_01x08
- added P3, P4: CONN_01X02, Pin_Headers:Pin_Header_Straight_1x02_Pitch2.54mm, symbol Conn_01x02
- added R5: 1, Resistors_SMD:R_2512_HandSoldering, symbol R
- added TP3, TP4, TP5: Test_Point, myParts:Test_Point_S1751-46R, symbol Test_Point
Connections:
- net GND: now also J9.8 (Pin_8), P3.2 (Pin_2); no longer J5.6 (Pin_6)
- net I+: now also J9.1 (Pin_1); no longer J5.1 (Pin_1)
- net I-: now also TP2.1, U1.5 (AIN1), J9.5 (Pin_5), P4.2 (Pin_2), R5.2; no longer J5.4 (Pin_4)
- net V+: now also J9.2 (Pin_2); no longer J5.2 (Pin_2)
- net V-: now also J9.3 (Pin_3); no longer J5.3 (Pin_3)
- net V_D_LOC: now also TP5.1
- net Vin: now also J9.7 (Pin_7); no longer J5.5 (Pin_5)
- net at JP2.1, R1.1, U1.6 (AIN2): now also TP3.1
- net at JP4.1, R2.1, U1.7 (AIN3): now also TP4.1
- new net I-_EXT: J9.4 (Pin_4), P3.1 (Pin_1), P4.1 (Pin_1), R5.1
- no-connect marks 34 -> 41
Other:
- moved on the sheet: J5
Changed lines of the file:
@@
-$EndComp
-$Comp
-L +5V #PWR011
-U 1 1 58FF8E76
-P 3300 7400
-F 0 "#PWR011" H 3300 7250 50  0001 C CNN
-F 1 "+5V" H 3300 7540 28  0000 C CNN
-F 2 "" H 3300 7400 50  0000 C CNN
-F 3 "" H 3300 7400 50  0000 C CNN
-	1    3300 7400
-	1    0    0    -1
-$EndComp
-$Comp
-L PWR_FLAG #FLG02
-U 1 1 58FF8E7C
-P 3300 7400
-F 0 "#FLG02" H 3300 7475 50  0001 C CNN
-F 1 "PWR_FLAG" H 3300 7550 50  0000 C CNN
-F 2 "" H 3300 7400 50  0000 C CNN
-F 3 "" H 3300 7400 50  0000 C CNN
-	1    3300 7400
-	-1   0    0    1
 $EndComp
 $Comp
@@
 Text Notes 2400 5900 2    60   ~ 0
 LEFT SIDE BUS CONNECTIONS
-Text GLabel 10150 800  1    60   Input ~ 0
+Text GLabel 10550 1150 1    60   Input ~ 0
 I+
-Text GLabel 10050 800  1    60   Input ~ 0
+Text GLabel 10450 1150 1    60   Input ~ 0
 V+
 $Comp
@@
 Text GLabel 1550 3450 2    60   Input ~ 0
 SCL
-Text GLabel 9850 800  1    60   Input ~ 0
-I-
-Text GLabel 9950 800  1    60   Input ~ 0
+Text GLabel 10250 1150 1    60   Input ~ 0
+I-_EXT
+Text GLabel 10350 1150 1    60   Input ~ 0
 V-
-Text Notes 9900 600  0    60   ~ 0
+Text Notes 10300 950  0    60   ~ 0
 To Sourcemeter
-Text Label 9750 800  1    60   ~ 0
+Text Label 9950 1150 1    60   ~ 0
 Vin
-Text Notes 9100 600  0    60   ~ 0
+Text Notes 9300 950  0    60   ~ 0
 External Power
 $Comp
@@
 	1550 3350 1950 3350
 Wire Wire Line
-	9750 800  9750 650
-Wire Wire Line
-	9650 800  9650 650
+	9950 1150 9950 1000
+Wire Wire Line
+	9850 1150 9850 1000
 Wire Wire Line
 	3300 6550 3300 6650
@@
 L Screw_Terminal_01x06 J5
 U 1 1 59DCB366
-P 9950 1000
-F 0 "J5" V 9823 1280 50  0000 L CNN
-F 1 "Screw_Terminal_01x06" V 9914 1280 50  0000 L CNN
-F 2 "Connectors_Phoenix:PhoenixContact_MC-GF_06x3.50mm_Angled_ThreadedFlange_MountHole" H 9950 1000 50  0001 C CNN
-F 3 "" H 9950 1000 50  0001 C CNN
-F 4 "2776336+1793013" V 9950 1000 60  0001 C CNN "farnellCode"
-	1    9950 1000
+P 10900 1850
+F 0 "J5" V 10773 2130 50  0000 L CNN
+F 1 "Screw_Terminal_01x06" V 10864 2130 50  0000 L CNN
+F 2 "Connectors_Phoenix:PhoenixContact_MC-GF_06x3.50mm_Angled_ThreadedFlange_MountHole" H 10900 1850 50  0001 C CNN
+F 3 "" H 10900 1850 50  0001 C CNN
+F 4 "2776336+1793013" V 10900 1850 60  0001 C CNN "farnellCode"
+	1    10900 1850
 	0    1    1    0
 $EndComp
@@
 L GND #PWR024
 U 1 1 59F71C15
-P 9350 900
-F 0 "#PWR024" H 9350 650 50  0001 C CNN
-F 1 "GND" H 9350 750 50  0000 C CNN
-F 2 "" H 9350 900 50  0000 C CNN
-F 3 "" H 9350 900 50  0000 C CNN
-	1    9350 900
-	1    0    0    -1
-$EndComp
-Wire Wire Line
-	9650 650  9350 650
-Wire Wire Line
-	9350 650  9350 900
+P 9550 1250
+F 0 "#PWR024" H 9550 1000 50  0001 C CNN
+F 1 "GND" H 9550 1100 50  0000 C CNN
+F 2 "" H 9550 1250 50  0000 C CNN
+F 3 "" H 9550 1250 50  0000 C CNN
+	1    9550 1250
+	1    0    0    -1
+$EndComp
+Wire Wire Line
+	9850 1000 9550 1000
+Wire Wire Line
+	9550 1000 9550 1250
 Wire Wire Line
 	1050 3550 700  3550
@@
 Text GLabel 1200 4650 2    60   Input ~ 0
 V_D_EXT
-Text GLabel 5300 2150 0    60   Input ~ 0
-V_D_LOC
 Text GLabel 1050 3350 0    60   Input ~ 0
 V_D_EXT
@@
 Wire Wire Line
 	4700 6750 4700 6450
+$Comp
+L Screw_Terminal_01x08 J9
+U 1 1 5A36A6E7
+P 10250 1350
+F 0 "J9" V 10374 1296 50  0000 C CNN
+F 1 "Screw_Terminal_01x08" V 10465 1296 50  0000 C CNN
+F 2 "Connectors_Phoenix:PhoenixContact_MC-GF_08x3.50mm_Angled_ThreadedFlange_MountHole" H 10250 1350 50  0001 C CNN
+F 3 "" H 10250 1350 50  0001 C CNN
+F 4 "2776340+1793014" V 10250 1350 60  0001 C CNN "farnellCode"
+	1    10250 1350
+	0    1    1    0
+$EndComp
+Wire Wire Line
+	10150 1150 10150 1000
+Text Label 10350 3350 0    60   ~ 0
+I_sense
+Text Label 10150 1150 1    60   ~ 0
+I_sense
+$Comp
+L R R5
+U 1 1 5A36BE72
+P 10350 3050
+F 0 "R5" H 10420 3096 50  0000 L CNN
+F 1 "1" H 10420 3005 50  0000 L CNN
+F 2 "Resistors_SMD:R_2512_HandSoldering" V 10280 3050 50  0001 C CNN
+F 3 "" H 10350 3050 50  0001 C CNN
+F 4 "2663692" H 10350 3050 60  0001 C CNN "farnellCode"
+	1    10350 3050
+	1    0    0    -1
+$EndComp
+$Comp
+L Conn_01x02 P4
+U 1 1 5A36C25C
+P 9950 3000
+F 0 "P4" H 9950 3150 50  0000 C CNN
+F 1 "CONN_01X02" V 10050 3000 50  0000 C CNN
+F 2 "Pin_Headers:Pin_Header_Straight_1x02_Pitch2.54mm" H 9950 3000 50  0001 C CNN
+F 3 "" H 9950 3000 50  0000 C CNN
+	1    9950 3000
+	-1   0    0    -1
+$EndComp
+Wire Wire Line
+	10350 2900 10150 2900
+Wire Wire Line
+	10150 2900 10150 3000
+Wire Wire Line
+	10150 3200 10350 3200
+Wire Wire Line
+	10150 3200 10150 3100
+Text GLabel 10250 3200 3    60   Input ~ 0
+I-
+Text GLabel 10250 2900 1    60   Input ~ 0
+I-_EXT
+$Comp
+L Conn_01x02 P3
+U 1 1 5A36D44F
+P 9900 2000
+F 0 "P3" H 9900 2150 50  0000 C CNN
+F 1 "CONN_01X02" V 10000 2000 50  0000 C CNN
+F 2 "Pin_Headers:Pin_Header_Straight_1x02_Pitch2.54mm" H 9900 2000 50  0001 C CNN
+F 3 "" H 9900 2000 50  0000 C CNN
+	1    9900 2000
+	-1   0    0    -1
+$EndComp
+Text GLabel 10200 2000 2    60   Input ~ 0
+I-_EXT
+Wire Wire Line
+	10100 2000 10200 2000
+$Comp
+L GND #PWR033
+U 1 1 5A36D756
+P 10200 2250
+F 0 "#PWR033" H 10200 2000 50  0001 C CNN
+F 1 "GND" H 10200 2100 50  0000 C CNN
+F 2 "" H 10200 2250 50  0000 C CNN
+F 3 "" H 10200 2250 50  0000 C CNN
+	1    10200 2250
+	1    0    0    -1
+$EndComp
+Wire Wire Line
+	10100 2100 10200 2100
+Wire Wire Line
+	10200 2100 10200 2250
+Wire Wire Line
+	10350 3200 10350 3350
+NoConn ~ 10050 1150
+NoConn ~ 10600 1650
+NoConn ~ 10700 1650
+NoConn ~ 10800 1650
+NoConn ~ 10900 1650
+NoConn ~ 11000 1650
+NoConn ~ 11100 1650
+$Comp
+L Test_Point TP3
+U 1 1 5A3700D5
+P 4450 2200
+F 0 "TP3" H 4508 2320 50  0000 L CNN
+F 1 "Test_Point" H 4508 2229 50  0000 L CNN
+F 2 "myParts:Test_Point_S1751-46R" H 4650 2200 50  0001 C CNN
+F 3 "" H 4650 2200 50  0001 C CNN
+	1    4450 2200
+	1    0    0    -1
+$EndComp
+$Comp
+L Test_Point TP4
+U 1 1 5A370173
+P 5000 2850
+F 0 "TP4" H 5058 2970 50  0000 L CNN
+F 1 "Test_Point" H 5058 2879 50  0000 L CNN
+F 2 "myParts:Test_Point_S1751-46R" H 5200 2850 50  0001 C CNN
+F 3 "" H 5200 2850 50  0001 C CNN
+	1    5000 2850
+	-1   0    0    1
+$EndComp
+Wire Wire Line
+	4700 1950 4150 1950
+Connection ~ 4700 1950
+Text Label 4150 1950 0    60   ~ 0
+I_sense
+Text GLabel 4650 1200 0    60   Input ~ 0
+V_D_LOC
+Wire Wire Line
+	5300 2150 5150 2150
+Wire Wire Line
+	5150 2150 5150 1200
+Wire Wire Line
+	5150 1200 4650 1200
+$Comp
+L Test_Point TP5
+U 1 1 5A371768
+P 5150 1200
+F 0 "TP5" H 5208 1320 50  0000 L CNN
+F 1 "Test_Point" H 5208 1229 50  0000 L CNN
+F 2 "myParts:Test_Point_S1751-46R" H 5350 1200 50  0001 C CNN
+F 3 "" H 5350 1200 50  0001 C CNN
+	1    5150 1200
+	1    0    0    -1
+$EndComp
 $EndSCHEMATC
