File: KiCAD/megaHalfShield/megaHalfShield.sch (KiCad schematic (older format))
At the start: 9 parts, among them J1 Conn_02x05_Odd_Even, J2 Conn_01x01, P1 Digital, P10 CONN_01X01, P13 CONN_01X01, P4 Analog, P7 Communication

Commit message: move arduino headers into myparts
Parts:
- added L1: GREY@CHRISTOFORO.NET, myparts:logo, symbol myParts:GREY@CHRISTOFORO.NET
- J1: symbol Conn_02x05_Odd_Even -> Connector:Conn_02x05_Odd_Even
- J2: symbol Conn_01x01 -> Connector:Conn_01x01
- P1: footprint Socket_Arduino_Mega:Socket_Strip_Arduino_2x18 -> myparts:Socket_Strip_Arduino_2x18; symbol CONN_02X18 -> Connector:Conn_02x18_Odd_Even
- P10, P13: footprint Socket_Arduino_Mega:Arduino_1pin -> myparts:Arduino_1pin; symbol CONN_01X01 -> Connector:Conn_01x01
- P4, P7: footprint Socket_Arduino_Mega:Socket_Strip_Arduino_1x08 -> myparts:Socket_Strip_Arduino_1x08; symbol CONN_01X08 -> Connector:Conn_01x08
- R1, R2: symbol R_Small -> device:R_Small
Connections:
- wire segments 69 -> 72
Changed lines of the file:
@@
-EESchema Schematic File Version 2
-LIBS:ac-dc
-LIBS:adc-dac
-LIBS:Altera
-LIBS:analog_devices
-LIBS:analog_switches
-LIBS:atmel
-LIBS:audio
-LIBS:Battery_Management
-LIBS:bbd
-LIBS:Bosch
-LIBS:brooktre
-LIBS:Connector
-LIBS:contrib
-LIBS:cypress
-LIBS:dc-dc
-LIBS:device
-LIBS:digital-audio
-LIBS:Diode
-LIBS:Display
-LIBS:driver_gate
-LIBS:dsp
-LIBS:DSP_Microchip_DSPIC33
-LIBS:elec-unifil
-LIBS:ESD_Protection
-LIBS:Espressif
-LIBS:FPGA_Actel
-LIBS:ftdi
-LIBS:gennum
-LIBS:Graphic
-LIBS:hc11
-LIBS:infineon
-LIBS:intel
-LIBS:interface
-LIBS:intersil
-LIBS:ir
-LIBS:Lattice
-LIBS:LED
-LIBS:LEM
-LIBS:linear
-LIBS:Logic_74xgxx
-LIBS:Logic_74xx
-LIBS:Logic_CMOS_4000
-LIBS:Logic_CMOS_IEEE
-LIBS:logic_programmable
-LIBS:Logic_TTL_IEEE
-LIBS:maxim
-LIBS:MCU_Microchip_PIC10
-LIBS:MCU_Microchip_PIC12
-LIBS:MCU_Microchip_PIC16
-LIBS:MCU_Microchip_PIC18
-LIBS:MCU_Microchip_PIC24
-LIBS:MCU_Microchip_PIC32
-LIBS:MCU_NXP_Kinetis
-LIBS:MCU_NXP_LPC
-LIBS:MCU_NXP_S08
-LIBS:MCU_Parallax
-LIBS:MCU_ST_STM8
-LIBS:MCU_ST_STM32
-LIBS:MCU_Texas_MSP430
-LIBS:Mechanical
-LIBS:memory
-LIBS:microchip
-LIBS:microcontrollers
-LIBS:modules
-LIBS:Motor
-LIBS:motor_drivers
-LIBS:motorola
-LIBS:nordicsemi
-LIBS:nxp
-LIBS:onsemi
-LIBS:opto
-LIBS:Oscillators
-LIBS:philips
-LIBS:power
-LIBS:powerint
-LIBS:Power_Management
-LIBS:pspice
-LIBS:references
-LIBS:regul
-LIBS:Relay
-LIBS:rfcom
-LIBS:RFSolutions
-LIBS:Sensor_Current
-LIBS:sensors
-LIBS:silabs
-LIBS:siliconi
-LIBS:supertex
-LIBS:Switch
-LIBS:texas
-LIBS:Transformer
-LIBS:Transistor
-LIBS:triac_thyristor
-LIBS:Valve
-LIBS:video
-LIBS:wiznet
-LIBS:Worldsemi
-LIBS:Xicor
-LIBS:xilinx
-LIBS:zetex
-LIBS:Zilog
+EESchema Schematic File Version 4
 LIBS:megaHalfShield-cache
 EELAYER 26 0
@@
 Holes
 $Comp
-L CONN_01X01 P10
+L Connector:Conn_01x01 P10
 U 1 1 56D70CE6
 P 11000 650
 F 0 "P10" V 11100 650 31  0000 C CNN
 F 1 "CONN_01X01" V 11100 650 50  0001 C CNN
-F 2 "Socket_Arduino_Mega:Arduino_1pin" H 11000 650 50  0001 C CNN
+F 2 "myparts:Arduino_1pin" H 11000 650 50  0001 C CNN
 F 3 "" H 11000 650 50  0000 C CNN
 	1    11000 650
@@
 $EndComp
 $Comp
-L CONN_01X01 P13
+L Connector:Conn_01x01 P13
 U 1 1 56D711F0
 P 11100 650
 F 0 "P13" V 11200 650 31  0000 C CNN
 F 1 "CONN_01X01" V 11200 650 50  0001 C CNN
-F 2 "Socket_Arduino_Mega:Arduino_1pin" H 11100 650 50  0001 C CNN
+F 2 "myparts:Arduino_1pin" H 11100 650 50  0001 C CNN
 F 3 "" H 11100 650 50  0000 C CNN
 	1    11100 650
@@
 NoConn ~ 11100 850
 $Comp
-L CONN_01X08 P4
+L Connector:Conn_01x08 P4
 U 1 1 56D73A0E
-P 9350 1200
-F 0 "P4" H 9350 1650 50  0000 C CNN
-F 1 "Analog" V 9450 1200 50  0000 C CNN
-F 2 "Socket_Arduino_Mega:Socket_Strip_Arduino_1x08" H 9350 1200 50  0001 C CNN
-F 3 "" H 9350 1200 50  0000 C CNN
-	1    9350 1200
-	1    0    0    -1
-$EndComp
-$Comp
-L CONN_01X08 P7
+P 9350 1150
+F 0 "P4" H 9350 1600 50  0000 C CNN
+F 1 "Analog" V 9450 1150 50  0000 C CNN
+F 2 "myparts:Socket_Strip_Arduino_1x08" H 9350 1150 50  0001 C CNN
+F 3 "" H 9350 1150 50  0000 C CNN
+	1    9350 1150
+	1    0    0    -1
+$EndComp
+$Comp
+L Connector:Conn_01x08 P7
 U 1 1 56D73F2C
-P 9750 1200
-F 0 "P7" H 9750 1650 50  0000 C CNN
-F 1 "Communication" V 9850 1200 50  0000 C CNN
-F 2 "Socket_Arduino_Mega:Socket_Strip_Arduino_1x08" H 9750 1200 50  0001 C CNN
-F 3 "" H 9750 1200 50  0000 C CNN
-	1    9750 1200
+P 9750 1150
+F 0 "P7" H 9750 1600 50  0000 C CNN
+F 1 "Communication" V 9850 1150 50  0000 C CNN
+F 2 "myparts:Socket_Strip_Arduino_1x08" H 9750 1150 50  0001 C CNN
+F 3 "" H 9750 1150 50  0000 C CNN
+	1    9750 1150
 	-1   0    0    -1
 $EndComp
 $Comp
-L CONN_02X18 P1
+L Connector:Conn_02x18_Odd_Even P1
 U 1 1 56D743B5
-P 9550 2550
-F 0 "P1" H 9550 3500 50  0000 C CNN
-F 1 "Digital" V 9550 2550 50  0000 C CNN
-F 2 "Socket_Arduino_Mega:Socket_Strip_Arduino_2x18" H 9550 1500 50  0001 C CNN
-F 3 "" H 9550 1500 50  0000 C CNN
-	1    9550 2550
+P 9500 2500
+F 0 "P1" H 9500 3450 50  0000 C CNN
+F 1 "Digital" V 9550 2450 50  0000 C CNN
+F 2 "myparts:Socket_Strip_Arduino_2x18" H 9500 1450 50  0001 C CNN
+F 3 "" H 9500 1450 50  0000 C CNN
+	1    9500 2500
 	0    -1   1    0
 $EndComp
@@
 	8700 2300 8450 2300
 $Comp
-L GND #PWR05
+L power:GND #PWR05
 U 1 1 56D758F6
 P 8450 3200
@@
 	10550 2300 10400 2300
 $Comp
-L +5V #PWR06
+L power:+5V #PWR06
 U 1 1 56D75AB8
 P 10550 2000
@@
 Connection ~ 10550 2300
 Wire Wire Line
-	10550 2000 10550 2800
-Wire Wire Line
-	8450 2300 8450 3200
+	10550 2000 10550 2300
+Wire Wire Line
+	8450 2300 8450 2800
 Wire Notes Line
 	11200 3500 8350 3500
@@
 	5550 4300 5950 4300
 $Comp
-L Conn_02x05_Odd_Even J1
+L Connector:Conn_02x05_Odd_Even J1
 U 1 1 5A444940
 P 5250 4300
@@
 ~CS0
 $Comp
-L R_Small R1
+L device:R_Small R1
 U 1 1 5A445572
 P 6750 4750
@@
 $EndComp
 $Comp
-L R_Small R2
+L device:R_Small R2
 U 1 1 5A44577C
 P 7150 4750
@@
 	6750 4650 6750 4550
 Wire Wire Line
-	6750 4550 7150 4550
+	6750 4550 6950 4550
 Wire Wire Line
 	6950 4550 6950 4450
@@
 48
 $Comp
-L Conn_01x01 J2
+L Connector:Conn_01x01 J2
 U 1 1 5A446B3B
 P 7450 2450
@@
 	7250 2450 6650 2450
 $Comp
-L +5V #PWR03
+L power:+5V #PWR03
 U 1 1 5A446F5F
 P 6950 4450
@@
 $EndComp
 $Comp
-L +5V #PWR01
+L power:+5V #PWR01
 U 1 1 5A446FC7
 P 5700 4100
@@
 $EndComp
 $Comp
-L GND #PWR02
+L power:GND #PWR02
 U 1 1 5A447171
 P 5950 4300
@@
 NoConn ~ 8700 850
 $Comp
-L GND #PWR04
+L power:GND #PWR04
 U 1 1 5A447B04
 P 9150 5100
@@
 $EndComp
 $Comp
-L +5V #PWR07
+L power:+5V #PWR07
 U 1 1 5A447B21
 P 9150 4600
@@
 $EndComp
 $Comp
-L PWR_FLAG #FLG01
+L power:PWR_FLAG #FLG01
 U 1 1 5A447BB9
 P 9150 5100
@@
 $EndComp
 $Comp
-L PWR_FLAG #FLG02
+L power:PWR_FLAG #FLG02
 U 1 1 5A447BF8
 P 9150 4600
@@
 	-1   0    0    1
 $EndComp
+Wire Wire Line
+	8450 2800 8450 3200
+Wire Wire Line
+	10550 2300 10550 2800
+Wire Wire Line
+	6950 4550 7150 4550
+$Comp
+L myParts:GREY@CHRISTOFORO.NET L1
+U 1 1 5A893AFD
+P 8250 6850
+F 0 "L1" H 8250 6725 60  0001 C CNN
+F 1 "GREY@CHRISTOFORO.NET" H 8275 6850 100 0000 L CNB
+F 2 "myparts:logo" H 8250 6850 60  0001 C CNN
+F 3 "" H 8250 6850 60  0001 C CNN
+	1    8250 6850
+	1    0    0    -1
+$EndComp
 $EndSCHEMATC

Commit message: update farnell codes
Parts:
- P1: farnellcode (none) -> SSQ-118-03-T-D
- P4, P7: farnellcode (none) -> 2505051
- R1, R2: farnellcode (none) -> 2447551
Changed lines of the file:
@@
 F 2 "myparts:Socket_Strip_Arduino_1x08" H 9350 1150 50  0001 C CNN
 F 3 "" H 9350 1150 50  0000 C CNN
+F 4 "2505051" H 0   0   50  0001 C CNN "farnellcode"
 	1    9350 1150
 	1    0    0    -1
@@
 F 2 "myparts:Socket_Strip_Arduino_1x08" H 9750 1150 50  0001 C CNN
 F 3 "" H 9750 1150 50  0000 C CNN
+F 4 "2505051" H 0   0   50  0001 C CNN "farnellcode"
 	1    9750 1150
 	-1   0    0    -1
@@
 F 2 "myparts:Socket_Strip_Arduino_2x18" H 9500 1450 50  0001 C CNN
 F 3 "" H 9500 1450 50  0000 C CNN
+F 4 "SSQ-118-03-T-D" H 9500 2500 50  0001 C CNN "farnellcode"
 	1    9500 2500
 	0    -1   1    0
@@
 F 2 "Resistors_SMD:R_0805_HandSoldering" H 6750 4750 50  0001 C CNN
 F 3 "" H 6750 4750 50  0001 C CNN
+F 4 "2447551" H 0   0   50  0001 C CNN "farnellcode"
 	1    6750 4750
 	-1   0    0    1
@@
 F 2 "Resistors_SMD:R_0805_HandSoldering" H 7150 4750 50  0001 C CNN
 F 3 "" H 7150 4750 50  0001 C CNN
+F 4 "2447551" H 0   0   50  0001 C CNN "farnellcode"
 	1    7150 4750
 	-1   0    0    1

Commit message: upgrade syms and layouts to kicad5
Parts:
- J1: footprint Pin_Headers:Pin_Header_Straight_2x05_Pitch2.54mm -> Connector_IDC:IDC-Header_2x05_P2.54mm_Vertical; symbol Connector:Conn_02x05_Odd_Even -> Connector_Generic:Conn_02x05_Odd_Even; farnellcode (none) -> 2215304
- J2: footprint Pin_Headers:Pin_Header_Straight_1x01_Pitch2.54mm -> Connector_PinSocket_2.54mm:PinSocket_1x01_P2.54mm_Vertical; symbol Connector:Conn_01x01 -> Connector_Generic:Conn_01x01
- P1: symbol Connector:Conn_02x18_Odd_Even -> Connector_Generic:Conn_02x18_Odd_Even
- P10, P13: symbol Connector:Conn_01x01 -> Connector_Generic:Conn_01x01
- P4, P7: symbol Connector:Conn_01x08 -> Connector_Generic:Conn_01x08
- R1, R2: footprint Resistors_SMD:R_0805_HandSoldering -> Resistor_SMD:R_1206_3216Metric; symbol device:R_Small -> Device:R_Small
Changed lines of the file:
@@
 Holes
 $Comp
-L Connector:Conn_01x01 P10
+L Connector_Generic:Conn_01x01 P10
 U 1 1 56D70CE6
 P 11000 650
@@
 $EndComp
 $Comp
-L Connector:Conn_01x01 P13
+L Connector_Generic:Conn_01x01 P13
 U 1 1 56D711F0
 P 11100 650
@@
 NoConn ~ 11100 850
 $Comp
-L Connector:Conn_01x08 P4
+L Connector_Generic:Conn_01x08 P4
 U 1 1 56D73A0E
 P 9350 1150
@@
 $EndComp
 $Comp
-L Connector:Conn_01x08 P7
+L Connector_Generic:Conn_01x08 P7
 U 1 1 56D73F2C
 P 9750 1150
@@
 $EndComp
 $Comp
-L Connector:Conn_02x18_Odd_Even P1
+L Connector_Generic:Conn_02x18_Odd_Even P1
 U 1 1 56D743B5
 P 9500 2500
@@
 	5550 4300 5950 4300
 $Comp
-L Connector:Conn_02x05_Odd_Even J1
+L Connector_Generic:Conn_02x05_Odd_Even J1
 U 1 1 5A444940
 P 5250 4300
 F 0 "J1" H 5300 4717 50  0000 C CNN
 F 1 "Conn_02x05_Odd_Even" H 5300 4626 50  0001 C CNN
-F 2 "Pin_Headers:Pin_Header_Straight_2x05_Pitch2.54mm" H 5250 4300 50  0001 C CNN
+F 2 "Connector_IDC:IDC-Header_2x05_P2.54mm_Vertical" H 5250 4300 50  0001 C CNN
 F 3 "" H 5250 4300 50  0001 C CNN
+F 4 "2215304" H 5250 4300 50  0001 C CNN "farnellcode"
 	1    5250 4300
 	1    0    0    -1
@@
 ~CS0
 $Comp
-L device:R_Small R1
+L Device:R_Small R1
 U 1 1 5A445572
 P 6750 4750
 F 0 "R1" V 6554 4750 50  0000 C CNN
 F 1 "100K" V 6645 4750 50  0000 C CNN
-F 2 "Resistors_SMD:R_0805_HandSoldering" H 6750 4750 50  0001 C CNN
+F 2 "Resistor_SMD:R_1206_3216Metric" H 6750 4750 50  0001 C CNN
 F 3 "" H 6750 4750 50  0001 C CNN
 F 4 "2447551" H 0   0   50  0001 C CNN "farnellcode"
@@
 $EndComp
 $Comp
-L device:R_Small R2
+L Device:R_Small R2
 U 1 1 5A44577C
 P 7150 4750
 F 0 "R2" V 6954 4750 50  0000 C CNN
 F 1 "100K" V 7045 4750 50  0000 C CNN
-F 2 "Resistors_SMD:R_0805_HandSoldering" H 7150 4750 50  0001 C CNN
+F 2 "Resistor_SMD:R_1206_3216Metric" H 7150 4750 50  0001 C CNN
 F 3 "" H 7150 4750 50  0001 C CNN
 F 4 "2447551" H 0   0   50  0001 C CNN "farnellcode"
@@
 48
 $Comp
-L Connector:Conn_01x01 J2
+L Connector_Generic:Conn_01x01 J2
 U 1 1 5A446B3B
 P 7450 2450
 F 0 "J2" H 7530 2492 50  0000 L CNN
 F 1 "Conn_01x01" H 7530 2401 50  0000 L CNN
-F 2 "Pin_Headers:Pin_Header_Straight_1x01_Pitch2.54mm" H 7450 2450 50  0001 C CNN
+F 2 "Connector_PinSocket_2.54mm:PinSocket_1x01_P2.54mm_Vertical" H 7450 2450 50  0001 C CNN
 F 3 "" H 7450 2450 50  0001 C CNN
 	1    7450 2450
