File: KiCAD/megaHalfShield/megaHalfShield.kicad_pcb (KiCad board)
At the start: 2 copper layers, 35.1 x 53.3 mm, 10 parts, among them J1 Conn_02x05_Odd_Even, J2 Conn_01x01, P1 Digital, P10 CONN_01X01, P13 CONN_01X01, P4 Analog, P7 Communication

Commit message: update silk before order 629bf0f
Other:
- board text added: "629bf0f"
- board text removed: "3ec2e93"
Changed lines of the file:
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@@
   )
   (setup
-    (last_trace_width 1)
+    (last_trace_width 0.25)
     (user_trace_width 0.4)
     (user_trace_width 1)
@@
     (effects (font (size 1 1) (thickness 0.25)) (justify right))
   )
-  (gr_text 3ec2e93 (at 177.038 78.486 90) (layer F.SilkS)
+  (gr_text 629bf0f (at 177.038 78.486 90) (layer F.SilkS)
     (effects (font (size 1.5 1.5) (thickness 0.3)))
   )

Commit message: update silk
Other:
- board text added: "779dfac"
- board text removed: "629bf0f"
