File: KiCAD/newMUX/newMUX.sch (KiCad schematic (older format))
At the start: 43 parts, among them J1 Conn_01x14, J2 Conn_02x06_Odd_Even, J3 Conn_02x06_Odd_Even, J4 Conn_01x14, U1 ASSR-1611, U10 ASSR-1611, U11 ASSR-1611, U12 ASSR-1611, U13 ASSR-1611, U14 ASSR-1611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

Commit message: update farnell codes
Parts:
- C1: farnellCode (none) -> 1759143
- J1, J4: farnellCode (none) -> 2037821
- J2, J3: farnellCode (none) -> 1930232
- R1: farnellCode (none) -> 2073783
- R2: farnellCode (none) -> 2073790
- R3: farnellCode (none) -> 2073607
- U1, U10, U11, U12, U13, U14, U15, U16, U17, U18, U19, U2, U20, U21, U3, U4, U5, U6, U7, U8, U9: farnellCode (none) -> 1708441
- U22: farnellCode (none) -> 1292238
Changed lines of the file:
@@
 F 2 "Housings_DIP:DIP-6_W7.62mm" H 1650 4450 50  0001 L CIN
 F 3 "" H 1800 4700 50  0001 L CNN
+F 4 "1708441" H 0   0   50  0001 C CNN "farnellCode"
 	1    1850 4650
 	-1   0    0    -1
@@
 F 2 "Housings_DIP:DIP-28_W7.62mm" H 10000 1150 50  0001 L CNN
 F 3 "" H 10200 3100 50  0001 C CNN
+F 4 "1292238" H 0   0   50  0001 C CNN "farnellCode"
 	1    9950 2100
 	1    0    0    -1
@@
 F 2 "Housings_DIP:DIP-6_W7.62mm" H 1650 4000 50  0001 L CIN
 F 3 "" H 1800 4250 50  0001 L CNN
+F 4 "1708441" H 0   0   50  0001 C CNN "farnellCode"
 	1    1850 4200
 	-1   0    0    -1
@@
 F 2 "Housings_DIP:DIP-6_W7.62mm" H 1650 5350 50  0001 L CIN
 F 3 "" H 1800 5600 50  0001 L CNN
+F 4 "1708441" H 0   0   50  0001 C CNN "farnellCode"
 	1    1850 5550
 	-1   0    0    -1
@@
 F 2 "Housings_DIP:DIP-6_W7.62mm" H 1650 4900 50  0001 L CIN
 F 3 "" H 1800 5150 50  0001 L CNN
+F 4 "1708441" H 0   0   50  0001 C CNN "farnellCode"
 	1    1850 5100
 	-1   0    0    -1
@@
 F 2 "Housings_DIP:DIP-6_W7.62mm" H 1650 3550 50  0001 L CIN
 F 3 "" H 1800 3800 50  0001 L CNN
+F 4 "1708441" H 0   0   50  0001 C CNN "farnellCode"
 	1    1850 3750
 	-1   0    0    -1
@@
 F 2 "Housings_DIP:DIP-6_W7.62mm" H 1650 2200 50  0001 L CIN
 F 3 "" H 1800 2450 50  0001 L CNN
+F 4 "1708441" H 0   0   50  0001 C CNN "farnellCode"
 	1    1850 2400
 	-1   0    0    -1
@@
 F 2 "Housings_DIP:DIP-6_W7.62mm" H 1650 1750 50  0001 L CIN
 F 3 "" H 1800 2000 50  0001 L CNN
+F 4 "1708441" H 0   0   50  0001 C CNN "farnellCode"
 	1    1850 1950
 	-1   0    0    -1
@@
 F 2 "Housings_DIP:DIP-6_W7.62mm" H 1650 3100 50  0001 L CIN
 F 3 "" H 1800 3350 50  0001 L CNN
+F 4 "1708441" H 0   0   50  0001 C CNN "farnellCode"
 	1    1850 3300
 	-1   0    0    -1
@@
 F 2 "Housings_DIP:DIP-6_W7.62mm" H 1650 2650 50  0001 L CIN
 F 3 "" H 1800 2900 50  0001 L CNN
+F 4 "1708441" H 0   0   50  0001 C CNN "farnellCode"
 	1    1850 2850
 	-1   0    0    -1
@@
 F 2 "Housings_DIP:DIP-6_W7.62mm" H 1650 1300 50  0001 L CIN
 F 3 "" H 1800 1550 50  0001 L CNN
+F 4 "1708441" H 0   0   50  0001 C CNN "farnellCode"
 	1    1850 1500
 	-1   0    0    -1
@@
 F 2 "Housings_DIP:DIP-6_W7.62mm" H 3850 4450 50  0001 L CIN
 F 3 "" H 4000 4700 50  0001 L CNN
+F 4 "1708441" H 0   0   50  0001 C CNN "farnellCode"
 	1    4050 4650
 	1    0    0    -1
@@
 F 2 "Housings_DIP:DIP-6_W7.62mm" H 3850 4000 50  0001 L CIN
 F 3 "" H 4000 4250 50  0001 L CNN
+F 4 "1708441" H 0   0   50  0001 C CNN "farnellCode"
 	1    4050 4200
 	1    0    0    -1
@@
 F 2 "Housings_DIP:DIP-6_W7.62mm" H 3850 5350 50  0001 L CIN
 F 3 "" H 4000 5600 50  0001 L CNN
+F 4 "1708441" H 0   0   50  0001 C CNN "farnellCode"
 	1    4050 5550
 	1    0    0    -1
@@
 F 2 "Housings_DIP:DIP-6_W7.62mm" H 3850 4900 50  0001 L CIN
 F 3 "" H 4000 5150 50  0001 L CNN
+F 4 "1708441" H 0   0   50  0001 C CNN "farnellCode"
 	1    4050 5100
 	1    0    0    -1
@@
 F 2 "Housings_DIP:DIP-6_W7.62mm" H 3850 3550 50  0001 L CIN
 F 3 "" H 4000 3800 50  0001 L CNN
+F 4 "1708441" H 0   0   50  0001 C CNN "farnellCode"
 	1    4050 3750
 	1    0    0    -1
@@
 F 2 "Housings_DIP:DIP-6_W7.62mm" H 3850 2200 50  0001 L CIN
 F 3 "" H 4000 2450 50  0001 L CNN
+F 4 "1708441" H 0   0   50  0001 C CNN "farnellCode"
 	1    4050 2400
 	1    0    0    -1
@@
 F 2 "Housings_DIP:DIP-6_W7.62mm" H 3850 1750 50  0001 L CIN
 F 3 "" H 4000 2000 50  0001 L CNN
+F 4 "1708441" H 0   0   50  0001 C CNN "farnellCode"
 	1    4050 1950
 	1    0    0    -1
@@
 F 2 "Housings_DIP:DIP-6_W7.62mm" H 3850 3100 50  0001 L CIN
 F 3 "" H 4000 3350 50  0001 L CNN
+F 4 "1708441" H 0   0   50  0001 C CNN "farnellCode"
 	1    4050 3300
 	1    0    0    -1
@@
 F 2 "Housings_DIP:DIP-6_W7.62mm" H 3850 2650 50  0001 L CIN
 F 3 "" H 4000 2900 50  0001 L CNN
+F 4 "1708441" H 0   0   50  0001 C CNN "farnellCode"
 	1    4050 2850
 	1    0    0    -1
@@
 F 2 "Housings_DIP:DIP-6_W7.62mm" H 3850 1300 50  0001 L CIN
 F 3 "" H 4000 1550 50  0001 L CNN
+F 4 "1708441" H 0   0   50  0001 C CNN "farnellCode"
 	1    4050 1500
 	1    0    0    -1
@@
 F 2 "Socket_Strips:Socket_Strip_Straight_2x06_Pitch2.54mm" H 7850 4400 50  0001 C CNN
 F 3 "" H 7850 4400 50  0001 C CNN
+F 4 "1930232" H 0   0   50  0001 C CNN "farnellCode"
 	1    7850 4400
 	0    1    -1   0
@@
 F 2 "Socket_Strips:Socket_Strip_Straight_2x06_Pitch2.54mm" H 7850 3050 50  0001 C CNN
 F 3 "" H 7850 3050 50  0001 C CNN
+F 4 "1930232" H 0   0   50  0001 C CNN "farnellCode"
 	1    7850 3050
 	0    1    -1   0
@@
 F 2 "Capacitors_SMD:C_0805_HandSoldering" H 10938 800 50  0001 C CNN
 F 3 "" H 10900 950 50  0001 C CNN
+F 4 "1759143" H 0   0   50  0001 C CNN "farnellCode"
 	1    10900 950
 	1    0    0    -1
@@
 F 2 "Resistors_SMD:R_0805_HandSoldering" V 5230 1350 50  0001 C CNN
 F 3 "" H 5300 1350 50  0000 C CNN
+F 4 "2073783" H 0   0   50  0001 C CNN "farnellCode"
 	1    5300 1350
 	-1   0    0    1
@@
 F 2 "Pin_Headers:Pin_Header_Straight_1x14_Pitch2.54mm" H 10900 5450 50  0001 C CNN
 F 3 "" H 10900 5450 50  0001 C CNN
+F 4 "2037821" H 0   0   50  0001 C CNN "farnellCode"
 	1    10900 5450
 	1    0    0    -1
@@
 F 2 "Pin_Headers:Pin_Header_Straight_1x14_Pitch2.54mm" H 750 6900 50  0001 C CNN
 F 3 "" H 750 6900 50  0001 C CNN
+F 4 "2037821" H 0   0   50  0001 C CNN "farnellCode"
 	1    750  6900
 	-1   0    0    -1
@@
 F 2 "Housings_DIP:DIP-6_W7.62mm" H 5850 900 50  0001 L CIN
 F 3 "" H 6000 1150 50  0001 L CNN
+F 4 "1708441" H 0   0   50  0001 C CNN "farnellCode"
 	1    6050 1100
 	1    0    0    -1
@@
 F 2 "Resistors_SMD:R_0805_HandSoldering" V 6530 1350 50  0001 C CNN
 F 3 "" H 6600 1350 50  0000 C CNN
+F 4 "2073790" H 0   0   50  0001 C CNN "farnellCode"
 	1    6600 1350
 	1    0    0    -1
@@
 F 2 "Resistors_SMD:R_0805_HandSoldering" V 10530 1000 50  0001 C CNN
 F 3 "" H 10600 1000 50  0000 C CNN
+F 4 "2073607" H 0   0   50  0001 C CNN "farnellCode"
 	1    10600 1000
 	1    0    0    -1

Commit message: upgrade syms and layouts to kicad5
Parts:
- C1: footprint Capacitors_SMD:C_0805_HandSoldering -> Capacitor_SMD:C_0805_2012Metric; symbol device:C -> Device:C
- J1, J4: footprint Pin_Headers:Pin_Header_Straight_1x14_Pitch2.54mm -> Connector_PinHeader_2.54mm:PinHeader_1x14_P2.54mm_Vertical; symbol Connector:Conn_01x14 -> Connector_Generic:Conn_01x14
- J2, J3: footprint Socket_Strips:Socket_Strip_Straight_2x06_Pitch2.54mm -> Connector_PinSocket_2.54mm:PinSocket_2x06_P2.54mm_Vertical; symbol Connector:Conn_02x06_Odd_Even -> Connector_Generic:Conn_02x06_Odd_Even
- JP1, JP6: footprint Connect:GS2 -> Jumper:SolderJumper-2_P1.3mm_Open_RoundedPad1.0x1.5mm; symbol device:Jumper_NC_Small -> Device:Jumper_NC_Small
- JP2, JP3, JP4, JP5: footprint Connect:GS3 -> Jumper:SolderJumper-3_P1.3mm_Open_RoundedPad1.0x1.5mm_NumberLabels; symbol device:Jumper_NC_Dual -> Device:Jumper_NC_Dual
- R1, R2, R3: footprint Resistors_SMD:R_0805_HandSoldering -> Resistor_SMD:R_1206_3216Metric; symbol device:R -> Device:R
- RN1, RN2, RN3, RN4, RN5: symbol device:R_Pack04 -> Device:R_Pack04
- TP1: symbol Connector:Test_Point -> Connector_Specialized:Test_Point
- U1, U10, U11, U12, U13, U14, U15, U16, U17, U18, U19, U2, U20, U21, U3, U4, U5, U6, U7, U8, U9: footprint Housings_DIP:DIP-6_W7.62mm -> Package_DIP:DIP-6_W7.62mm
- U22: footprint Housings_DIP:DIP-28_W7.62mm -> Package_DIP:DIP-28_W7.62mm
