File: KiCAD/springPins30x30NoWindow/springPins30x30NoWindow.sch (KiCad schematic (older format))
At the start: 21 parts, among them J1 CONN_02X06, J2 CONN_02X06

Commit message: add dbg substrate layout and 8x1 backplane
Parts:
- J1, J2: footprint Pin_Headers:Pin_Header_Straight_2x06_Pitch2.54mm -> Connector_PinHeader_2.54mm:PinHeader_2x06_P2.54mm_Vertical; symbol Connector:Conn_02x06_Odd_Even -> Connector_Generic:Conn_02x06_Odd_Even
- JP1: footprint Connectors:GS2 -> Jumper:SolderJumper-2_P1.3mm_Open_RoundedPad1.0x1.5mm; symbol device:Jumper_NO_Small -> Device:Jumper_NO_Small
- R1: footprint Resistors_SMD:R_0805_HandSoldering -> Resistor_SMD:R_1206_3216Metric; symbol device:R -> Device:R
- TP10, TP11, TP12, TP15, TP16, TP17, TP18, TP19, TP20, TP3, TP4, TP5, TP6, TP7, TP8, TP9: symbol Connector:Test_Point -> Connector_Specialized:Test_Point
Changed lines of the file:
@@
 $EndDescr
 $Comp
-L Connector:Test_Point TP10
+L Connector_Specialized:Test_Point TP10
 U 1 1 58E4C4C8
 P 5100 5550
@@
 $EndComp
 $Comp
-L Connector:Test_Point TP6
+L Connector_Specialized:Test_Point TP6
 U 1 1 58E4C4F2
 P 3750 4250
@@
 $EndComp
 $Comp
-L Connector:Test_Point TP5
+L Connector_Specialized:Test_Point TP5
 U 1 1 58E4C553
 P 3750 4100
@@
 $EndComp
 $Comp
-L Connector:Test_Point TP8
+L Connector_Specialized:Test_Point TP8
 U 1 1 58E4C6B7
 P 3750 4800
@@
 $EndComp
 $Comp
-L Connector:Test_Point TP7
+L Connector_Specialized:Test_Point TP7
 U 1 1 58E4C6BD
 P 3750 4650
@@
 $EndComp
 $Comp
-L Connector:Test_Point TP4
+L Connector_Specialized:Test_Point TP4
 U 1 1 58E4C747
 P 3750 3700
@@
 $EndComp
 $Comp
-L Connector:Test_Point TP3
+L Connector_Specialized:Test_Point TP3
 U 1 1 58E4C74D
 P 3750 3550
@@
 $EndComp
 $Comp
-L Connector:Test_Point TP18
+L Connector_Specialized:Test_Point TP18
 U 1 1 58E4CA5F
 P 6650 4250
@@
 $EndComp
 $Comp
-L Connector:Test_Point TP17
+L Connector_Specialized:Test_Point TP17
 U 1 1 58E4CA65
 P 6650 4100
@@
 $EndComp
 $Comp
-L Connector:Test_Point TP20
+L Connector_Specialized:Test_Point TP20
 U 1 1 58E4CA6B
 P 6650 4800
@@
 $EndComp
 $Comp
-L Connector:Test_Point TP19
+L Connector_Specialized:Test_Point TP19
 U 1 1 58E4CA71
 P 6650 4650
@@
 $EndComp
 $Comp
-L Connector:Test_Point TP16
+L Connector_Specialized:Test_Point TP16
 U 1 1 58E4CA77
 P 6650 3700
@@
 $EndComp
 $Comp
-L Connector:Test_Point TP15
+L Connector_Specialized:Test_Point TP15
 U 1 1 58E4CA7D
 P 6650 3550
@@
 $EndComp
 $Comp
-L Connector:Test_Point TP9
+L Connector_Specialized:Test_Point TP9
 U 1 1 58E4CC43
 P 4950 2300
@@
 $EndComp
 $Comp
-L Connector:Test_Point TP11
+L Connector_Specialized:Test_Point TP11
 U 1 1 58E4CC49
 P 5150 2300
@@
 6
 $Comp
-L Connector:Conn_02x06_Odd_Even J1
+L Connector_Generic:Conn_02x06_Odd_Even J1
 U 1 1 599DB107
 P 4550 3950
 F 0 "J1" H 4450 4250 50  0000 C CNN
 F 1 "CONN_02X06" H 4550 3500 50  0000 C CNN
-F 2 "Pin_Headers:Pin_Header_Straight_2x06_Pitch2.54mm" H 4550 2750 50  0001 C CNN
+F 2 "Connector_PinHeader_2.54mm:PinHeader_2x06_P2.54mm_Vertical" H 4550 2750 50  0001 C CNN
 F 3 "" H 4550 2750 50  0001 C CNN
 	1    4550 3950
@@
 $EndComp
 $Comp
-L Connector:Conn_02x06_Odd_Even J2
+L Connector_Generic:Conn_02x06_Odd_Even J2
 U 1 1 599DB1BB
 P 5700 3950
 F 0 "J2" H 5600 4250 50  0000 C CNN
 F 1 "CONN_02X06" H 5700 3500 50  0000 C CNN
-F 2 "Pin_Headers:Pin_Header_Straight_2x06_Pitch2.54mm" H 5700 2750 50  0001 C CNN
+F 2 "Connector_PinHeader_2.54mm:PinHeader_2x06_P2.54mm_Vertical" H 5700 2750 50  0001 C CNN
 F 3 "" H 5700 2750 50  0001 C CNN
 	1    5700 3950
@@
 $EndComp
 $Comp
-L device:R R1
+L Device:R R1
 U 1 1 599DBDE1
 P 4850 4400
 F 0 "R1" V 4930 4400 50  0000 C CNN
 F 1 "200k" V 4850 4400 50  0000 C CNN
-F 2 "Resistors_SMD:R_0805_HandSoldering" V 4780 4400 50  0001 C CNN
+F 2 "Resistor_SMD:R_1206_3216Metric" V 4780 4400 50  0001 C CNN
 F 3 "" H 4850 4400 50  0001 C CNN
 	1    4850 4400
@@
 	4000 3550 3750 3550
 $Comp
-L Connector:Test_Point TP12
+L Connector_Specialized:Test_Point TP12
 U 1 1 58E4C3ED
 P 5250 5550
@@
 $EndComp
 $Comp
-L device:Jumper_NO_Small JP1
+L Device:Jumper_NO_Small JP1
 U 1 1 59F4B423
 P 5600 4550
 F 0 "JP1" H 5600 4735 50  0000 C CNN
 F 1 "Jumper_NO_Small" H 5600 4644 50  0000 C CNN
-F 2 "Connectors:GS2" H 5600 4550 50  0001 C CNN
+F 2 "Jumper:SolderJumper-2_P1.3mm_Open_RoundedPad1.0x1.5mm" H 5600 4550 50  0001 C CNN
 F 3 "" H 5600 4550 50  0001 C CNN
 	1    5600 4550
