File: KiCAD/base8x/base8x.kicad_pcb (KiCad board)
At the start: 4 copper layers, 350 x 110 mm, 58 parts, among them J1 Conn_02x05_Odd_Even, J10 Conn_02x14_Counter_Clockwise, J11 Conn_02x14_Counter_Clockwise, J12 Conn_02x14_Counter_Clockwise, J13 Conn_02x14_Counter_Clockwise, J14 Conn_02x14_Counter_Clockwise, J15 Conn_02x14_Counter_Clockwise, J16 Conn_01x14, J2 GS3, J3 Conn_02x14_Counter_Clockwise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

Commit message: update silk before order 629bf0f
Other:
- board text added: "629bf0f"
- board text removed: "20b2bb8"
Changed lines of the file:
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@@
     (effects (font (size 1.5 1.5) (thickness 0.3)) (justify left))
   )
-  (gr_text 20b2bb8 (at 25.5 47) (layer F.SilkS)
+  (gr_text 629bf0f (at 25.5 47) (layer F.SilkS)
     (effects (font (size 1.5 1.5) (thickness 0.3)))
   )

Commit message: add substrate markers
Parts:
- moved L1 82.6 mm to (27.2, -32.2), turned to 90 degrees
Other:
- board text added: "SUBSTRATE B"
- board text added: "SUBSTRATE C"
- board text added: "SUBSTRATE D"
- board text added: "SUBSTRATE E"
- board text added: "SUBSTRATE F"
- board text added: "SUBSTRATE G"
- board text added: "SUBSTRATE H"
- board text added: "b2b8b2c"
- board text removed: "629bf0f"
Changed lines of the file:
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@@
   (general
     (thickness 1.6)
-    (drawings 51)
+    (drawings 58)
     (tracks 220)
     (zones 0)
@@
   )
   (module myParts:logo (layer F.Cu)
-    (at 0 45.72)
-    (fp_text reference L1 (at 0 -4) (layer F.SilkS) hide
+    (at 27.25 -32.25 90)
+    (fp_text reference L1 (at 0 -4 90) (layer F.SilkS) hide
       (effects (font (size 1.524 1.524) (thickness 0.2)))
     )
-    (fp_text value GREY@CHRISTOFORO.NET (at 0 4) (layer F.SilkS) hide
+    (fp_text value GREY@CHRISTOFORO.NET (at 0 4 90) (layer F.SilkS) hide
       (effects (font (size 1.524 1.524) (thickness 0.2)))
     )
@@
     (descr "Generic Phoenix Contact connector footprint for: MC_1,5/8-GF-3.5; number of pins: 08; pin pitch: 3.50mm; Angled; threaded flange; footprint includes mount hole for mounting screw: ISO 1481-ST 2.2x4.5 C or ISO 7049-ST 2.2x4.5 C (http://www.fasteners.eu/standards/ISO/7049/) || order number: 1843855 8A 160V")
     (tags "phoenix_contact connector MC_01x08_GF_3.5mm_MH")
-    (fp_text reference J9 (at 12.25 -2.8) (layer F.SilkS)
+    (fp_text reference J9 (at -2.5 -2.35) (layer F.SilkS)
       (effects (font (size 1 1) (thickness 0.15)))
     )
@@
     (pad 1 np_thru_hole circle (at 0 0) (size 3.2 3.2) (drill 3.2) (layers *.Cu *.Mask))
   )
+  (gr_text "SUBSTRATE H" (at -280 45.75) (layer F.SilkS)
+    (effects (font (size 1.5 1.5) (thickness 0.3)))
+  )
+  (gr_text "SUBSTRATE G" (at -240 45.75) (layer F.SilkS)
+    (effects (font (size 1.5 1.5) (thickness 0.3)))
+  )
+  (gr_text "SUBSTRATE F" (at -200 45.75) (layer F.SilkS)
+    (effects (font (size 1.5 1.5) (thickness 0.3)))
+  )
+  (gr_text "SUBSTRATE E" (at -160 45.75) (layer F.SilkS)
+    (effects (font (size 1.5 1.5) (thickness 0.3)))
+  )
+  (gr_text "SUBSTRATE D" (at -120 45.75) (layer F.SilkS)
+    (effects (font (size 1.5 1.5) (thickness 0.3)))
+  )
+  (gr_text "SUBSTRATE C" (at -80 45.75) (layer F.SilkS)
+    (effects (font (size 1.5 1.5) (thickness 0.3)))
+  )
+  (gr_text "SUBSTRATE B" (at -40 45.75) (layer F.SilkS)
+    (effects (font (size 1.5 1.5) (thickness 0.3)))
+  )
   (gr_text 30x30mm (at 0 16.5) (layer F.SilkS)
     (effects (font (size 1.5 1.5) (thickness 0.3)))
@@
   (gr_line (start -12.5 -12.5) (end 12.5 -12.5) (layer F.SilkS) (width 0.15))
   (gr_line (start 39.69 52) (end 39.69 -52) (layer Edge.Cuts) (width 0.15))
-  (gr_text "SUBSTRATE A" (at 0 20) (layer F.SilkS)
+  (gr_text "SUBSTRATE A" (at 0 45.75) (layer F.SilkS)
     (effects (font (size 1.5 1.5) (thickness 0.3)))
   )
@@
     (effects (font (size 1.5 1.5) (thickness 0.3)) (justify left))
   )
-  (gr_text 629bf0f (at 25.5 47) (layer F.SilkS)
+  (gr_text b2b8b2c (at 29.75 -48 90) (layer F.SilkS)
     (effects (font (size 1.5 1.5) (thickness 0.3)))
   )

Commit message: update silk
Other:
- board text added: "779dfac"
- board text removed: "b2b8b2c"
Changed lines of the file:
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@@
     (effects (font (size 1.5 1.5) (thickness 0.3)) (justify left))
   )
-  (gr_text b2b8b2c (at 29.75 -48 90) (layer F.SilkS)
+  (gr_text 779dfac (at 29.75 -48 90) (layer F.SilkS)
     (effects (font (size 1.5 1.5) (thickness 0.3)))
   )
