File: KiCAD/springPins28x28MRG/springPins28x28MRG.kicad_pcb (KiCad board)
At the start: 2 copper layers, 28 x 28 mm, 25 parts, among them J1 CONN_02X06, J2 CONN_02X06

Commit message: mrg adapter board done
Parts:
- moved TP1 1.84 mm to (-10.3, 12.6)
- moved TP13 1.84 mm to (-10.3, -12.6)
- moved TP20 1.84 mm to (10.3, -12.6)
- moved TP8 1.84 mm to (10.3, 12.6)
- moved TP14 1.42 mm to (-7.73, -12.6)
- moved TP19 1.42 mm to (7.73, -12.6)
- moved TP2 1.42 mm to (-7.73, 12.6)
- moved TP7 1.42 mm to (7.73, 12.6)
- moved TP15 0.96 mm to (-4.27, -12.6)
- moved TP18 0.96 mm to (4.27, -12.6)
- moved TP3 0.96 mm to (-4.27, 12.6)
- moved TP6 0.96 mm to (4.27, 12.6)
- moved TP16 0.68 mm to (-1.73, -12.6)
- moved TP17 0.68 mm to (1.73, -12.6)
- moved TP4 0.68 mm to (-1.73, 12.6)
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Routing:
- net /V7: track 15.2 -> 18.5 mm
- net /I7: track 9.29 -> 11.3 mm
- net /VB: track 11.7 -> 13.4 mm
- net /VT: track 15.5 -> 16.9 mm
- net /IB: track 15.5 -> 16.7 mm
- net /IT: track 12.6 -> 13.7 mm
- net /I8: track 9.29 -> 10.3 mm
- net /V6: track 6.21 -> 7.14 mm
- net /V5: track 6.21 -> 7.14 mm
- net /I6: track 6.40 -> 7.14 mm
- net /I5: track 6.40 -> 7.14 mm
- net /V2: track 7.80 -> 8.36 mm
- net /V1: track 7.80 -> 8.36 mm
- net /V4: track 7.00 -> 7.52 mm
- net /V3: track 7.00 -> 7.52 mm

Commit message: update silk before order 629bf0f
Other:
- board text added: "629bf0f"
- board text removed: "20b2bb8"
Changed lines of the file:
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@@
   )
   (setup
-    (last_trace_width 0.56)
+    (last_trace_width 0.25)
     (user_trace_width 0.2)
     (user_trace_width 0.56)
@@
     (effects (font (size 1 1) (thickness 0.25)))
   )
-  (gr_text 20b2bb8 (at -12.5 -6.5 90) (layer F.SilkS)
+  (gr_text 629bf0f (at -12.5 -6.5 90) (layer F.SilkS)
     (effects (font (size 1 1) (thickness 0.175)))
   )

Commit message: fix dbg board adapter
Other:
- board text added: "MRG ~"
Changed lines of the file:
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@@
   (general
     (thickness 1.6)
-    (drawings 75)
+    (drawings 77)
     (tracks 90)
     (zones 0)
@@
     (pcbplotparams
       (layerselection 0x010fc_ffffffff)
-      (usegerberextensions true)
+      (usegerberextensions false)
       (usegerberattributes true)
       (usegerberadvancedattributes true)
-      (creategerberjobfile false)
+      (creategerberjobfile true)
       (excludeedgelayer true)
       (linewidth 0.150000)
@@
     )
   )
+  (gr_text "MRG\n~    " (at 13.75 9.75 90) (layer B.SilkS)
+    (effects (font (size 1.5 1.5) (thickness 0.3)) (justify mirror))
+  )
+  (gr_text "MRG\n~    " (at 13.75 9.75 90) (layer F.SilkS)
+    (effects (font (size 1.5 1.5) (thickness 0.3)))
+  )
   (gr_text 4I (at 1.3 8.285 90) (layer F.SilkS)

Commit message: add substrate markers
Other:
- board text added: "b2b8b2c"
- board text removed: "629bf0f"
Changed lines of the file:
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@@
     (effects (font (size 1 1) (thickness 0.25)))
   )
-  (gr_text 629bf0f (at -12.5 -6.5 90) (layer F.SilkS)
+  (gr_text b2b8b2c (at -12.5 -6.5 90) (layer F.SilkS)
     (effects (font (size 1 1) (thickness 0.175)))
   )

Commit message: update silk
Other:
- board text added: "779dfac"
- board text removed: "b2b8b2c"
Changed lines of the file:
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@@
     (effects (font (size 1 1) (thickness 0.25)))
   )
-  (gr_text b2b8b2c (at -12.5 -6.5 90) (layer F.SilkS)
+  (gr_text 779dfac (at -12.5 -6.5 90) (layer F.SilkS)
     (effects (font (size 1 1) (thickness 0.175)))
   )
