File: KiCAD/MKRPOEPB/MKRPOEPB.kicad_pcb (KiCad board)
At the start: 2 copper layers, 20 x 25 mm, 8 parts, among them J1 UDE_PoE, J2 Conn_01x02

Commit message: update silk
Other:
- board text added: "cd9cd45"
- board text removed: "234567"
Changed lines of the file:
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@@
       (outputformat 1)
       (mirror false)
-      (drillshape 1)
+      (drillshape 0)
       (scaleselection 1)
-      (outputdirectory ""))
+      (outputdirectory "output/"))
   )
   (net 0 "")
@@
       (xy 3.307808 1.349265)) (layer F.SilkS) (width 0))
   )
-  (gr_text 234567 (at 6 -24) (layer B.SilkS)
+  (gr_text cd9cd45 (at 6 -24) (layer B.SilkS)
     (effects (font (size 1 1) (thickness 0.15)) (justify mirror))
   )
-  (gr_text 234567 (at 6 -24) (layer F.SilkS)
+  (gr_text cd9cd45 (at 6 -24) (layer F.SilkS)
     (effects (font (size 1 1) (thickness 0.15)))
   )
