File: Myattempt/newMUX/newMUX.kicad_pcb (KiCad board)
At the start: 4 copper layers, 40 x 89 mm, 41 parts, among them J1 Conn_01x14, J2 Conn_02x06_Odd_Even, J3 Conn_02x06_Odd_Even, J4 Conn_01x14, U1 ASSR-1611, U10 ASSR-1611, U11 ASSR-1611, U12 ASSR-1611, U13 ASSR-1611, U14 ASSR-1611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

Commit message: adding ssr and sensor
Parts:
- removed L1: grey@mutovis.com, logo:text
Other:
- board text removed: "8694043"
