File: Myattempt/newMUX/newMUX.sch (KiCad schematic (older format))
At the start: 41 parts, among them J1 Conn_01x14, J2 Conn_02x06_Odd_Even, J3 Conn_02x06_Odd_Even, J4 Conn_01x14, U1 ASSR-1611, U10 ASSR-1611, U11 ASSR-1611, U12 ASSR-1611, U13 ASSR-1611, U14 ASSR-1611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

Commit message: adding ssr and sensor
Parts:
- removed L1: grey@mutovis.com, logo:text, symbol newMUX-rescue:logo_text-logo
- U1, U10, U11, U12, U13, U14, U15, U16, U17, U18, U19, U2, U20, U21, U3, U4, U5, U6, U7, U8, U9: symbol myParts:ASSR-1611 -> newMUX-rescue:ASSR-1611-myParts
Changed lines of the file:
@@
 $EndComp
 $Comp
-L myParts:ASSR-1611 U8
+L newMUX-rescue:ASSR-1611-myParts U8
 U 1 1 59B12693
 P 1850 4650
@@
 $EndComp
 $Comp
-L myParts:ASSR-1611 U7
+L newMUX-rescue:ASSR-1611-myParts U7
 U 1 1 59B14970
 P 1850 4200
@@
 $EndComp
 $Comp
-L myParts:ASSR-1611 U10
+L newMUX-rescue:ASSR-1611-myParts U10
 U 1 1 59B15747
 P 1850 5550
@@
 $EndComp
 $Comp
-L myParts:ASSR-1611 U9
+L newMUX-rescue:ASSR-1611-myParts U9
 U 1 1 59B1574D
 P 1850 5100
@@
 $EndComp
 $Comp
-L myParts:ASSR-1611 U6
+L newMUX-rescue:ASSR-1611-myParts U6
 U 1 1 59B15786
 P 1850 3750
@@
 $EndComp
 $Comp
-L myParts:ASSR-1611 U3
+L newMUX-rescue:ASSR-1611-myParts U3
 U 1 1 59B15ABC
 P 1850 2400
@@
 $EndComp
 $Comp
-L myParts:ASSR-1611 U2
+L newMUX-rescue:ASSR-1611-myParts U2
 U 1 1 59B15AC2
 P 1850 1950
@@
 $EndComp
 $Comp
-L myParts:ASSR-1611 U5
+L newMUX-rescue:ASSR-1611-myParts U5
 U 1 1 59B15AC8
 P 1850 3300
@@
 $EndComp
 $Comp
-L myParts:ASSR-1611 U4
+L newMUX-rescue:ASSR-1611-myParts U4
 U 1 1 59B15ACE
 P 1850 2850
@@
 $EndComp
 $Comp
-L myParts:ASSR-1611 U1
+L newMUX-rescue:ASSR-1611-myParts U1
 U 1 1 59B15AD4
 P 1850 1500
@@
 $EndComp
 $Comp
-L myParts:ASSR-1611 U18
+L newMUX-rescue:ASSR-1611-myParts U18
 U 1 1 59B16DFF
 P 4050 4650
@@
 $EndComp
 $Comp
-L myParts:ASSR-1611 U17
+L newMUX-rescue:ASSR-1611-myParts U17
 U 1 1 59B16E05
 P 4050 4200
@@
 $EndComp
 $Comp
-L myParts:ASSR-1611 U20
+L newMUX-rescue:ASSR-1611-myParts U20
 U 1 1 59B16E0B
 P 4050 5550
@@
 $EndComp
 $Comp
-L myParts:ASSR-1611 U19
+L newMUX-rescue:ASSR-1611-myParts U19
 U 1 1 59B16E11
 P 4050 5100
@@
 $EndComp
 $Comp
-L myParts:ASSR-1611 U16
+L newMUX-rescue:ASSR-1611-myParts U16
 U 1 1 59B16E17
 P 4050 3750
@@
 $EndComp
 $Comp
-L myParts:ASSR-1611 U13
+L newMUX-rescue:ASSR-1611-myParts U13
 U 1 1 59B16E1D
 P 4050 2400
@@
 $EndComp
 $Comp
-L myParts:ASSR-1611 U12
+L newMUX-rescue:ASSR-1611-myParts U12
 U 1 1 59B16E23
 P 4050 1950
@@
 $EndComp
 $Comp
-L myParts:ASSR-1611 U15
+L newMUX-rescue:ASSR-1611-myParts U15
 U 1 1 59B16E29
 P 4050 3300
@@
 $EndComp
 $Comp
-L myParts:ASSR-1611 U14
+L newMUX-rescue:ASSR-1611-myParts U14
 U 1 1 59B16E2F
 P 4050 2850
@@
 $EndComp
 $Comp
-L myParts:ASSR-1611 U11
+L newMUX-rescue:ASSR-1611-myParts U11
 U 1 1 59B16E35
 P 4050 1500
@@
 V_D
 $Comp
-L myParts:ASSR-1611 U21
+L newMUX-rescue:ASSR-1611-myParts U21
 U 1 1 59B306AE
 P 6050 1100
@@
 VB
 $Comp
-L newMUX-rescue:logo_text-logo L1
-U 1 1 59B41702
-P 9000 6750
-F 0 "L1" H 9000 6625 60  0001 C CNN
-F 1 "grey@mutovis.com" H 9000 6450 100 0000 C CNB
-F 2 "logo:text" H 9000 6750 60  0001 C CNN
-F 3 "" H 9000 6750 60  0001 C CNN
-	1    9000 6750
-	1    0    0    -1
-$EndComp
-$Comp
 L Device:R R3
